File: mcu.kicad_sch (KiCad schematic)
At the start: 76 parts, among them J2 Conn_02x12_Odd_Even, J3 DE9_Pins, J4 Conn_01x12, J5 Conn_ARM_JTAG_SWD_20, J6 Conn_02x12_Odd_Even, J7 USB_B_Mini, J9 RJ45_Hanrun_HR911105A_Horizon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, U15 MAX3232, U16 STM32F407VETx, U18 DP83848C, Y1 8MHz, Y2 32.768KHz, Y4 25MHz

Commit message: update
Parts:
- removed R100, R103, R104: 33R, Resistor_SMD:R_0603_1608Metric, symbol Device:R_Small
- added R55: 2.2K, Resistor_SMD:R_0603_1608Metric, symbol Device:R_Small
- R101: value 33R -> 2.2K
Connections:
- net +3.3V: now also R101.1, R55.1
- net PA7-RMII-CRS-DV: now also U18.40 (CRS/CRS_DV/LED_CFG), R55.2; no longer R101.1
Other:
- moved on the sheet: R101, R110, Y4

Commit message: update
Parts:
- removed R95: 33R, Resistor_SMD:R_0603_1608Metric, symbol Device:R_Small
- added J10: Conn_02x12_Odd_Even, Connector_PinHeader_2.54mm:PinHeader_2x12_P2.54mm_Vertical, symbol Connector_Generic:Conn_02x12_Odd_Even
- added J11, J7: Conn_02x04_Odd_Even, Connector_PinHeader_2.54mm:PinHeader_2x04_P2.54mm_Vertical, symbol Connector_Generic:Conn_02x04_Odd_Even
- added R43, R52, R60: DNI, Resistor_SMD:R_0603_1608Metric, symbol Device:R_Small
- added R44, R53, R54, R55: 0R, Resistor_SMD:R_0603_1608Metric, symbol Device:R_Small
- added R59: 1.5K, Resistor_SMD:R_0603_1608Metric, symbol Device:R_Small
- added R70, R71: 33R, Resistor_SMD:R_0603_1608Metric, symbol Device:R_Small
- C101: renamed from C107; footprint Capacitor_SMD:C_01005_0402Metric_Pad0.57x0.30mm_HandSolder -> Capacitor_SMD:C_0603_1608Metric
- C102: renamed from C108; footprint Capacitor_SMD:C_01005_0402Metric_Pad0.57x0.30mm_HandSolder -> Capacitor_SMD:C_0603_1608Metric
- C103: renamed from C104; footprint Capacitor_SMD:C_01005_0402Metric_Pad0.57x0.30mm_HandSolder -> Capacitor_SMD:C_0603_1608Metric
- C104: renamed from C109; footprint Capacitor_SMD:C_01005_0402Metric_Pad0.57x0.30mm_HandSolder -> Capacitor_SMD:C_0603_1608Metric
- C105: renamed from C110; footprint Capacitor_SMD:C_01005_0402Metric_Pad0.57x0.30mm_HandSolder -> Capacitor_SMD:C_0603_1608Metric
- C106: renamed from C111; footprint Capacitor_SMD:C_01005_0402Metric_Pad0.57x0.30mm_HandSolder -> Capacitor_SMD:C_0603_1608Metric
- C107: renamed from C112; footprint Capacitor_SMD:C_01005_0402Metric_Pad0.57x0.30mm_HandSolder -> Capacitor_SMD:C_0603_1608Metric
- C108: renamed from C121; value 22pF -> 33pF; footprint Capacitor_SMD:C_01005_0402Metric_Pad0.57x0.30mm_HandSolder -> Capacitor_SMD:C_0603_1608Metric
- C109: renamed from C126; value 22pF -> 33pF; footprint Capacitor_SMD:C_01005_0402Metric_Pad0.57x0.30mm_HandSolder -> Capacitor_SMD:C_0603_1608Metric
- C110: renamed from C100; footprint Capacitor_SMD:C_01005_0402Metric_Pad0.57x0.30mm_HandSolder -> Capacitor_SMD:C_0603_1608Metric
- C111: renamed from C99; footprint Capacitor_SMD:C_01005_0402Metric_Pad0.57x0.30mm_HandSolder -> Capacitor_SMD:C_0603_1608Metric
- C112: renamed from C101; footprint Capacitor_SMD:C_01005_0402Metric_Pad0.57x0.30mm_HandSolder -> Capacitor_SMD:C_0603_1608Metric
- C113: renamed from C105; footprint Capacitor_SMD:C_01005_0402Metric_Pad0.57x0.30mm_HandSolder -> Capacitor_SMD:C_0603_1608Metric
- C114: renamed from C106; footprint Capacitor_SMD:C_01005_0402Metric_Pad0.57x0.30mm_HandSolder -> Capacitor_SMD:C_0603_1608Metric
- C115: renamed from C122; footprint Capacitor_SMD:C_01005_0402Metric_Pad0.57x0.30mm_HandSolder -> Capacitor_SMD:C_0603_1608Metric
- C116: renamed from C123; footprint Capacitor_SMD:C_01005_0402Metric_Pad0.57x0.30mm_HandSolder -> Capacitor_SMD:C_0603_1608Metric
- C117: renamed from C124; footprint Capacitor_SMD:C_01005_0402Metric_Pad0.57x0.30mm_HandSolder -> Capacitor_SMD:C_0603_1608Metric
- C118: renamed from C125; footprint Capacitor_SMD:C_01005_0402Metric_Pad0.57x0.30mm_HandSolder -> Capacitor_SMD:C_0603_1608Metric
- C119: renamed from C120; footprint Capacitor_SMD:C_01005_0402Metric_Pad0.57x0.30mm_HandSolder -> Capacitor_SMD:C_0603_1608Metric
- J2: renamed from J7; footprint Connector_USB:USB_Mini-B_Tensility_54-00023_Vertical -> Connector_USB:USB_Mini-B_Wuerth_65100516121_Horizontal
- R61: renamed from R114; value 33R -> 0R
- renumbered J5 to J3, J3 to J4, J9 to J5, J2 to J8, J4 to J9, R44 to R46, R43 to R47, R53 to R48, R54 to R49, R52 to R50, R46 to R51, R55 to R56, R110 to R57, R101 to R58, R91 to R62, R92 to R63, R93 to R64, R94 to R65, R96 to R66, R97 to R67, R98 to R68, R99 to R69, R106 to R72, R108 to R73, R47 to R74, R51 to R75, R48 to R76, R49 to R77, R50 to R78, R85 to R79, R102 to R80, R105 to R81, R107 to R82, R109 to R83, R111 to R84, R112 to R85, R113 to R88, R88 to R89, R89 to R90, R90 to R91, U16 to U15, U15 to U16, U18 to U17, Y4 to Y3
Connections:
- net +3.3V: now also R47.2, J7.2 (Pin_2), J7.4 (Pin_4), J7.6 (Pin_6), J7.8 (Pin_8), R43.2, R52.2, R59.1; no longer R47.1
- net +5V: now also J11.2 (Pin_2), J11.4 (Pin_4), J11.6 (Pin_6), J11.8 (Pin_8); no longer J6.2 (Pin_2), J6.4 (Pin_4)
- net GND: now also R57.2, SW1.2, J10.22 (Pin_22), J10.23 (Pin_23), J10.24 (Pin_24), J11.1 (Pin_1), J11.3 (Pin_3), J11.5 (Pin_5), J11.7 (Pin_7), J7.1 (Pin_1), J7.3 (Pin_3), J7.5 (Pin_5), J7.7 (Pin_7), R44.2, R53.2; no longer J6.1 (Pin_1), J6.3 (Pin_3), R51.1, R57.1, SW1.1
- net PA1-RMII-REF-CLK: now also R60.2
- net PA2-ETH-MDIO: now also R59.2
- net PA7-RMII-CRS-DV: now also R54.1, R55.1; no longer R56.2, U17.40 (CRS/CRS_DV/LED_CFG)
- net PA8-ETH-RESET: now also R57.1; no longer R57.2
- net RESET: now also R47.1, SW1.1; no longer R47.2, SW1.2
- net PB7: now reaches J6.10 (Pin_10)
- net PB7: now also U15.93 (PB7)
- net PB8: now reaches J6.11 (Pin_11)
- net PB8: now also U15.95 (PB8)
- net PB9: now reaches J6.12 (Pin_12)
- net PB9: now also U15.96 (PB9)
- net PB14: now reaches J6.13 (Pin_13)
- net PB14: now also U15.53 (PB14)
- net PB15: now reaches J6.14 (Pin_14)
- net PB15: now also U15.54 (PB15)
- net PC0: now reaches J6.15 (Pin_15)
- net PC0: now also U15.15 (PC0)
- net PC2: now reaches J6.16 (Pin_16)
- net PC2: now also U15.17 (PC2)
- net PC3: now reaches J6.17 (Pin_17)
- net PC3: now also U15.18 (PC3)
- net PC6: now reaches J6.18 (Pin_18)
- net PC6: now also U15.63 (PC6)
- net PC7: now reaches J6.19 (Pin_19)
- net PC7: now also U15.64 (PC7)
- net PC8: now reaches J6.20 (Pin_20)
- net PC8: now also U15.65 (PC8)
- net PC9: now reaches J6.21 (Pin_21)
- net PC9: now also U15.66 (PC9)
- net PC10: now reaches J6.22 (Pin_22)
- net PC10: now also U15.78 (PC10)
- net PC11: now reaches J6.23 (Pin_23)
- net PC11: now also U15.79 (PC11)
- net PC12: now reaches J6.24 (Pin_24)
- net PC12: now also U15.80 (PC12)
- net PA6: now reaches J6.5 (Pin_5)
- net PA6: now also U15.31 (PA6)
- net PB0: now reaches J6.6 (Pin_6)
- net PB0: now also U15.35 (PB0)
- net PB1: now reaches J6.7 (Pin_7)
- net PB1: now also U15.36 (PB1)
- net PB5: now reaches J6.8 (Pin_8)
- net PB5: now also U15.91 (PB5)
- net PB6: now reaches J6.9 (Pin_9)
- net PB6: now also U15.92 (PB6)
- net at C108.2, U17.34 (X1), Y3.2: now also R60.1
- net at U17.39 (RX_DV/MII_MODE): now also R70.2; no longer R58.2
- net PE2: now reaches U15.1 (PE2)
- net PE2: now also J9.3 (Pin_3)
- net PE3: now reaches U15.2 (PE3)
- net PE3: now also J9.4 (Pin_4)
- net PA0: now reaches U15.23 (PA0)
- net PA0: now also J6.1 (Pin_1)
- net PA3: now reaches U15.26 (PA3)
- net PA3: now also J6.2 (Pin_2)
- net PA4: now reaches U15.29 (PA4)
- net PA4: now also J6.3 (Pin_3)
- net PE4: now reaches U15.3 (PE4)
- net PE4: now also J9.5 (Pin_5)
- net PA5: now reaches U15.30 (PA5)
- net PA5: now also J6.4 (Pin_4)
- net PE7: now reaches U15.38 (PE7)
- net PE7: now also J9.8 (Pin_8)
- net PE8: now reaches U15.39 (PE8)
- net PE8: now also J9.9 (Pin_9)
- net PE5: now reaches U15.4 (PE5)
- net PE5: now also J9.6 (Pin_6)
- net PE9: now reaches U15.40 (PE9)
- net PE9: now also J9.10 (Pin_10)
- net PE10: now reaches U15.41 (PE10)
- net PE10: now also J9.11 (Pin_11)
- net PE11: now reaches U15.42 (PE11)
- net PE11: now also J9.12 (Pin_12)
- net PE12: now reaches U15.43 (PE12)
- net PE12: now also J10.18 (Pin_18)
- net PE13: now reaches U15.44 (PE13)
- net PE13: now also J10.19 (Pin_19)
- net PE14: now reaches U15.45 (PE14)
- net PE14: now also J10.20 (Pin_20)
- net PE15: now reaches U15.46 (PE15)
- net PE15: now also J10.21 (Pin_21)
- net PE6: now reaches U15.5 (PE6)
- net PE6: now also J9.7 (Pin_7)
- net PD8: now reaches U15.55 (PD8)
- net PD8: now also J10.10 (Pin_10)
- net PD9: now reaches U15.56 (PD9)
- net PD9: now also J10.11 (Pin_11)
- net PD10: now reaches U15.57 (PD10)
- net PD10: now also J10.12 (Pin_12)
- net PD11: now reaches U15.58 (PD11)
- net PD11: now also J10.13 (Pin_13)
- net PD12: now reaches U15.59 (PD12)
- net PD12: now also J10.14 (Pin_14)
- net PD13: now reaches U15.60 (PD13)
- net PD13: now also J10.15 (Pin_15)
- net PD14: now reaches U15.61 (PD14)
- net PD14: now also J10.16 (Pin_16)
- net PD15: now reaches U15.62 (PD15)
- net PD15: now also J10.17 (Pin_17)
- net PC13: now reaches U15.7 (PC13)
- net PC13: now also J10.1 (Pin_1)
- net PD0: now reaches U15.81 (PD0)
- net PD0: now also J10.2 (Pin_2)
- net PD1: now reaches U15.82 (PD1)
- net PD1: now also J10.3 (Pin_3)
- net PD2: now reaches U15.83 (PD2)
- net PD2: now also J10.4 (Pin_4)
- net PD3: now reaches U15.84 (PD3)
- net PD3: now also J10.5 (Pin_5)
- net PD4: now reaches U15.85 (PD4)
- net PD4: now also J10.6 (Pin_6)
- net PD5: now reaches U15.86 (PD5)
- net PD5: now also J10.7 (Pin_7)
- net PD6: now reaches U15.87 (PD6)
- net PD6: now also J10.8 (Pin_8)
- net PD7: now reaches U15.88 (PD7)
- net PD7: now also J10.9 (Pin_9)
- net PE0: now reaches U15.97 (PE0)
- net PE0: now also J9.1 (Pin_1)
- net PE1: now reaches U15.98 (PE1)
- net PE1: now also J9.2 (Pin_2)
- net Earth: no longer names the net of R46.1
- net Earth: now also R43.1, R44.1
- new net: R51.1, R52.1, R53.1
- new net: R54.2, R56.2, R70.1
- new net: R71.2, U17.40 (CRS/CRS_DV/LED_CFG)
- new net: R55.2, R58.2, R71.1
Other:
- moved on the sheet: BT1, C101, C102, C103, C104, C105, C106, C107, C108, C109, C110, C111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

Commit message: update
Parts:
- renumbered C111 to C115, C103 to C116, C110 to C117, C112 to C118, C113 to C119, C114 to C120, C101 to C121, C102 to C122, C104 to C123, C105 to C124, C106 to C125, C107 to C126, C119 to C127, C108 to C128, C115 to C129, C116 to C130, C117 to C131, C118 to C132, C109 to C133, J5 to J10, J2 to J11, J8 to J2, J9 to J3, J6 to J5, J10 to J6, J11 to J8, J3 to J9, R47 to R43, R43 to R44, R44 to R45, R45 to R47, R52 to R48, R51 to R49, R53 to R50, R74 to R51, R76 to R52, R77 to R53, R78 to R54, R75 to R55, R50 to R56, R79 to R57, R86 to R58, R87 to R59, R89 to R60, R90 to R61, R91 to R62, R62 to R63, R63 to R64, R64 to R65, R65 to R66, R66 to R67, R48 to R68, R49 to R69, R67 to R70, R68 to R71, R56 to R72, R58 to R73, R59 to R74, R69 to R75, R54 to R76, R70 to R77, R80 to R78, R55 to R79, R71 to R80, R72 to R82, R82 to R83, R73 to R84, R83 to R85, R57 to R86, R84 to R87, R85 to R88, R60 to R89, R88 to R90, R61 to R91, U16 to U15, U15 to U16
Other:
- moved on the sheet: C121, C122, C123, C124, C127, C128, C129, C130, C131, C132, C133, J10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

Commit message: update
Parts:
- removed J2, J5: Conn_02x12_Odd_Even, Connector_PinHeader_2.54mm:PinHeader_2x12_P2.54mm_Vertical, symbol Connector_Generic:Conn_02x12_Odd_Even
- removed J3: Conn_01x12, Connector_PinHeader_2.54mm:PinHeader_1x12_P2.54mm_Vertical, symbol Connector_Generic:Conn_01x12
- added H1, H2, H3, H4: MountingHole, MountingHole:MountingHole_2.2mm_M2, symbol Mechanical:MountingHole
- added J2: Conn_02x08_Odd_Even, Connector_PinHeader_2.54mm:PinHeader_2x08_P2.54mm_Vertical, symbol Connector_Generic:Conn_02x08_Odd_Even
- added J3: Conn_01x08, Connector_PinHeader_2.54mm:PinHeader_1x08_P2.54mm_Vertical, symbol Connector_Generic:Conn_01x08
- added J6: Conn_02x16_Odd_Even, Connector_PinHeader_2.54mm:PinHeader_2x16_P2.54mm_Vertical, symbol Connector_Generic:Conn_02x16_Odd_Even
- J4: footprint Connector_Dsub:DSUB-9_Pins_Horizontal_P2.77x2.54mm_EdgePinOffset9.40mm -> Connector_Dsub:DSUB-9_Pins_Horizontal_P2.77x2.84mm_EdgePinOffset4.94mm_Housed_MountingHolesOffset4.94mm
- Y1: footprint Crystal:Crystal_HC49-4H_Vertical -> Crystal:Crystal_SMD_5032-2Pin_5.0x3.2mm
- Y3: footprint Crystal:Crystal_HC49-4H_Vertical -> Crystal:Crystal_SMD_HC49-SD
- renumbered C132 to C100, C133 to C101, C115 to C83, C116 to C84, C117 to C85, C118 to C86, C119 to C87, C120 to C88, C121 to C89, C122 to C90, C123 to C91, C124 to C92, C125 to C93, C126 to C94, C127 to C95, C128 to C96, C129 to C97, C130 to C98, C131 to C99, J6 to J5, J8 to J7, J7 to J8, R43 to R31, R44 to R32, R45 to R33, R46 to R34, R47 to R35, R48 to R36, R49 to R37, R50 to R38, R51 to R39, R52 to R40, R53 to R41, R54 to R42, R55 to R43, R56 to R44, R57 to R45, R58 to R46, R59 to R47, R60 to R48, R61 to R49, R62 to R50, R63 to R51, R64 to R52, R65 to R53, R66 to R54, R67 to R55, R70 to R56, R71 to R57, R72 to R58, R73 to R59, R74 to R60, R75 to R61, R68 to R62, R76 to R63, R77 to R64, R69 to R65, R78 to R66, R79 to R67, R80 to R68, R81 to R69, R82 to R70, R83 to R71, R84 to R72, R85 to R73, R86 to R74, R87 to R75, R88 to R76, R89 to R77, R90 to R78, R91 to R79, U15 to U11, U16 to U12, U17 to U13
Connections:
- net PC0 is gone; now on net PC0-ETH-RESET: U12.15 (PC0)
- net +7V_M1: now also J2.2 (Pin_2)
- net +7V_M2: now also J2.4 (Pin_4)
- net +7V_M3: now also J2.6 (Pin_6)
- net +7V_M4: now also J2.8 (Pin_8)
- net +7V_M5: now also J2.10 (Pin_10)
- net +7V_M6: now also J2.12 (Pin_12)
- net +7V_M7: now also J2.14 (Pin_14)
- net +7V_M8: now also J2.16 (Pin_16)
- net GND: now also J2.1 (Pin_1), J2.11 (Pin_11), J2.13 (Pin_13), J2.15 (Pin_15), J2.3 (Pin_3), J2.5 (Pin_5), J2.7 (Pin_7), J2.9 (Pin_9); no longer J5.22 (Pin_22), J5.23 (Pin_23), J5.24 (Pin_24)
- net PC13: no longer J5.1 (Pin_1)
- net PD0: no longer J5.2 (Pin_2)
- net PD1: no longer J5.3 (Pin_3)
- net PD10: no longer J5.12 (Pin_12)
- net PD11: no longer J5.13 (Pin_13)
- net PD12: no longer J5.14 (Pin_14)
- net PD13: no longer J5.15 (Pin_15)
- net PD14: no longer J5.16 (Pin_16)
- net PD15: no longer J5.17 (Pin_17)
- net PD2: no longer J5.4 (Pin_4)
- net PD3: no longer J5.5 (Pin_5)
- net PD4: no longer J5.6 (Pin_6)
- net PD5: no longer J5.7 (Pin_7)
- net PD6: no longer J5.8 (Pin_8)
- net PD7: no longer J5.9 (Pin_9)
- net PD8: no longer J5.10 (Pin_10)
- net PD9: no longer J5.11 (Pin_11)
- net PE12: no longer J5.18 (Pin_18)
- net PE13: no longer J5.19 (Pin_19)
- net PE14: no longer J5.20 (Pin_20)
- net PE15: no longer J5.21 (Pin_21)
- net PA8-ETH-RESET renamed PC0-ETH-RESET
- net PC0-ETH-RESET: no longer U12.67 (PA8)
- new net PA8: U12.67 (PA8)
Other:
- moved on the sheet: J8

Commit message: update
Parts:
- removed J5: Conn_02x12_Odd_Even, Connector_PinHeader_2.54mm:PinHeader_2x12_P2.54mm_Vertical, symbol Connector_Generic:Conn_02x12_Odd_Even
- added C102, C103, C104, C105: 0.1uF, Capacitor_SMD:C_0603_1608Metric, symbol Device:C_Small
- added D1, D2, D3, D4, D5, D6: LED, LED_SMD:LED_0603_1608Metric, symbol Device:LED
- added J9: Conn_02x04_Odd_Even, Connector_PinHeader_2.54mm:PinHeader_2x04_P2.54mm_Vertical, symbol Connector_Generic:Conn_02x04_Odd_Even
- added R80, R81, R82, R83: 10K, Resistor_SMD:R_0603_1608Metric, symbol Device:R_Small
- added R84, R85, R86, R87, R88, R89: 680, Resistor_SMD:R_0603_1608Metric, symbol Device:R_Small
- added SW2, SW3, SW4, SW5: ~, Button_Switch_SMD:SW_SPST_B3SL-1002P, symbol Switch:SW_Push
- Y2: footprint Crystal:Crystal_C26-LF_D2.1mm_L6.5mm_Horizontal -> Crystal:Crystal_SMD_3215-2Pin_3.2x1.5mm
- Y3: footprint Crystal:Crystal_SMD_HC49-SD -> Crystal:Crystal_SMD_5032-2Pin_5.0x3.2mm
- renumbered J8 to J10, J7 to J11, J10 to J2, J11 to J3, J6 to J4, J4 to J5, J9 to J6, J3 to J7, J2 to J8
Connections:
- net +3.3V: now also R80.2, R81.2, R82.2, R83.2
- net GND: now also C102.1, C103.1, C104.1, C105.1, D1.1 (K), D2.1 (K), D3.1 (K), D4.1 (K), D5.1 (K), D6.1 (K), J9.8 (Pin_8), SW2.2, SW3.2, SW4.2, SW5.2
- net PA0: now also J9.3 (Pin_3)
- net PA3: now also J9.4 (Pin_4)
- net PA4: now also J9.1 (Pin_1)
- net PA5: now also J9.2 (Pin_2)
- net PA6: now also J9.5 (Pin_5)
- net PA8: now also J4.9 (Pin_9)
- net PB0: now also J4.32 (Pin_32)
- net PB1: now also J9.7 (Pin_7)
- net PB14: now also J4.23 (Pin_23)
- net PB15: now also J4.22 (Pin_22)
- net PB5: now also J4.5 (Pin_5)
- net PB6: now also R87.2
- net PB7: now also R86.2
- net PB8: now also R85.2
- net PB9: now also R84.2
- net PC10: now also J4.6 (Pin_6)
- net PC11: now also J4.4 (Pin_4)
- net PC12: now also J4.3 (Pin_3)
- net PC13: now also J7.6 (Pin_6)
- net PC2: now also J7.7 (Pin_7)
- net PC3: now also J7.8 (Pin_8)
- net PC6: now also J4.13 (Pin_13)
- net PC7: now also J4.12 (Pin_12)
- net PC8: now also J4.11 (Pin_11)
- net PC9: now also J4.10 (Pin_10)
- net PD0: now also J4.7 (Pin_7)
- net PD1: now also J4.8 (Pin_8)
- net PD10: now also J4.19 (Pin_19)
- net PD11: now also J4.18 (Pin_18)
- net PD12: now also J4.17 (Pin_17)
- net PD13: now also J4.16 (Pin_16)
- net PD14: now also J4.15 (Pin_15)
- net PD15: now also J4.14 (Pin_14)
- net PD2: now also J4.2 (Pin_2)
- net PD3: now also J4.1 (Pin_1)
- net PD4: now also C102.2, R80.1, SW2.1
- net PD5: now also C103.2, R81.1, SW3.1
- net PD6: now also C104.2, R82.1, SW4.1
- net PD7: now also C105.2, R83.1, SW5.1
- net PD8: now also J4.21 (Pin_21)
- net PD9: now also J4.20 (Pin_20)
- net PE0: now also R88.2
- net PE1: now also R89.2
- net PE10: now also J4.24 (Pin_24)
- net PE11: now also J4.25 (Pin_25)
- net PE12: now also J4.29 (Pin_29)
- net PE13: now also J4.26 (Pin_26)
- net PE14: now also J4.28 (Pin_28)
- net PE15: now also J4.27 (Pin_27)
- net PE2: now also J7.3 (Pin_3)
- net PE3: now also J7.1 (Pin_1)
- net PE4: now also J7.2 (Pin_2)
- net PE5: now also J7.4 (Pin_4)
- net PE6: now also J7.5 (Pin_5)
- net PE7: now also J4.31 (Pin_31)
- net PE8: now also J4.30 (Pin_30)
- net PE9: now also J9.6 (Pin_6)
- net +7V_M1 renamed V_M1
- net +7V_M2 renamed V_M2
- net +7V_M3 renamed V_M3
- net +7V_M4 renamed V_M4
- net +7V_M5 renamed V_M5
- net +7V_M6 renamed V_M6
- net +7V_M7 renamed V_M7
- net +7V_M8 renamed V_M8
- new net: D4.2 (A), R85.1
- new net: D5.2 (A), R84.1
- new net: D2.2 (A), R87.1
- new net: D6.2 (A), R89.1
- new net: D3.2 (A), R86.1
- new net: D1.2 (A), R88.1
Other:
- moved on the sheet: H1, H2, H3, H4, J10, J11, J3, J4, J6, J7, R39, R40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

Commit message: update
Parts:
- added C106, C107: 100nF, Capacitor_SMD:C_0603_1608Metric, symbol Device:C_Small
- C99: value 100nF -> 10uF
- SW1, SW2, SW3, SW4, SW5: footprint Button_Switch_SMD:SW_SPST_B3SL-1002P -> Button_Switch_SMD:SW_Push_1P1T_NO_CK_KSC7xxJ
Connections:
- net +3.3V: now also C106.2, C107.2
- net GND: now also C106.1, C107.1
Other:
- moved on the sheet: H1, H2, H3, H4, J10, J11, J3, J4, J5, J7, J8, J9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

Commit message: update
Parts:
- D1: renamed from D2; value LED -> WHITE LED
- D2: renamed from D3; value LED -> WHITE LED
- D3: renamed from D4; value LED -> ORANGE LED
- D4: renamed from D5; value LED -> ORANGE LED
- D5: renamed from D1; value LED -> RED LED
- D6: value LED -> RED LED
- R84: renamed from R87; value 680 -> 220
- R85: renamed from R86; value 680 -> 220
- R86: renamed from R85; value 680 -> 220
- R87: renamed from R84; value 680 -> 220
- R88, R89: value 680 -> 220
Changed lines of the file:
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@@
 		(on_board yes)
 		(dnp no)
-		(property "Reference" "R85"
+		(property "Reference" "R86"
 			(at 346.456 146.812 90)
 			(effects
@@
 			)
 		)
-		(property "Value" "680"
+		(property "Value" "220"
 			(at 346.456 150.876 90)
 			(effects
@@
 			(project "sac_board"
 				(path "/74ff6d0b-648c-43d9-a5b1-cc8d6cd1c1ef/52e20330-efd4-4d59-a57b-f0ea443c9be4"
-					(reference "R85")
+					(reference "R86")
 					(unit 1)
 				)
@@
 		(on_board yes)
 		(dnp no)
-		(property "Reference" "R84"
+		(property "Reference" "R87"
 			(at 379.476 146.812 90)
 			(effects
@@
 			)
 		)
-		(property "Value" "680"
+		(property "Value" "220"
 			(at 379.476 150.876 90)
 			(effects
@@
 			(project "sac_board"
 				(path "/74ff6d0b-648c-43d9-a5b1-cc8d6cd1c1ef/52e20330-efd4-4d59-a57b-f0ea443c9be4"
-					(reference "R84")
+					(reference "R87")
 					(unit 1)
 				)
@@
 		(on_board yes)
 		(dnp no)
-		(property "Reference" "D2"
+		(property "Reference" "D1"
 			(at 288.29 142.748 0)
 			(effects
@@
 			)
 		)
-		(property "Value" "LED"
+		(property "Value" "WHITE LED"
 			(at 288.29 145.288 0)
 			(effects
@@
 			(project "sac_board"
 				(path "/74ff6d0b-648c-43d9-a5b1-cc8d6cd1c1ef/52e20330-efd4-4d59-a57b-f0ea443c9be4"
-					(reference "D2")
+					(reference "D1")
 					(unit 1)
 				)
@@
 			)
 		)
-		(property "Value" "680"
+		(property "Value" "220"
 			(at 379.476 164.846 90)
 			(effects
@@
 			)
 		)
-		(property "Value" "LED"
+		(property "Value" "RED LED"
 			(at 387.604 159.512 0)
 			(effects
@@
 		)
 		(property "Value" "GND"
-			(at 363.22 166.37 0)
+			(at 365.76 162.5599 0)
 			(effects
 				(font
 					(size 1.27 1.27)
 				)
+				(justify left)
 			)
 		)
@@
 		(on_board yes)
 		(dnp no)
-		(property "Reference" "D3"
+		(property "Reference" "D2"
 			(at 322.58 142.748 0)
 			(effects
@@
 			)
 		)
-		(property "Value" "LED"
+		(property "Value" "WHITE LED"
 			(at 322.58 145.288 0)
 			(effects
@@
 			(project "sac_board"
 				(path "/74ff6d0b-648c-43d9-a5b1-cc8d6cd1c1ef/52e20330-efd4-4d59-a57b-f0ea443c9be4"
-					(reference "D3")
+					(reference "D2")
 					(unit 1)
 				)
@@
 		)
 		(property "Value" "GND"
-			(at 294.64 153.67 0)
+			(at 297.18 149.8599 0)
 			(effects
 				(font
 					(size 1.27 1.27)
 				)
+				(justify left)
 			)
 		)
@@
 		(on_board yes)
 		(dnp no)
-		(property "Reference" "D1"
+		(property "Reference" "D5"
 			(at 357.124 155.702 0)
 			(effects
@@
 			)
 		)
-		(property "Value" "LED"
+		(property "Value" "RED LED"
 			(at 357.124 158.242 0)
 			(effects
@@
 			(project ""
 				(path "/74ff6d0b-648c-43d9-a5b1-cc8d6cd1c1ef/52e20330-efd4-4d59-a57b-f0ea443c9be4"
-					(reference "D1")
+					(reference "D5")
 					(unit 1)
 				)
@@
 			)
 		)
-		(property "Value" "680"
+		(property "Value" "220"
 			(at 348.996 163.576 90)
 			(effects
@@
 		)
 		(property "Value" "GND"
-			(at 361.95 153.67 0)
+			(at 364.49 149.8599 0)
 			(effects
 				(font
 					(size 1.27 1.27)
 				)
+				(justify left)
 			)
 		)
@@
 		)
 		(property "Value" "GND"
-			(at 393.7 153.67 0)
+			(at 396.24 149.8599 0)
 			(effects
 				(font
 					(size 1.27 1.27)
 				)
+				(justify left)
 			)
 		)
@@
 		(on_board yes)
 		(dnp no)
-		(property "Reference" "R87"
+		(property "Reference" "R84"
 			(at 279.146 146.812 90)
 			(effects
@@
 			)
 		)
-		(property "Value" "680"
+		(property "Value" "220"
 			(at 279.146 150.876 90)
 			(effects
@@
 			(project "sac_board"
 				(path "/74ff6d0b-648c-43d9-a5b1-cc8d6cd1c1ef/52e20330-efd4-4d59-a57b-f0ea443c9be4"
-					(reference "R87")
+					(reference "R84")
 					(unit 1)
 				)
@@
 		(on_board yes)
 		(dnp no)
-		(property "Reference" "D4"
+		(property "Reference" "D3"
 			(at 356.108 142.24 0)
 			(effects
@@
 			)
 		)
-		(property "Value" "LED"
+		(property "Value" "ORANGE LED"
 			(at 356.108 144.78 0)
 			(effects
@@
 			(project "sac_board"
 				(path "/74ff6d0b-648c-43d9-a5b1-cc8d6cd1c1ef/52e20330-efd4-4d59-a57b-f0ea443c9be4"
-					(reference "D4")
+					(reference "D3")
 					(unit 1)
 				)
@@
 		(on_board yes)
 		(dnp no)
-		(property "Reference" "D5"
+		(property "Reference" "D4"
 			(at 387.858 142.494 0)
 			(effects
@@
 			)
 		)
-		(property "Value" "LED"
+		(property "Value" "ORANGE LED"
 			(at 387.858 145.034 0)
 			(effects
@@
 			(project "sac_board"
 				(path "/74ff6d0b-648c-43d9-a5b1-cc8d6cd1c1ef/52e20330-efd4-4d59-a57b-f0ea443c9be4"
-					(reference "D5")
+					(reference "D4")
 					(unit 1)
 				)
@@
 		)
 		(property "Value" "GND"
-			(at 393.7 167.64 0)
+			(at 396.24 163.8299 0)
 			(effects
 				(font
 					(size 1.27 1.27)
 				)
+				(justify left)
 			)
 		)
@@
 		(on_board yes)
 		(dnp no)
-		(property "Reference" "R86"
+		(property "Reference" "R85"
 			(at 313.436 146.812 90)
 			(effects
@@
 			)
 		)
-		(property "Value" "680"
+		(property "Value" "220"
 			(at 313.436 150.876 90)
 			(effects
@@
 			(project "sac_board"
 				(path "/74ff6d0b-648c-43d9-a5b1-cc8d6cd1c1ef/52e20330-efd4-4d59-a57b-f0ea443c9be4"
-					(reference "R86")
+					(reference "R85")
 					(unit 1)
 				)
@@
 		)
 		(property "Value" "GND"
-			(at 328.93 153.67 0)
+			(at 331.47 149.8599 0)
 			(effects
 				(font
 					(size 1.27 1.27)
 				)
+				(justify left)
 			)
 		)

Commit message: update
Parts:
- added C108: 0.1uF, Capacitor_SMD:C_0603_1608Metric, symbol Device:C_Small
- added J12: Micro_SD_Card_Det1, Connector_Card:microSD_HC_Molex_104031-0811, symbol Connector:Micro_SD_Card_Det1
- added R100, R101, R102, R103, R104, R105, R106: 10K, Resistor_SMD:R_0603_1608Metric, symbol Device:R_Small
- C100, C106, C107, C97, C98: value 100nF -> 0.1uF
- J6: value Conn_ARM_JTAG_SWD_20 -> ARM JTAG/SWD
Connections:
- net +3.3V: now also C108.2, J12.4 (VDD), R100.2, R101.2, R102.2, R103.2, R104.2, R105.2, R106.2
- net GND: now also J4.26 (Pin_26), J4.27 (Pin_27), J4.28 (Pin_28), J4.29 (Pin_29), J4.30 (Pin_30), J4.31 (Pin_31), J4.32 (Pin_32), C108.1, J12.10 (SHIELD), J12.6 (VSS)
- net PA8: now also J4.4 (Pin_4); no longer J4.9 (Pin_9)
- net PB0: now also J4.25 (Pin_25); no longer J4.32 (Pin_32)
- net PB14: now also J4.16 (Pin_16); no longer J4.23 (Pin_23)
- net PB15: now also J4.15 (Pin_15); no longer J4.22 (Pin_22)
- net PB5: now also J4.1 (Pin_1); no longer J4.5 (Pin_5)
- net PC6: now also J4.6 (Pin_6); no longer J4.13 (Pin_13)
- net PC7: now also J4.5 (Pin_5); no longer J4.12 (Pin_12)
- net PD0: now also J4.2 (Pin_2); no longer J4.7 (Pin_7)
- net PD1: now also J4.3 (Pin_3); no longer J4.8 (Pin_8)
- net PD10: now also J4.12 (Pin_12); no longer J4.19 (Pin_19)
- net PD11: now also J4.11 (Pin_11); no longer J4.18 (Pin_18)
- net PD12: now also J4.10 (Pin_10); no longer J4.17 (Pin_17)
- net PD13: now also J4.9 (Pin_9); no longer J4.16 (Pin_16)
- net PD14: now also J4.8 (Pin_8); no longer J4.15 (Pin_15)
- net PD15: now also J4.7 (Pin_7); no longer J4.14 (Pin_14)
- net PD8: now also J4.14 (Pin_14); no longer J4.21 (Pin_21)
- net PD9: now also J4.13 (Pin_13); no longer J4.20 (Pin_20)
- net PE10: now also J4.17 (Pin_17); no longer J4.24 (Pin_24)
- net PE11: now also J4.18 (Pin_18); no longer J4.25 (Pin_25)
- net PE12: now also J4.22 (Pin_22); no longer J4.29 (Pin_29)
- net PE13: now also J4.19 (Pin_19); no longer J4.26 (Pin_26)
- net PE14: now also J4.21 (Pin_21); no longer J4.28 (Pin_28)
- net PE15: now also J4.20 (Pin_20); no longer J4.27 (Pin_27)
- net PE2: now also J7.1 (Pin_1); no longer J7.3 (Pin_3)
- net PE3: now also J7.2 (Pin_2); no longer J7.1 (Pin_1)
- net PE4: now also J7.3 (Pin_3); no longer J7.2 (Pin_2)
- net PE7: now also J4.24 (Pin_24); no longer J4.31 (Pin_31)
- net PE8: now also J4.23 (Pin_23); no longer J4.30 (Pin_30)
- net PC10 renamed PC10-SDIO-D2
- net PC10-SDIO-D2: now also J12.1 (DAT2), R100.1; no longer J4.6 (Pin_6)
- net PC11 renamed PC11-SDIO-D3
- net PC11-SDIO-D3: now also J12.2 (DAT3/CD), R101.1; no longer J4.4 (Pin_4)
- net PC12 renamed PC12-SDIO-CLK
- net PC12-SDIO-CLK: now also J12.5 (CLK), R103.1; no longer J4.3 (Pin_3)
- net PC8 renamed PC8-SDIO-D0
- net PC8-SDIO-D0: now also J12.7 (DAT0), R104.1; no longer J4.11 (Pin_11)
- net PC9 renamed PC9-SDIO-D1
- net PC9-SDIO-D1: now also J12.8 (DAT1), R105.1; no longer J4.10 (Pin_10)
- net PD2 renamed PD2-SDIO-CMD
- net PD2-SDIO-CMD: now also J12.3 (CMD), R102.1; no longer J4.2 (Pin_2)
- net PD3 renamed PD3-Card-CD
- net PD3-Card-CD: now also J12.9 (DET), R106.1; no longer J4.1 (Pin_1)
Other:
- moved on the sheet: C89, C90, J3, R35, R62, R65, Y1
