File: mcu.kicad_sch (KiCad schematic)
At the start: 125 parts, among them J10 Conn_02x04_Odd_Even, J11 Conn_02x04_Odd_Even, J12 Micro_SD_Card_Det1, J2 RJ45_Hanrun_HR911105A_Horizon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, J3 USB_B_Mini, J4 Conn_02x16_Odd_Even, J5 DE9_Pins, J6 ARM JTAG/SWD, J7 Conn_01x08, J8 Conn_02x08_Odd_Even, J9 Conn_02x04_Odd_Even, U11 MAX3232, U12 STM32F407VETx, U13 DP83848C, Y1 8MHz, Y2 32.768KHz, Y3 25MHz

Commit message: update
Parts:
- removed D6: RED LED, LED_SMD:LED_0603_1608Metric, symbol Device:LED
- removed J4: Conn_02x16_Odd_Even, Connector_PinHeader_2.54mm:PinHeader_2x16_P2.54mm_Vertical, symbol Connector_Generic:Conn_02x16_Odd_Even
- removed J7: Conn_01x08, Connector_PinHeader_2.54mm:PinHeader_1x08_P2.54mm_Vertical, symbol Connector_Generic:Conn_01x08
- removed R54, R58, R59, R69, R73, R75: 2.2K, Resistor_SMD:R_0603_1608Metric, symbol Device:R_Small
- removed R55, R56, R57, R61, R64, R68, R70, R72: 33R, Resistor_SMD:R_0603_1608Metric, symbol Device:R_Small
- removed R60: 1.5K, Resistor_SMD:R_0603_1608Metric, symbol Device:R_Small
- removed R63, R67, R78, R79: 0R, Resistor_SMD:R_0603_1608Metric, symbol Device:R_Small
- removed R76: 4.87K, Resistor_SMD:R_0603_1608Metric, symbol Device:R_Small
- removed R77: DNI, Resistor_SMD:R_0603_1608Metric, symbol Device:R_Small
- removed R89: 220, Resistor_SMD:R_0603_1608Metric, symbol Device:R_Small
- removed U13: DP83848C, Package_QFP:LQFP-48_7x7mm_P0.5mm, symbol Interface_Ethernet:DP83848C
- added C109, C110, C111: 10pF, Capacitor_SMD:C_0603_1608Metric, symbol Device:C_Small
- added C112, C113: 0.1uF, Capacitor_SMD:C_0603_1608Metric, symbol Device:C_Small
- added J4: Conn_02x10_Odd_Even, Connector_PinHeader_2.54mm:PinHeader_2x10_P2.54mm_Vertical, symbol Connector_Generic:Conn_02x10_Odd_Even
- added J7: Conn_02x08_Odd_Even, Connector_PinHeader_2.54mm:PinHeader_2x08_P2.54mm_Vertical, symbol Connector_Generic:Conn_02x08_Odd_Even
- added U14: LAN8742A, Package_DFN_QFN:VQFN-24-1EP_4x4mm_P0.5mm_EP2.5x2.5mm, symbol Interface_Ethernet:LAN8742A
- C100, C106: value 0.1uF -> 22nF
- C101, C96: value 33pF -> 22pF
- C107: value 0.1uF -> 10pF
- C99: value 10uF -> 0.1uF
- J12: value Micro_SD_Card_Det1 -> Micro_SD
- J2: value RJ45_Hanrun_HR911105A_Horizontal -> RJ45
- J5: value DE9_Pins -> UART
- R49, R50: value 470R -> 1K
- R51: value 33R -> 12.1K
- R52: value 33R -> 510
- R53: value 2.2K -> 1M
- R66, R71: value 2.2K -> 10K
- renumbered SW5 to SW2, SW4 to SW3, SW3 to SW4, SW2 to SW5
Connections:
- net +3.3V: now also C100.2, C97.2, C98.2, C99.2, U14.1 (VDD2A), U14.19 (VDD1A), U14.9 (VDDIO); no longer C107.2, R49.2, R50.2, R66.2, R71.2
- net GND: now also R49.1, R50.1, R51.2, R66.2, R71.2, C109.1, C110.1, C111.1, C112.2, C113.2, U14.25 (VSS); no longer J9.8 (Pin_8), R53.1
- net PA0: now also J9.1 (Pin_1); no longer J9.3 (Pin_3)
- net PA1-RMII-REF-CLK: now also U14.14 (~{INT}/REFCLKO)
- net PA2-ETH-MDIO: now also R52.1
- net PA3: now also J9.2 (Pin_2); no longer J9.4 (Pin_4)
- net PA4: now also J9.3 (Pin_3); no longer J9.1 (Pin_1)
- net PA5: now also J9.4 (Pin_4); no longer J9.2 (Pin_2)
- net PA7-RMII-CRS-DV: now also U14.11 (CRS_DV/MODE2)
- net PA8: now also C105.2, R83.1, SW2.1
- net PB0: now also J9.6 (Pin_6)
- net PB11-RMII-TXEN: now also U14.16 (TXEN)
- net PB12-RMII-TXD0: now also U14.17 (TXD0); no longer R51.1
- net PB13-RMII-TXD1: now also U14.18 (TXD1); no longer R52.1
- net PB5: now also J7.1 (Pin_1)
- net PB6: now also J7.4 (Pin_4); no longer R84.2
- net PB7: now also J7.3 (Pin_3); no longer R85.2
- net PB8: now also J7.6 (Pin_6); no longer R86.2
- net PB9: now also J7.5 (Pin_5); no longer R87.2
- net PC0-ETH-RESET: now also U14.15 (~{RST})
- net PC1-ETH-MDC: now also U14.13 (MDC)
- net PC13: now also J7.13 (Pin_13)
- net PC2: now also J7.16 (Pin_16)
- net PC3: now also J7.15 (Pin_15)
- net PC4-RMII-RXD0: now also U14.8 (RXD0/MODE0)
- net PC5-RMII-RXD1: now also U14.7 (RXD1/MODE1)
- net PC7: now also C104.2, R82.1, SW3.1
- net PD0: now also R87.2
- net PD1: now also R88.2
- net PD10: now also C103.2, R81.1, SW4.1
- net PD4: now also R86.2; no longer C102.2, R80.1, SW5.1
- net PD5: now also R85.2; no longer C103.2, R81.1, SW4.1
- net PD6: now also R84.2; no longer C104.2, R82.1, SW3.1
- net PD7: now also J7.2 (Pin_2); no longer C105.2, R83.1, SW2.1
- net PE0: now also J7.8 (Pin_8); no longer R88.2
- net PE1: now also J7.7 (Pin_7)
- net PE10: now also C102.2, R80.1, SW5.1
- net PE2: now also J7.10 (Pin_10)
- net PE3: now also J7.9 (Pin_9)
- net PE4: now also J7.12 (Pin_12)
- net PE5: now also J7.11 (Pin_11)
- net PE6: now also J7.14 (Pin_14)
- net PE7: now also J9.8 (Pin_8)
- net PE9: no longer J9.6 (Pin_6)
- net RD-N: now also C111.2, U14.22 (RXN)
- net RD-P: now also C110.2, U14.23 (RXP)
- net TD-N: now also C109.2, U14.20 (TXN)
- net TD-P: now also C107.2, U14.21 (TXP)
- net at R53.2: now also C96.2, Y3.2, U14.5 (XTAL1/CLKIN)
- net at R52.2: now also U14.12 (MDIO)
- net at C101.2, Y3.1: now also R53.1, U14.4 (XTAL2)
- net LED-SPEED: now reaches J2.9
- net LED-SPEED: now also R71.1, U14.2 (LED2/~{INTSEL}); no longer R50.1
- net LED-LINK: now reaches J2.12
- net LED-LINK: now also R66.1, U14.3 (LED1/REGOFF); no longer R49.1
- net LEDACT: no longer names the net of J2.10
- net LEDACT: now also R50.2; no longer R71.1
- net LEDLINK: no longer names the net of J2.11
- net LEDLINK: now also R49.2; no longer R66.1
- new net: C112.1, C113.1, U14.6 (VDDCR)
- new net: R51.1, U14.24 (RBIAS)
- no-connect marks 23 -> 17
Other:
- moved on the sheet: C101, C106, C95, C96, D5, J2, R45, R46, R47, R48, R66, R71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

Commit message: update
Parts:
- removed J12: Micro_SD, Connector_Card:microSD_HC_Molex_104031-0811, symbol Connector:Micro_SD_Card_Det1
- added J12: Micro_SD_Card_TF_01A, Connector_Card:microSD_HC_Hirose_DM3AT-SF-PEJM5, symbol Connector:Micro_SD_CARD_TF01A
- C112: value 0.1uF -> 10uF
- J5: footprint Connector_Dsub:DSUB-9_Pins_Horizontal_P2.77x2.84mm_EdgePinOffset4.94mm_Housed_MountingHolesOffset4.94mm -> Connector_Dsub:DSUB-9_Pins_Horizontal_P2.77x2.84mm_EdgePinOffset7.70mm_Housed_MountingHolesOffset9.12mm
Connections:
- net PB10-RMII-RX-ER is gone; now on net PB10: U12.47 (PB10)
- net +3.3V: now also J12.4 (VDD)
- net GND: now also J4.19 (Pin_19), J4.20 (Pin_20), J12.10 (MP1), J12.6 (VSS)
- net PA8: now also J4.1 (Pin_1); no longer C105.2, R83.1, SW2.1
- net PB14: now also J4.13 (Pin_13)
- net PB15: now also J4.12 (Pin_12)
- net PC10-SDIO-D2: now also J12.1 (DAT2)
- net PC11-SDIO-D3: now also J12.2 (DAT3/CD)
- net PC12-SDIO-CLK: now also J12.5 (CLK)
- net PC6: now also J4.3 (Pin_3)
- net PC7: now also J4.2 (Pin_2); no longer C104.2, R82.1, SW3.1
- net PC8-SDIO-D0: now also J12.7 (DAT0)
- net PC9-SDIO-D1: now also J12.8 (DAT1)
- net PD10: now also J4.9 (Pin_9); no longer C103.2, R81.1, SW4.1
- net PD11: now also J4.8 (Pin_8)
- net PD12: now also J4.7 (Pin_7)
- net PD13: now also J4.6 (Pin_6)
- net PD14: now also J4.5 (Pin_5)
- net PD15: now also J4.4 (Pin_4)
- net PD2-SDIO-CMD: now also J12.3 (CMD)
- net PD3-Card-CD: now also J12.9 (CD1)
- net PD8: now also J4.11 (Pin_11)
- net PD9: now also J4.10 (Pin_10)
- net PE10: now also C103.2, R81.1, SW4.1; no longer C102.2, R80.1, SW5.1
- net PE11: now also C102.2, R80.1, SW5.1
- net PE12: now also J4.18 (Pin_18)
- net PE13: now also J4.17 (Pin_17)
- net PE14: now also J4.16 (Pin_16)
- net PE15: now also J4.15 (Pin_15)
- net PE8: now also C105.2, R83.1, SW2.1
- net PE9: now also C104.2, R82.1, SW3.1
- net PB10: now reaches J4.14 (Pin_14)
Other:
- moved on the sheet: C100, C101, C106, C107, C108, C109, C110, C111, C112, C113, C95, C96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

Commit message: update
Parts:
- H1, H2, H3, H4: footprint MountingHole:MountingHole_2.2mm_M2 -> MountingHole:MountingHole_2.5mm
Changed lines of the file:
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@@
 			)
 		)
-		(property "Footprint" "MountingHole:MountingHole_2.2mm_M2"
+		(property "Footprint" "MountingHole:MountingHole_2.5mm"
 			(at 375.92 100.33 0)
 			(effects
@@
 			)
 		)
-		(property "Footprint" "MountingHole:MountingHole_2.2mm_M2"
+		(property "Footprint" "MountingHole:MountingHole_2.5mm"
 			(at 375.92 87.63 0)
 			(effects
@@
 			)
 		)
-		(property "Footprint" "MountingHole:MountingHole_2.2mm_M2"
+		(property "Footprint" "MountingHole:MountingHole_2.5mm"
 			(at 375.92 93.98 0)
 			(effects
@@
 			)
 		)
-		(property "Footprint" "MountingHole:MountingHole_2.2mm_M2"
+		(property "Footprint" "MountingHole:MountingHole_2.5mm"
 			(at 375.92 106.68 0)
 			(effects

Commit message: update
Parts:
- U11: footprint Package_SO:SOIC-16W_5.3x10.2mm_P1.27mm -> Package_SO:SOIC-16_4.55x10.3mm_P1.27mm
Changed lines of the file:
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@@
 			)
 		)
-		(property "Footprint" "Package_SO:SOIC-16W_5.3x10.2mm_P1.27mm"
+		(property "Footprint" "Package_SO:SOIC-16_4.55x10.3mm_P1.27mm"
 			(at 215.9 83.82 0)
 			(effects

Commit message: update
Parts:
- removed C102: 0.1uF, Capacitor_SMD:C_0603_1608Metric, symbol Device:C_Small
- removed D4: ORANGE LED, LED_SMD:LED_0603_1608Metric, symbol Device:LED
- removed D5: RED LED, LED_SMD:LED_0603_1608Metric, symbol Device:LED
- removed J12: Micro_SD_Card_TF_01A, Connector_Card:microSD_HC_Hirose_DM3AT-SF-PEJM5, symbol Connector:Micro_SD_CARD_TF01A
- removed J5: UART, Connector_Dsub:DSUB-9_Pins_Horizontal_P2.77x2.84mm_EdgePinOffset7.70mm_Housed_MountingHolesOffset9.12mm, symbol Connector:DE9_Pins
- removed J7: Conn_02x08_Odd_Even, Connector_PinHeader_2.54mm:PinHeader_2x08_P2.54mm_Vertical, symbol Connector_Generic:Conn_02x08_Odd_Even
- removed J9: Conn_02x04_Odd_Even, Connector_PinHeader_2.54mm:PinHeader_2x04_P2.54mm_Vertical, symbol Connector_Generic:Conn_02x04_Odd_Even
- removed R80: 10K, Resistor_SMD:R_0603_1608Metric, symbol Device:R_Small
- removed R87, R88: 220, Resistor_SMD:R_0603_1608Metric, symbol Device:R_Small
- removed SW5: ~, Button_Switch_SMD:SW_Push_1P1T_NO_CK_KSC7xxJ, symbol Switch:SW_Push
- added J10: Conn_02x12_Odd_Even, Connector_PinHeader_2.54mm:PinHeader_2x12_P2.54mm_Vertical, symbol Connector_Generic:Conn_02x12_Odd_Even
- added J3: Micro_SD_Card_Det1, Connector_Card:microSD_HC_Hirose_DM3AT-SF-PEJM5, symbol Connector:Micro_SD_Card_Det1
- added J5: DE9_Socket, Custom:DSUB-9_Pins_Horizontal_P2.77x2.84mm_EdgePinOffset7.70mm_Housed_MountingHolesOffset9.12mm_Female, symbol Connector:DE9_Socket
- renumbered C113 to C100, C97 to C101, C98 to C102, C107 to C103, C109 to C104, C110 to C105, C103 to C106, C111 to C107, C100 to C108, C106 to C109, C104 to C110, C95 to C111, C105 to C112, C89 to C83, C90 to C84, C108 to C85, C84 to C86, C91 to C87, C92 to C88, C93 to C89, C94 to C90, C85 to C91, C96 to C92, C101 to C93, C99 to C94, C83 to C95, C112 to C96, C86 to C97, C87 to C98, C88 to C99, D1 to D3, D2 to D4, D3 to D5, J10 to J11, J3 to J2, J6 to J4, J8 to J6, J11 to J7, J4 to J8, J2 to J9, R32 to R33, R33 to R34, R62 to R36, R65 to R37, R31 to R38, R34 to R39, R106 to R40, R105 to R41, R104 to R42, R103 to R43, R102 to R44, R101 to R45, R100 to R46, R44 to R47, R37 to R48, R36 to R49, R38 to R50, R74 to R51, R39 to R54, R43 to R55, R40 to R56, R41 to R57, R42 to R58, R51 to R59, R66 to R60, R71 to R61, R84 to R62, R81 to R63, R45 to R64, R46 to R65, R47 to R66, R48 to R67, R82 to R68, R85 to R69, R86 to R70, R83 to R71, R50 to R72, R49 to R73, SW4 to SW2, SW2 to SW4, U12 to U11, U11 to U12, U14 to U13
Connections:
- net +3.3V: now also J3.4 (VDD)
- net GND: now also J3.10 (SHIELD), J3.6 (VSS), J5.5
- net PA0: now also J10.1 (Pin_1)
- net PA3: now also J10.2 (Pin_2)
- net PA4: now also J10.3 (Pin_3)
- net PA5: now also J10.4 (Pin_4)
- net PA6: now also J10.5 (Pin_5)
- net PB0: now also J10.6 (Pin_6)
- net PB1: now also J10.7 (Pin_7)
- net PB5: now also J10.9 (Pin_9)
- net PB6: now also J10.12 (Pin_12)
- net PB7: now also J10.11 (Pin_11)
- net PB8: now also J10.14 (Pin_14)
- net PB9: now also J10.13 (Pin_13)
- net PC10-SDIO-D2: now also J3.1 (DAT2)
- net PC11-SDIO-D3: now also J3.2 (DAT3/CD)
- net PC12-SDIO-CLK: now also J3.5 (CLK)
- net PC13: now also J10.21 (Pin_21)
- net PC2: now also J10.24 (Pin_24)
- net PC3: now also J10.23 (Pin_23)
- net PC8-SDIO-D0: now also J3.7 (DAT0)
- net PC9-SDIO-D1: now also J3.8 (DAT1)
- net PD2-SDIO-CMD: now also J3.3 (CMD)
- net PD3-Card-CD: now also J3.9 (DET)
- net PD7: now also J10.10 (Pin_10)
- net PE0: now also J10.16 (Pin_16)
- net PE1: now also J10.15 (Pin_15)
- net PE2: now also J10.18 (Pin_18)
- net PE3: now also J10.17 (Pin_17)
- net PE4: now also J10.20 (Pin_20)
- net PE5: now also J10.19 (Pin_19)
- net PE6: now also J10.22 (Pin_22)
- net PE7: now also J10.8 (Pin_8)
- net at U12.7 (T2OUT): now also J5.2
- net at U12.8 (R2IN): now also J5.3
- no-connect marks 17 -> 16
Other:
- moved on the sheet: C106, C110, C112, C85, D3, D4, D5, J2, J7, R36, R37, R40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

Commit message: update
Parts:
- removed J10: Conn_02x12_Odd_Even, Connector_PinHeader_2.54mm:PinHeader_2x12_P2.54mm_Vertical, symbol Connector_Generic:Conn_02x12_Odd_Even
- removed J8: Conn_02x10_Odd_Even, Connector_PinHeader_2.54mm:PinHeader_2x10_P2.54mm_Vertical, symbol Connector_Generic:Conn_02x10_Odd_Even
- added C113: 0.1uF, Capacitor_SMD:C_0603_1608Metric, symbol Device:C_Small
- added D6: ORANGE LED, LED_SMD:LED_0603_1608Metric, symbol Device:LED
- added J10: Conn_02x09_Odd_Even, Connector_PinHeader_2.54mm:PinHeader_2x09_P2.54mm_Vertical, symbol Connector_Generic:Conn_02x09_Odd_Even
- added J8: Conn_02x14_Odd_Even, Connector_PinHeader_2.54mm:PinHeader_2x14_P2.54mm_Vertical, symbol Connector_Generic:Conn_02x14_Odd_Even
- added R74: 220, Resistor_SMD:R_0603_1608Metric, symbol Device:R_Small
- added R75: 10K, Resistor_SMD:R_0603_1608Metric, symbol Device:R_Small
- added SW5: ~, Button_Switch_SMD:SW_Push_1P1T_NO_CK_KSC7xxJ, symbol Switch:SW_Push
Connections:
- net +3.3V: now also R75.2
- net GND: now also C113.1, D6.1 (K), J8.26 (Pin_26), J8.27 (Pin_27), J8.28 (Pin_28), SW5.2
- net PA0: now also J10.18 (Pin_18)
- net PA3: now also C110.2, R68.1, SW3.1
- net PA4: now also C106.2, R63.1, SW2.1
- net PA5: now also C112.2, R71.1, SW4.1
- net PA6: now also C113.2, R75.1, SW5.1
- net PA8: now also J8.2 (Pin_2)
- net PB0: now also J8.25 (Pin_25)
- net PB1: now also J8.23 (Pin_23)
- net PB10: now also J8.13 (Pin_13)
- net PB14: now also J8.14 (Pin_14)
- net PB15: now also J8.11 (Pin_11)
- net PB5: now also J10.3 (Pin_3)
- net PB6: now also J10.4 (Pin_4)
- net PB7: now also J10.5 (Pin_5)
- net PB8: now also J10.6 (Pin_6)
- net PB9: now also J10.7 (Pin_7)
- net PC13: now also J10.15 (Pin_15)
- net PC2: now also J10.16 (Pin_16)
- net PC3: now also J10.17 (Pin_17)
- net PC6: now also J8.4 (Pin_4)
- net PC7: now also J8.1 (Pin_1)
- net PD0: now also R62.2
- net PD1: now also R69.2
- net PD10: now also J8.10 (Pin_10)
- net PD11: now also J8.7 (Pin_7)
- net PD12: now also J8.8 (Pin_8)
- net PD13: now also J8.5 (Pin_5)
- net PD14: now also J8.6 (Pin_6)
- net PD15: now also J8.3 (Pin_3)
- net PD5: now also R74.2; no longer R69.2
- net PD6: now also J10.1 (Pin_1); no longer R62.2
- net PD7: now also J10.2 (Pin_2)
- net PD8: now also J8.12 (Pin_12)
- net PD9: now also J8.9 (Pin_9)
- net PE0: now also J10.8 (Pin_8)
- net PE1: now also J10.9 (Pin_9)
- net PE10: now also J8.19 (Pin_19); no longer C106.2, R63.1, SW2.1
- net PE11: now also J8.20 (Pin_20)
- net PE12: now also J8.17 (Pin_17)
- net PE13: now also J8.18 (Pin_18)
- net PE14: now also J8.15 (Pin_15)
- net PE15: now also J8.16 (Pin_16)
- net PE2: now also J10.10 (Pin_10)
- net PE3: now also J10.11 (Pin_11)
- net PE4: now also J10.12 (Pin_12)
- net PE5: now also J10.13 (Pin_13)
- net PE6: now also J10.14 (Pin_14)
- net PE7: now also J8.24 (Pin_24)
- net PE8: now also J8.21 (Pin_21); no longer C112.2, R71.1, SW4.1
- net PE9: now also J8.22 (Pin_22); no longer C110.2, R68.1, SW3.1
- new net: D6.2 (A), R74.1
Other:
- moved on the sheet: C106, C110, C112, D3, D4, D5, R62, R63, R68, R69, R70, R71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

Commit message: update
Parts:
- C83, C84, C86, C87, C88, C89, C90, C91, C95, C97, C98, C99: footprint Capacitor_SMD:C_0603_1608Metric -> Capacitor_SMD:C_0805_2012Metric
- R33, R34, R35, R36, R37, R38, R39, R47, R54, R55, R56, R57, R58: footprint Resistor_SMD:R_0603_1608Metric -> Resistor_SMD:R_0805_2012Metric
Changed lines of the file:
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@@
 			)
 		)
-		(property "Footprint" "Resistor_SMD:R_0603_1608Metric"
+		(property "Footprint" "Resistor_SMD:R_0805_2012Metric"
 			(at 39.37 66.04 0)
 			(effects
@@
 			)
 		)
-		(property "Footprint" "Capacitor_SMD:C_0603_1608Metric"
+		(property "Footprint" "Capacitor_SMD:C_0805_2012Metric"
 			(at 240.03 38.1 0)
 			(effects
@@
 			)
 		)
-		(property "Footprint" "Resistor_SMD:R_0603_1608Metric"
+		(property "Footprint" "Resistor_SMD:R_0805_2012Metric"
 			(at 124.46 172.72 0)
 			(effects
@@
 			)
 		)
-		(property "Footprint" "Capacitor_SMD:C_0603_1608Metric"
+		(property "Footprint" "Capacitor_SMD:C_0805_2012Metric"
 			(at 241.3 46.99 0)
 			(effects
@@
 			)
 		)
-		(property "Footprint" "Capacitor_SMD:C_0603_1608Metric"
+		(property "Footprint" "Capacitor_SMD:C_0805_2012Metric"
 			(at 229.87 25.4 0)
 			(effects
@@
 			)
 		)
-		(property "Footprint" "Resistor_SMD:R_0603_1608Metric"
+		(property "Footprint" "Resistor_SMD:R_0805_2012Metric"
 			(at 46.99 191.77 0)
 			(effects
@@
 			)
 		)
-		(property "Footprint" "Resistor_SMD:R_0603_1608Metric"
+		(property "Footprint" "Resistor_SMD:R_0805_2012Metric"
 			(at 39.37 48.26 0)
 			(effects
@@
 			)
 		)
-		(property "Footprint" "Resistor_SMD:R_0603_1608Metric"
+		(property "Footprint" "Resistor_SMD:R_0805_2012Metric"
 			(at 229.87 139.7 0)
 			(effects
@@
 			)
 		)
-		(property "Footprint" "Resistor_SMD:R_0603_1608Metric"
+		(property "Footprint" "Resistor_SMD:R_0805_2012Metric"
 			(at 232.41 105.41 0)
 			(effects
@@
 			)
 		)
-		(property "Footprint" "Resistor_SMD:R_0603_1608Metric"
+		(property "Footprint" "Resistor_SMD:R_0805_2012Metric"
 			(at 46.99 194.31 0)
 			(effects
@@
 			)
 		)
-		(property "Footprint" "Capacitor_SMD:C_0603_1608Metric"
+		(property "Footprint" "Capacitor_SMD:C_0805_2012Metric"
 			(at 52.07 27.94 0)
 			(effects
@@
 			)
 		)
-		(property "Footprint" "Resistor_SMD:R_0603_1608Metric"
+		(property "Footprint" "Resistor_SMD:R_0805_2012Metric"
 			(at 234.95 105.41 0)
 			(effects
@@
 			)
 		)
-		(property "Footprint" "Capacitor_SMD:C_0603_1608Metric"
+		(property "Footprint" "Capacitor_SMD:C_0805_2012Metric"
 			(at 25.4 74.93 0)
 			(effects
@@
 			)
 		)
-		(property "Footprint" "Resistor_SMD:R_0603_1608Metric"
+		(property "Footprint" "Resistor_SMD:R_0805_2012Metric"
 			(at 229.87 105.41 0)
 			(effects
@@
 			)
 		)
-		(property "Footprint" "Resistor_SMD:R_0603_1608Metric"
+		(property "Footprint" "Resistor_SMD:R_0805_2012Metric"
 			(at 237.49 105.41 0)
 			(effects
@@
 			)
 		)
-		(property "Footprint" "Resistor_SMD:R_0603_1608Metric"
+		(property "Footprint" "Resistor_SMD:R_0805_2012Metric"
 			(at 58.42 48.26 0)
 			(effects
@@
 			)
 		)
-		(property "Footprint" "Resistor_SMD:R_0603_1608Metric"
+		(property "Footprint" "Resistor_SMD:R_0805_2012Metric"
 			(at 39.37 41.91 0)
 			(effects
@@
 			)
 		)
-		(property "Footprint" "Capacitor_SMD:C_0603_1608Metric"
+		(property "Footprint" "Capacitor_SMD:C_0805_2012Metric"
 			(at 62.23 152.4 0)
 			(effects
@@
 			)
 		)
-		(property "Footprint" "Capacitor_SMD:C_0603_1608Metric"
+		(property "Footprint" "Capacitor_SMD:C_0805_2012Metric"
 			(at 25.4 58.42 0)
 			(effects
@@
 			)
 		)
-		(property "Footprint" "Capacitor_SMD:C_0603_1608Metric"
+		(property "Footprint" "Capacitor_SMD:C_0805_2012Metric"
 			(at 137.16 181.61 0)
 			(effects
@@
 			)
 		)
-		(property "Footprint" "Capacitor_SMD:C_0603_1608Metric"
+		(property "Footprint" "Capacitor_SMD:C_0805_2012Metric"
 			(at 241.3 54.61 0)
 			(effects
@@
 			)
 		)
-		(property "Footprint" "Resistor_SMD:R_0603_1608Metric"
+		(property "Footprint" "Resistor_SMD:R_0805_2012Metric"
 			(at 58.42 21.59 0)
 			(effects
@@
 			)
 		)
-		(property "Footprint" "Capacitor_SMD:C_0603_1608Metric"
+		(property "Footprint" "Capacitor_SMD:C_0805_2012Metric"
 			(at 189.23 38.1 0)
 			(effects
@@
 			)
 		)
-		(property "Footprint" "Capacitor_SMD:C_0603_1608Metric"
+		(property "Footprint" "Capacitor_SMD:C_0805_2012Metric"
 			(at 62.23 157.48 0)
 			(effects
@@
 			)
 		)
-		(property "Footprint" "Capacitor_SMD:C_0603_1608Metric"
+		(property "Footprint" "Capacitor_SMD:C_0805_2012Metric"
 			(at 137.16 165.1 0)
 			(effects

Commit message: update
Parts:
- C100, C101, C102, C103, C104, C105, C106, C107, C108, C109, C110, C111, C112, C113, C85, C92, C93, C94, C96: footprint Capacitor_SMD:C_0603_1608Metric -> Capacitor_SMD:C_0805_2012Metric
- D3, D4, D5, D6: footprint LED_SMD:LED_0603_1608Metric -> LED_SMD:LED_0805_2012Metric
- R40, R41, R42, R43, R44, R45, R46, R48, R49, R50, R51, R52, R53, R59, R60, R61, R62, R63, R64, R65, R66, R67, R68, R69, R70, R71, R72, R73, R74, R75: footprint Resistor_SMD:R_0603_1608Metric -> Resistor_SMD:R_0805_2012Metric
