File: mcu.kicad_sch (KiCad schematic)
At the start: 104 parts, among them J10 Conn_02x09_Odd_Even, J11 Conn_02x04_Odd_Even, J2 USB_B_Mini, J3 Micro_SD_Card_Det1, J4 ARM JTAG/SWD, J5 DE9_Socket, J6 Conn_02x08_Odd_Even, J7 Conn_02x04_Odd_Even, J8 Conn_02x14_Odd_Even, J9 RJ45, U11 STM32F407VETx, U12 MAX3232, U13 LAN8742A, Y1 8MHz, Y2 32.768KHz, Y3 25MHz

Commit message: update
Parts:
- H1, H2, H3, H4: footprint MountingHole:MountingHole_2.5mm -> MountingHole:MountingHole_2.7mm_M2.5
Changed lines of the file:
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@@
 			)
 		)
-		(property "Footprint" "MountingHole:MountingHole_2.5mm"
+		(property "Footprint" "MountingHole:MountingHole_2.7mm_M2.5"
 			(at 375.92 100.33 0)
 			(effects
@@
 			)
 		)
-		(property "Footprint" "MountingHole:MountingHole_2.5mm"
+		(property "Footprint" "MountingHole:MountingHole_2.7mm_M2.5"
 			(at 375.92 87.63 0)
 			(effects
@@
 			)
 		)
-		(property "Footprint" "MountingHole:MountingHole_2.5mm"
+		(property "Footprint" "MountingHole:MountingHole_2.7mm_M2.5"
 			(at 375.92 93.98 0)
 			(effects
@@
 			)
 		)
-		(property "Footprint" "MountingHole:MountingHole_2.5mm"
+		(property "Footprint" "MountingHole:MountingHole_2.7mm_M2.5"
 			(at 375.92 106.68 0)
 			(effects

Commit message: update
Parts:
- removed J11, J7: Conn_02x04_Odd_Even, Connector_PinHeader_2.54mm:PinHeader_2x04_P2.54mm_Vertical, symbol Connector_Generic:Conn_02x04_Odd_Even
- removed J6: Conn_02x08_Odd_Even, Connector_PinHeader_2.54mm:PinHeader_2x08_P2.54mm_Vertical, symbol Connector_Generic:Conn_02x08_Odd_Even
- added J6: Conn_02x16_Odd_Even, Connector_PinHeader_2.54mm:PinHeader_2x16_P2.54mm_Vertical, symbol Connector_Generic:Conn_02x16_Odd_Even
- renumbered J10 to J7
Connections:
- net +3.3V: now also J6.18 (Pin_18), J6.20 (Pin_20), J6.22 (Pin_22), J6.24 (Pin_24)
- net +5V: now also J6.26 (Pin_26), J6.28 (Pin_28), J6.30 (Pin_30), J6.32 (Pin_32)
- net GND: now also J6.1 (Pin_1), J6.11 (Pin_11), J6.13 (Pin_13), J6.15 (Pin_15), J6.17 (Pin_17), J6.19 (Pin_19), J6.21 (Pin_21), J6.23 (Pin_23), J6.25 (Pin_25), J6.27 (Pin_27), J6.29 (Pin_29), J6.3 (Pin_3), J6.31 (Pin_31), J6.5 (Pin_5), J6.7 (Pin_7), J6.9 (Pin_9)
- net V_M1: now also J6.2 (Pin_2)
- net V_M2: now also J6.4 (Pin_4)
- net V_M3: now also J6.6 (Pin_6)
- net V_M4: now also J6.8 (Pin_8)
- net V_M5: now also J6.10 (Pin_10)
- net V_M6: now also J6.12 (Pin_12)
- net V_M7: now also J6.14 (Pin_14)
- net V_M8: now also J6.16 (Pin_16)
Other:
- moved on the sheet: J8

Commit message: update
Parts:
- added C114, C115, C116, C117, C118: 0.1uF, Capacitor_SMD:C_0805_2012Metric, symbol Device:C_Small
Connections:
- net +3.3V: now also C114.2, C115.2, C116.2, C117.2, C118.2
- net GND: now also C114.1, C115.1, C116.1, C117.1, C118.1
Other:
- note added: "CONNECTOR & MountingHole"
- note added: "Decoupling capacitors are connected to pins: 11, 19, 28, 50, 75, 100."
- note added: "ETHERNET"
- note added: "JTAG"
- note added: "LED & BUTTON"
- note added: "MCU"
- note added: "SDIO"
- note added: "USART1"
- note added: "USB"
- moved on the sheet: C100, C101, C102, C103, C104, C105, C106, C107, C108, C109, C110, C111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

Commit message: update
Parts:
- added C119: 0.1uF, Capacitor_SMD:C_0805_2012Metric, symbol Device:C_Small
Connections:
- net +3.3V: now also C119.2
- net GND: now also C119.1
Other:
- moved on the sheet: C108, C109
Changed lines of the file:
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@@
 	)
 	(junction
+		(at 148.59 25.4)
+		(diameter 0)
+		(color 0 0 0 0)
+	)
+	(junction
 		(at 215.9 139.7)
 		(diameter 0)
@@
 	(wire
 		(pts
-			(xy 334.01 204.47) (xy 334.01 199.39)
+			(xy 334.01 203.2) (xy 334.01 199.39)
 		)
 		(stroke
@@
 	(wire
 		(pts
+			(xy 154.94 36.83) (xy 148.59 36.83)
+		)
+		(stroke
+			(width 0)
+			(type default)
+		)
+	)
+	(wire
+		(pts
 			(xy 317.5 219.71) (xy 339.09 219.71)
 		)
@@
 	(wire
 		(pts
+			(xy 154.94 27.94) (xy 154.94 25.4)
+		)
+		(stroke
+			(width 0)
+			(type default)
+		)
+	)
+	(wire
+		(pts
 			(xy 332.74 27.94) (xy 336.55 27.94)
 		)
@@
 	(wire
 		(pts
-			(xy 330.2 204.47) (xy 330.2 199.39)
+			(xy 330.2 203.2) (xy 330.2 199.39)
 		)
 		(stroke
@@
 	(wire
 		(pts
+			(xy 154.94 33.02) (xy 154.94 36.83)
+		)
+		(stroke
+			(width 0)
+			(type default)
+		)
+	)
+	(wire
+		(pts
 			(xy 199.39 46.99) (xy 194.31 46.99)
 		)
@@
 	(wire
 		(pts
-			(xy 334.01 210.82) (xy 334.01 209.55)
+			(xy 334.01 210.82) (xy 334.01 208.28)
 		)
 		(stroke
@@
 	(wire
 		(pts
-			(xy 330.2 209.55) (xy 330.2 210.82)
+			(xy 330.2 208.28) (xy 330.2 210.82)
 		)
 		(stroke
@@
 	(wire
 		(pts
+			(xy 154.94 25.4) (xy 148.59 25.4)
+		)
+		(stroke
+			(width 0)
+			(type default)
+		)
+	)
+	(wire
+		(pts
 			(xy 130.81 165.1) (xy 134.62 165.1)
 		)
@@
 	(symbol
 		(lib_id "Device:C_Small")
+		(at 154.94 30.48 180)
+		(unit 1)
+		(exclude_from_sim no)
+		(in_bom yes)
+		(on_board yes)
+		(dnp no)
+		(property "Reference" "C119"
+			(at 152.146 34.29 90)
+			(effects
+				(font
+					(size 1.27 1.27)
+				)
+			)
+		)
+		(property "Value" "0.1uF"
+			(at 153.924 34.036 90)
+			(effects
+				(font
+					(size 1.27 1.27)
+				)
+			)
+		)
+		(property "Footprint" "Capacitor_SMD:C_0805_2012Metric"
+			(at 154.94 30.48 0)
+			(effects
+				(font
+					(size 1.27 1.27)
+				)
+				(hide yes)
+			)
+		)
+		(property "Datasheet" "~"
+			(at 154.94 30.48 0)
+			(effects
+				(font
+					(size 1.27 1.27)
+				)
+				(hide yes)
+			)
+		)
+		(property "Description" "Unpolarized capacitor, small symbol"
+			(at 154.94 30.48 0)
+			(effects
+				(font
+					(size 1.27 1.27)
+				)
+				(hide yes)
+			)
+		)
+		(property "Sim.Device" ""
+			(at 154.94 30.48 90)
+			(effects
+				(font
+					(size 1.27 1.27)
+				)
+				(hide yes)
+			)
+		)
+		(property "Sim.Pins" ""
+			(at 154.94 30.48 90)
+			(effects
+				(font
+					(size 1.27 1.27)
+				)
+				(hide yes)
+			)
+		)
+		(pin "1"
+		)
+		(pin "2"
+		)
+		(instances
+			(project "sac_board"
+				(path "/74ff6d0b-648c-43d9-a5b1-cc8d6cd1c1ef/52e20330-efd4-4d59-a57b-f0ea443c9be4"
+					(reference "C119")
+					(unit 1)
+				)
+			)
+		)
+	)
+	(symbol
+		(lib_id "Device:C_Small")
 		(at 234.95 30.48 270)
 		(unit 1)
@@
 		)
 		(property "Value" "0.1uF"
-			(at 120.396 34.036 90)
+			(at 120.396 33.528 90)
 			(effects
 				(font
@@
 	(symbol
 		(lib_id "Device:C_Small")
-		(at 334.01 207.01 180)
+		(at 334.01 205.74 180)
 		(unit 1)
 		(exclude_from_sim no)
@@
 		(dnp no)
 		(property "Reference" "C109"
-			(at 332.232 210.058 90)
+			(at 332.994 209.296 90)
 			(effects
 				(font
@@
 		)
 		(property "Value" "22nF"
-			(at 332.74 202.946 90)
+			(at 332.994 202.438 90)
 			(effects
 				(font
@@
 		)
 		(property "Footprint" "Capacitor_SMD:C_0805_2012Metric"
-			(at 334.01 207.01 0)
+			(at 334.01 205.74 0)
 			(effects
 				(font
@@
 		)
 		(property "Datasheet" "~"
-			(at 334.01 207.01 0)
+			(at 334.01 205.74 0)
 			(effects
 				(font
@@
 		)
 		(property "Description" "Unpolarized capacitor, small symbol"
-			(at 334.01 207.01 0)
+			(at 334.01 205.74 0)
 			(effects
 				(font
@@
 		)
 		(property "Sim.Device" ""
-			(at 334.01 207.01 90)
+			(at 334.01 205.74 90)
 			(effects
 				(font
@@
 		)
 		(property "Sim.Pins" ""
-			(at 334.01 207.01 90)
+			(at 334.01 205.74 90)
 			(effects
 				(font
@@
 	(symbol
 		(lib_id "Device:C_Small")
-		(at 330.2 207.01 180)
+		(at 330.2 205.74 180)
 		(unit 1)
 		(exclude_from_sim no)
@@
 		(dnp no)
 		(property "Reference" "C108"
-			(at 328.422 210.058 90)
+			(at 329.184 209.296 90)
 			(effects
 				(font
@@
 		)
 		(property "Value" "22nF"
-			(at 328.93 202.946 90)
+			(at 328.93 202.438 90)
 			(effects
 				(font
@@
 		)
 		(property "Footprint" "Capacitor_SMD:C_0805_2012Metric"
-			(at 330.2 207.01 0)
+			(at 330.2 205.74 0)
 			(effects
 				(font
@@
 		)
 		(property "Datasheet" "~"
-			(at 330.2 207.01 0)
+			(at 330.2 205.74 0)
 			(effects
 				(font
@@
 		)
 		(property "Description" "Unpolarized capacitor, small symbol"
-			(at 330.2 207.01 0)
+			(at 330.2 205.74 0)
 			(effects
 				(font
@@
 		)
 		(property "Sim.Device" ""
-			(at 330.2 207.01 90)
+			(at 330.2 205.74 90)
 			(effects
 				(font
@@
 		)
 		(property "Sim.Pins" ""
-			(at 330.2 207.01 90)
+			(at 330.2 205.74 90)
 			(effects
 				(font

Commit message: update
Parts:
- removed J4: ARM JTAG/SWD, Connector_IDC:IDC-Header_2x10_P2.54mm_Vertical, symbol Connector:Conn_ARM_JTAG_SWD_20
- removed J5: DE9_Socket, Custom:DSUB-9_Pins_Horizontal_P2.77x2.84mm_EdgePinOffset7.70mm_Housed_MountingHolesOffset9.12mm_Female, symbol Connector:DE9_Socket
- removed U12: MAX3232, Package_SO:SOIC-16_4.55x10.3mm_P1.27mm, symbol Interface_UART:MAX3232
- added C120, C121: 10uF, Capacitor_SMD:C_0805_2012Metric, symbol Device:C_Small
- added H5, H6, H7, H8: MountingHole, MountingHole:MountingHole_3mm, symbol Mechanical:MountingHole
- added J5: Conn_02x08_Odd_Even, Connector_PinHeader_2.54mm:PinHeader_2x08_P2.54mm_Vertical, symbol Connector_Generic:Conn_02x08_Odd_Even
- C91, C95, C97, C98, C99: value 0.1uF -> 10uF
- H1, H2, H3, H4: footprint MountingHole:MountingHole_2.7mm_M2.5 -> MountingHole:MountingHole_3mm
Connections:
- net +3.3V: now also C91.2, C97.2, C98.2, C99.2, C120.2, C121.2, J5.14 (Pin_14), J5.2 (Pin_2)
- net GND: now also C91.1, C97.1, C120.1, C121.1, J5.10 (Pin_10), J5.12 (Pin_12), J5.16 (Pin_16), J5.4 (Pin_4), J5.6 (Pin_6), J5.8 (Pin_8)
- net PA10-USART1-RX: now also J5.15 (Pin_15)
- net PA13-JTMS: now also J5.5 (Pin_5)
- net PA14-JTCK: now also J5.9 (Pin_9)
- net PA15-JTDI: now also R57.2, J5.3 (Pin_3); no longer R58.2
- net PA9-USART1-TX: now also J5.13 (Pin_13)
- net PB3-JTDO: now also R54.2, J5.7 (Pin_7); no longer R57.2
- net PB4-JNTRST: now also R58.2, J5.1 (Pin_1); no longer R54.2
- net RESET: now also J5.11 (Pin_11)
- no-connect marks 16 -> 3
Other:
- note added: "CONNECTOR"
- note added: "MOUNTING_HOLE"
- note removed: "CONNECTOR & MountingHole"
- note removed: "JTAG"
- note removed: "USART1"
- moved on the sheet: BT1, C100, C101, C102, C106, C110, C112, C113, C114, C115, C116, C117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

Commit message: update
Parts:
- removed H5, H6, H7, H8: MountingHole, MountingHole:MountingHole_3mm, symbol Mechanical:MountingHole

Commit message: update
Parts:
- H1, H2, H3, H4: footprint MountingHole:MountingHole_3mm -> MountingHole:MountingHole_3.2mm_M3
Changed lines of the file:
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@@
 				)
 				(justify left)
-			)
-		)
-		(property "Footprint" "MountingHole:MountingHole_3mm"
+				(hide yes)
+			)
+		)
+		(property "Footprint" "MountingHole:MountingHole_3.2mm_M3"
 			(at 377.19 53.34 0)
 			(effects
@@
 				)
 				(justify left)
-			)
-		)
-		(property "Footprint" "MountingHole:MountingHole_3mm"
+				(hide yes)
+			)
+		)
+		(property "Footprint" "MountingHole:MountingHole_3.2mm_M3"
 			(at 377.19 40.64 0)
 			(effects
@@
 				)
 				(justify left)
-			)
-		)
-		(property "Footprint" "MountingHole:MountingHole_3mm"
+				(hide yes)
+			)
+		)
+		(property "Footprint" "MountingHole:MountingHole_3.2mm_M3"
 			(at 377.19 46.99 0)
 			(effects
@@
 				)
 				(justify left)
-			)
-		)
-		(property "Footprint" "MountingHole:MountingHole_3mm"
+				(hide yes)
+			)
+		)
+		(property "Footprint" "MountingHole:MountingHole_3.2mm_M3"
 			(at 377.19 59.69 0)
 			(effects
