File: power_mcu.kicad_sch (KiCad schematic)
At the start: 28 parts, among them J1 12V_Input, U1 TPS563201, U2 TPS563201

Commit message: update
Parts:
- C1: renamed from C4; footprint Capacitor_SMD:C_01005_0402Metric_Pad0.57x0.30mm_HandSolder -> Capacitor_SMD:C_0603_1608Metric
- C10: renamed from C14; footprint Capacitor_SMD:C_01005_0402Metric_Pad0.57x0.30mm_HandSolder -> Capacitor_SMD:C_0603_1608Metric
- C11: renamed from C1; footprint Capacitor_SMD:C_01005_0402Metric_Pad0.57x0.30mm_HandSolder -> Capacitor_SMD:C_0603_1608Metric
- C12: renamed from C8; footprint Capacitor_SMD:C_01005_0402Metric_Pad0.57x0.30mm_HandSolder -> Capacitor_SMD:C_0603_1608Metric
- C13: renamed from C2; footprint Capacitor_SMD:C_01005_0402Metric_Pad0.57x0.30mm_HandSolder -> Capacitor_SMD:C_0603_1608Metric
- C14: renamed from C9; footprint Capacitor_SMD:C_01005_0402Metric_Pad0.57x0.30mm_HandSolder -> Capacitor_SMD:C_0603_1608Metric
- C15: renamed from C102; footprint Capacitor_SMD:C_01005_0402Metric_Pad0.57x0.30mm_HandSolder -> Capacitor_SMD:C_0603_1608Metric
- C16: renamed from C103; footprint Capacitor_Tantalum_SMD:CP_EIA-3216-12_Kemet-S_HandSolder -> Capacitor_SMD:C_0603_1608Metric
- C2: renamed from C11; footprint Capacitor_SMD:C_01005_0402Metric_Pad0.57x0.30mm_HandSolder -> Capacitor_SMD:C_0603_1608Metric
- C3: renamed from C5; footprint Capacitor_SMD:C_01005_0402Metric_Pad0.57x0.30mm_HandSolder -> Capacitor_SMD:C_0603_1608Metric
- C4: renamed from C12; footprint Capacitor_SMD:C_01005_0402Metric_Pad0.57x0.30mm_HandSolder -> Capacitor_SMD:C_0603_1608Metric
- C5: renamed from C6; footprint Capacitor_SMD:C_01005_0402Metric_Pad0.57x0.30mm_HandSolder -> Capacitor_SMD:C_0603_1608Metric
- C6: renamed from C13; footprint Capacitor_SMD:C_01005_0402Metric_Pad0.57x0.30mm_HandSolder -> Capacitor_SMD:C_0603_1608Metric
- C7: renamed from C3; footprint Capacitor_SMD:C_01005_0402Metric_Pad0.57x0.30mm_HandSolder -> Capacitor_SMD:C_0603_1608Metric
- C8: renamed from C10; footprint Capacitor_SMD:C_01005_0402Metric_Pad0.57x0.30mm_HandSolder -> Capacitor_SMD:C_0603_1608Metric
- C9: renamed from C7; footprint Capacitor_SMD:C_01005_0402Metric_Pad0.57x0.30mm_HandSolder -> Capacitor_SMD:C_0603_1608Metric
- J1: footprint Connector_BarrelJack:BarrelJack_Wuerth_694108106102_2.5x5.5mm -> Connector_BarrelJack:BarrelJack_CUI_PJ-102AH_Horizontal
- renumbered L15 to L3, R4 to R2, R6 to R4, R2 to R5, R5 to R6

Commit message: update
Parts:
- removed C10: 220uF, Capacitor_SMD:C_0603_1608Metric, symbol Device:C_Small
- removed C2, C6: 22uF, Capacitor_SMD:C_0603_1608Metric, symbol Device:C_Small
- removed C8: 0.1uF, Capacitor_SMD:C_0603_1608Metric, symbol Device:C_Small
- removed L2: 2.2uH, Inductor_SMD:L_0603_1608Metric_Pad1.05x0.95mm_HandSolder, symbol Device:L_Small
- removed R2: 10K, Resistor_SMD:R_0603_1608Metric, symbol Device:R_Small
- added C11, C15: 0.1uF, Capacitor_SMD:C_0603_1608Metric, symbol Device:C_Small
- added C13: 22uF, Capacitor_SMD:C_1206_3216Metric, symbol Device:C_Small
- added C16, C17: 10uF, Capacitor_SMD:C_1206_3216Metric, symbol Device:C_Small
- added C18: 10pF, Capacitor_SMD:C_0603_1608Metric, symbol Device:C_Small
- added L3: 2.2uH, Inductor_SMD:L_6.3x6.3_H3, symbol Device:L_Small
- added R5: 56K, Resistor_SMD:R_0603_1608Metric, symbol Device:R_Small
- C12: footprint Capacitor_SMD:C_0603_1608Metric -> Capacitor_SMD:C_1206_3216Metric
- C14, C4: value 22uF -> 10uF; footprint Capacitor_SMD:C_0603_1608Metric -> Capacitor_SMD:C_1206_3216Metric
- C2: renamed from C11; footprint Capacitor_SMD:C_0603_1608Metric -> Capacitor_SMD:C_1206_3216Metric
- C3: renamed from C13; footprint Capacitor_SMD:C_0603_1608Metric -> Capacitor_SMD:C_1206_3216Metric
- C5: renamed from C1; value 22uF -> 0.1uF
- C6: renamed from C3; value 22uF -> 10uF; footprint Capacitor_SMD:C_0603_1608Metric -> Capacitor_SMD:C_1206_3216Metric
- C7: renamed from C5; value 22uF -> 10uF; footprint Capacitor_SMD:C_0603_1608Metric -> Capacitor_SMD:C_1206_3216Metric
- C8: renamed from C9; value 220uF -> 10pF
- L1: footprint Inductor_SMD:L_0603_1608Metric_Pad1.05x0.95mm_HandSolder -> Inductor_SMD:L_6.3x6.3_H3
- R6: value 56K -> 10K
- renumbered C7 to C1, C16 to C10, C15 to C9, L3 to L2, R5 to R2
Connections:
- net +12V: now also R4.2, C15.1, C16.1, C17.1; no longer C4.1
- net +3.3V: now also C2.1, C3.1, C4.1; no longer C2.2, C3.2
- net +5V: now also C12.1, C14.1, C13.1, C18.2, L3.2, R5.1; no longer C12.2, C14.2, R6.1
- net GND: now also C12.2, C14.2, C2.2, C3.2, R6.2, C13.2, C15.2, C16.2, C17.2; no longer C12.1, C14.1, C2.1, C3.1, R4.2
- net at U2.6 (VBST): now also C11.1
- net at U2.2 (SW): now also C11.2, L3.1
- net at U2.5 (EN): now also R4.1
- new net: C18.1, R5.2, R6.1, U2.4 (VFB)
Other:
- moved on the sheet: C1, C10, C2, C3, C5, C6, C7, C8, C9, L1, L2, R1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

Commit message: update
Parts:
- L1, L3: footprint Inductor_SMD:L_6.3x6.3_H3 -> Inductor_SMD:L_Changjiang_FXL0630
- L2: footprint Inductor_SMD:L_0603_1608Metric_Pad1.05x0.95mm_HandSolder -> Inductor_SMD:L_0603_1608Metric
Changed lines of the file:
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@@
 			)
 		)
-		(property "Footprint" "Inductor_SMD:L_6.3x6.3_H3"
+		(property "Footprint" "Inductor_SMD:L_Changjiang_FXL0630"
 			(at 130.81 115.57 0)
 			(effects
@@
 			)
 		)
-		(property "Footprint" "Inductor_SMD:L_0603_1608Metric_Pad1.05x0.95mm_HandSolder"
+		(property "Footprint" "Inductor_SMD:L_0603_1608Metric"
 			(at 208.28 72.39 0)
 			(effects
@@
 			)
 		)
-		(property "Footprint" "Inductor_SMD:L_6.3x6.3_H3"
+		(property "Footprint" "Inductor_SMD:L_Changjiang_FXL0630"
 			(at 130.81 63.5 0)
 			(effects

Commit message: update
Parts:
- added D7, D8: GREEN LED, LED_SMD:LED_0603_1608Metric, symbol Device:LED
- added R90: 270, Resistor_SMD:R_0603_1608Metric, symbol Device:R_Small
- added R91: 470, Resistor_SMD:R_0603_1608Metric, symbol Device:R_Small
Connections:
- net +3.3V: now also R90.2
- net +5V: now also R91.2
- net GND: now also D7.1 (K), D8.1 (K)
- new net: D7.2 (A), R90.1
- new net: D8.2 (A), R91.1

Commit message: update
Parts:
- J1: footprint Connector_BarrelJack:BarrelJack_CUI_PJ-102AH_Horizontal -> Connector_BarrelJack:BarrelJack_GCT_DCJ200-10-A_Horizontal
Changed lines of the file:
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@@
 			)
 		)
-		(property "Footprint" "Connector_BarrelJack:BarrelJack_CUI_PJ-102AH_Horizontal"
+		(property "Footprint" "Connector_BarrelJack:BarrelJack_GCT_DCJ200-10-A_Horizontal"
 			(at 44.45 30.226 0)
 			(effects

Commit message: update
Other:
- moved on the sheet: C10, C9, L2
Changed lines of the file:
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@@
 	)
 	(junction
-		(at 214.63 83.82)
+		(at 212.09 83.82)
 		(diameter 0)
 		(color 0 0 0 0)
@@
 	)
 	(junction
-		(at 214.63 72.39)
+		(at 212.09 72.39)
 		(diameter 0)
 		(color 0 0 0 0)
@@
 	)
 	(junction
-		(at 219.71 72.39)
+		(at 217.17 72.39)
 		(diameter 0)
 		(color 0 0 0 0)
@@
 	(wire
 		(pts
-			(xy 214.63 72.39) (xy 214.63 76.2)
+			(xy 212.09 72.39) (xy 212.09 76.2)
 		)
 		(stroke
@@
 	(wire
 		(pts
-			(xy 201.93 83.82) (xy 214.63 83.82)
+			(xy 199.39 83.82) (xy 212.09 83.82)
 		)
 		(stroke
@@
 	(wire
 		(pts
-			(xy 201.93 69.85) (xy 201.93 72.39)
+			(xy 199.39 69.85) (xy 199.39 72.39)
 		)
 		(stroke
@@
 	(wire
 		(pts
-			(xy 214.63 83.82) (xy 226.06 83.82)
+			(xy 212.09 83.82) (xy 223.52 83.82)
 		)
 		(stroke
@@
 	(wire
 		(pts
-			(xy 201.93 83.82) (xy 201.93 86.36)
+			(xy 199.39 83.82) (xy 199.39 86.36)
 		)
 		(stroke
@@
 	(wire
 		(pts
-			(xy 210.82 72.39) (xy 214.63 72.39)
+			(xy 208.28 72.39) (xy 212.09 72.39)
 		)
 		(stroke
@@
 	(wire
 		(pts
-			(xy 219.71 72.39) (xy 226.06 72.39)
+			(xy 217.17 72.39) (xy 223.52 72.39)
 		)
 		(stroke
@@
 	(wire
 		(pts
-			(xy 226.06 82.55) (xy 226.06 83.82)
+			(xy 223.52 82.55) (xy 223.52 83.82)
 		)
 		(stroke
@@
 	(wire
 		(pts
-			(xy 219.71 66.04) (xy 219.71 72.39)
+			(xy 217.17 66.04) (xy 217.17 72.39)
 		)
 		(stroke
@@
 	(wire
 		(pts
-			(xy 214.63 72.39) (xy 219.71 72.39)
+			(xy 212.09 72.39) (xy 217.17 72.39)
 		)
 		(stroke
@@
 	(wire
 		(pts
-			(xy 201.93 72.39) (xy 205.74 72.39)
+			(xy 199.39 72.39) (xy 203.2 72.39)
 		)
 		(stroke
@@
 	(wire
 		(pts
-			(xy 226.06 72.39) (xy 226.06 74.93)
+			(xy 223.52 72.39) (xy 223.52 74.93)
 		)
 		(stroke
@@
 	(wire
 		(pts
-			(xy 214.63 81.28) (xy 214.63 83.82)
+			(xy 212.09 81.28) (xy 212.09 83.82)
 		)
 		(stroke
@@
 	(hierarchical_label "+3.3V"
 		(shape input)
-		(at 201.93 69.85 90)
+		(at 199.39 69.85 90)
 		(effects
 			(font
@@
 	(hierarchical_label "VDDA"
 		(shape output)
-		(at 219.71 66.04 90)
+		(at 217.17 66.04 90)
 		(effects
 			(font
@@
 	(symbol
 		(lib_id "Device:C_Small")
-		(at 214.63 78.74 0)
+		(at 212.09 78.74 0)
 		(unit 1)
 		(exclude_from_sim no)
@@
 		(dnp no)
 		(property "Reference" "C9"
-			(at 217.17 77.724 0)
+			(at 214.63 77.724 0)
 			(effects
 				(font
@@
 		)
 		(property "Value" "0.1uF"
-			(at 217.17 80.264 0)
+			(at 214.63 80.264 0)
 			(effects
 				(font
@@
 		)
 		(property "Footprint" "Capacitor_SMD:C_0603_1608Metric"
-			(at 214.63 78.74 0)
+			(at 212.09 78.74 0)
 			(effects
 				(font
@@
 		)
 		(property "Datasheet" "~"
-			(at 214.63 78.74 0)
+			(at 212.09 78.74 0)
 			(effects
 				(font
@@
 		)
 		(property "Description" "Unpolarized capacitor, small symbol"
-			(at 214.63 78.74 0)
+			(at 212.09 78.74 0)
 			(effects
 				(font
@@
 	(symbol
 		(lib_id "Device:L_Small")
-		(at 208.28 72.39 90)
+		(at 205.74 72.39 90)
 		(unit 1)
 		(exclude_from_sim no)
@@
 		(fields_autoplaced yes)
 		(property "Reference" "L2"
-			(at 208.28 67.31 90)
+			(at 205.74 67.31 90)
 			(effects
 				(font
@@
 		)
 		(property "Value" "10uH"
-			(at 208.28 69.85 90)
+			(at 205.74 69.85 90)
 			(effects
 				(font
@@
 		)
 		(property "Footprint" "Inductor_SMD:L_0603_1608Metric"
-			(at 208.28 72.39 0)
+			(at 205.74 72.39 0)
 			(effects
 				(font
@@
 		)
 		(property "Datasheet" "~"
-			(at 208.28 72.39 0)
+			(at 205.74 72.39 0)
 			(effects
 				(font
@@
 		)
 		(property "Description" "Inductor, small symbol"
-			(at 208.28 72.39 0)
+			(at 205.74 72.39 0)
 			(effects
 				(font
@@
 	(symbol
 		(lib_id "power:GND")
-		(at 201.93 86.36 0)
+		(at 199.39 86.36 0)
 		(unit 1)
 		(exclude_from_sim no)
@@
 		(fields_autoplaced yes)
 		(property "Reference" "#PWR04"
-			(at 201.93 92.71 0)
+			(at 199.39 92.71 0)
 			(effects
 				(font
@@
 		)
 		(property "Value" "GND"
-			(at 201.93 91.44 0)
+			(at 199.39 91.44 0)
 			(effects
 				(font
@@
 		)
 		(property "Footprint" ""
-			(at 201.93 86.36 0)
+			(at 199.39 86.36 0)
 			(effects
 				(font
@@
 		)
 		(property "Datasheet" ""
-			(at 201.93 86.36 0)
+			(at 199.39 86.36 0)
 			(effects
 				(font
@@
 		)
 		(property "Description" "Power symbol creates a global label with name \"GND\" , ground"
-			(at 201.93 86.36 0)
+			(at 199.39 86.36 0)
 			(effects
 				(font
@@
 	(symbol
 		(lib_id "Device:C_Polarized")
-		(at 226.06 78.74 0)
+		(at 223.52 78.74 0)
 		(unit 1)
 		(exclude_from_sim no)
@@
 		(dnp no)
 		(property "Reference" "C10"
-			(at 229.362 78.232 0)
+			(at 226.822 78.232 0)
 			(effects
 				(font
@@
 		)
 		(property "Value" "10uF"
-			(at 229.616 80.518 0)
+			(at 227.076 80.518 0)
 			(effects
 				(font
@@
 		)
 		(property "Footprint" "Capacitor_SMD:C_0603_1608Metric"
-			(at 227.0252 82.55 0)
+			(at 224.4852 82.55 0)
 			(effects
 				(font
@@
 		)
 		(property "Datasheet" "~"
-			(at 226.06 78.74 0)
+			(at 223.52 78.74 0)
 			(effects
 				(font
@@
 		)
 		(property "Description" "Polarized capacitor"
-			(at 226.06 78.74 0)
+			(at 223.52 78.74 0)
 			(effects
 				(font

Commit message: update
Parts:
- removed C10: 10uF, Capacitor_SMD:C_0603_1608Metric, symbol Device:C_Polarized
- added C10: 10uF, Capacitor_SMD:C_0603_1608Metric, symbol Device:C_Small
Connections:
- net GND: now also C10.2
- net VDDA: now also C10.1
Changed lines of the file:
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@@
 	(wire
 		(pts
-			(xy 223.52 82.55) (xy 223.52 83.82)
+			(xy 223.52 81.28) (xy 223.52 83.82)
 		)
 		(stroke
@@
 	(wire
 		(pts
-			(xy 223.52 72.39) (xy 223.52 74.93)
+			(xy 223.52 72.39) (xy 223.52 76.2)
 		)
 		(stroke
@@
 	)
 	(symbol
+		(lib_id "Device:C_Small")
+		(at 223.52 78.74 0)
+		(unit 1)
+		(exclude_from_sim no)
+		(in_bom yes)
+		(on_board yes)
+		(dnp no)
+		(property "Reference" "C10"
+			(at 226.06 77.724 0)
+			(effects
+				(font
+					(size 1.27 1.27)
+				)
+				(justify left)
+			)
+		)
+		(property "Value" "10uF"
+			(at 226.06 80.264 0)
+			(effects
+				(font
+					(size 1.27 1.27)
+				)
+				(justify left)
+			)
+		)
+		(property "Footprint" "Capacitor_SMD:C_0603_1608Metric"
+			(at 223.52 78.74 0)
+			(effects
+				(font
+					(size 1.27 1.27)
+				)
+				(hide yes)
+			)
+		)
+		(property "Datasheet" "~"
+			(at 223.52 78.74 0)
+			(effects
+				(font
+					(size 1.27 1.27)
+				)
+				(hide yes)
+			)
+		)
+		(property "Description" "Unpolarized capacitor, small symbol"
+			(at 223.52 78.74 0)
+			(effects
+				(font
+					(size 1.27 1.27)
+				)
+				(hide yes)
+			)
+		)
+		(pin "1"
+		)
+		(pin "2"
+		)
+		(instances
+			(project "sac_board"
+				(path "/74ff6d0b-648c-43d9-a5b1-cc8d6cd1c1ef/ef74aba3-bc90-4bc5-a138-19d4fe3a7e12"
+					(reference "C10")
+					(unit 1)
+				)
+			)
+		)
+	)
+	(symbol
 		(lib_id "power:GND")
 		(at 104.14 132.08 0)
@@
 					(unit 1)
 				)
-			)
-		)
-	)
-	(symbol
-		(lib_id "Device:C_Polarized")
-		(at 223.52 78.74 0)
-		(unit 1)
-		(exclude_from_sim no)
-		(in_bom yes)
-		(on_board yes)
-		(dnp no)
-		(property "Reference" "C10"
-			(at 226.822 78.232 0)
-			(effects
-				(font
-					(size 1.27 1.27)
-				)
-				(justify left)
-			)
-		)
-		(property "Value" "10uF"
-			(at 227.076 80.518 0)
-			(effects
-				(font
-					(size 1.27 1.27)
-				)
-				(justify left)
-			)
-		)
-		(property "Footprint" "Capacitor_SMD:C_0603_1608Metric"
-			(at 224.4852 82.55 0)
-			(effects
-				(font
-					(size 1.27 1.27)
-				)
-				(hide yes)
-			)
-		)
-		(property "Datasheet" "~"
-			(at 223.52 78.74 0)
-			(effects
-				(font
-					(size 1.27 1.27)
-				)
-				(hide yes)
-			)
-		)
-		(property "Description" "Polarized capacitor"
-			(at 223.52 78.74 0)
-			(effects
-				(font
-					(size 1.27 1.27)
-				)
-				(hide yes)
-			)
-		)
-		(pin "1"
-		)
-		(pin "2"
-		)
-		(instances
-			(project "SmartArm"
-				(path "/74ff6d0b-648c-43d9-a5b1-cc8d6cd1c1ef/ef74aba3-bc90-4bc5-a138-19d4fe3a7e12"
-					(reference "C10")
-					(unit 1)
-				)
