File: power_servo.kicad_sch (KiCad schematic)
At the start: 144 parts, among them U10 TPS563201, U11 TPS563201, U12 TPS563201, U13 TPS563201, U14 TPS563201, U3 TPS563201, U4 TPS563201, U5 TPS563201, U6 TPS563201, U7 TPS563201, U8 TPS563201, U9 TPS563201

Commit message: update
Parts:
- C100: renamed from C83; footprint Capacitor_SMD:C_01005_0402Metric_Pad0.57x0.30mm_HandSolder -> Capacitor_SMD:C_0603_1608Metric
- C17: renamed from C24; footprint Capacitor_SMD:C_01005_0402Metric_Pad0.57x0.30mm_HandSolder -> Capacitor_SMD:C_0603_1608Metric
- C18: renamed from C45; footprint Capacitor_SMD:C_01005_0402Metric_Pad0.57x0.30mm_HandSolder -> Capacitor_SMD:C_0603_1608Metric
- C19: renamed from C66; footprint Capacitor_SMD:C_01005_0402Metric_Pad0.57x0.30mm_HandSolder -> Capacitor_SMD:C_0603_1608Metric
- C20: renamed from C87; footprint Capacitor_SMD:C_01005_0402Metric_Pad0.57x0.30mm_HandSolder -> Capacitor_SMD:C_0603_1608Metric
- C21: renamed from C25; footprint Capacitor_SMD:C_01005_0402Metric_Pad0.57x0.30mm_HandSolder -> Capacitor_SMD:C_0603_1608Metric
- C22: renamed from C46; footprint Capacitor_SMD:C_01005_0402Metric_Pad0.57x0.30mm_HandSolder -> Capacitor_SMD:C_0603_1608Metric
- C23: renamed from C67; footprint Capacitor_SMD:C_01005_0402Metric_Pad0.57x0.30mm_HandSolder -> Capacitor_SMD:C_0603_1608Metric
- C24: renamed from C88; footprint Capacitor_SMD:C_01005_0402Metric_Pad0.57x0.30mm_HandSolder -> Capacitor_SMD:C_0603_1608Metric
- C25: renamed from C26; footprint Capacitor_SMD:C_01005_0402Metric_Pad0.57x0.30mm_HandSolder -> Capacitor_SMD:C_0603_1608Metric
- C26: renamed from C47; footprint Capacitor_SMD:C_01005_0402Metric_Pad0.57x0.30mm_HandSolder -> Capacitor_SMD:C_0603_1608Metric
- C27: renamed from C68; footprint Capacitor_SMD:C_01005_0402Metric_Pad0.57x0.30mm_HandSolder -> Capacitor_SMD:C_0603_1608Metric
- C28: renamed from C89; footprint Capacitor_SMD:C_01005_0402Metric_Pad0.57x0.30mm_HandSolder -> Capacitor_SMD:C_0603_1608Metric
- C29: renamed from C21; footprint Capacitor_SMD:C_01005_0402Metric_Pad0.57x0.30mm_HandSolder -> Capacitor_SMD:C_0603_1608Metric
- C30: renamed from C42; footprint Capacitor_SMD:C_01005_0402Metric_Pad0.57x0.30mm_HandSolder -> Capacitor_SMD:C_0603_1608Metric
- C31: renamed from C63; footprint Capacitor_SMD:C_01005_0402Metric_Pad0.57x0.30mm_HandSolder -> Capacitor_SMD:C_0603_1608Metric
- C32: renamed from C84; footprint Capacitor_SMD:C_01005_0402Metric_Pad0.57x0.30mm_HandSolder -> Capacitor_SMD:C_0603_1608Metric
- C33: footprint Capacitor_SMD:C_01005_0402Metric_Pad0.57x0.30mm_HandSolder -> Capacitor_SMD:C_0603_1608Metric
- C34: renamed from C54; footprint Capacitor_SMD:C_01005_0402Metric_Pad0.57x0.30mm_HandSolder -> Capacitor_SMD:C_0603_1608Metric
- C35: renamed from C75; footprint Capacitor_SMD:C_01005_0402Metric_Pad0.57x0.30mm_HandSolder -> Capacitor_SMD:C_0603_1608Metric
- C36: renamed from C96; footprint Capacitor_SMD:C_01005_0402Metric_Pad0.57x0.30mm_HandSolder -> Capacitor_SMD:C_0603_1608Metric
- C38: renamed from C36; footprint Capacitor_SMD:C_01005_0402Metric_Pad0.57x0.30mm_HandSolder -> Capacitor_SMD:C_0603_1608Metric
- C39: renamed from C57; footprint Capacitor_SMD:C_01005_0402Metric_Pad0.57x0.30mm_HandSolder -> Capacitor_SMD:C_0603_1608Metric
- C40: renamed from C78; footprint Capacitor_SMD:C_01005_0402Metric_Pad0.57x0.30mm_HandSolder -> Capacitor_SMD:C_0603_1608Metric
- C41: renamed from C16; footprint Capacitor_SMD:C_01005_0402Metric_Pad0.57x0.30mm_HandSolder -> Capacitor_SMD:C_0603_1608Metric
- C42: renamed from C37; footprint Capacitor_SMD:C_01005_0402Metric_Pad0.57x0.30mm_HandSolder -> Capacitor_SMD:C_0603_1608Metric
- C43: renamed from C58; footprint Capacitor_SMD:C_01005_0402Metric_Pad0.57x0.30mm_HandSolder -> Capacitor_SMD:C_0603_1608Metric
- C44: renamed from C79; footprint Capacitor_SMD:C_01005_0402Metric_Pad0.57x0.30mm_HandSolder -> Capacitor_SMD:C_0603_1608Metric
- C45: renamed from C27; footprint Capacitor_SMD:C_01005_0402Metric_Pad0.57x0.30mm_HandSolder -> Capacitor_SMD:C_0603_1608Metric
- C46: renamed from C48; footprint Capacitor_SMD:C_01005_0402Metric_Pad0.57x0.30mm_HandSolder -> Capacitor_SMD:C_0603_1608Metric
- C47: renamed from C69; footprint Capacitor_SMD:C_01005_0402Metric_Pad0.57x0.30mm_HandSolder -> Capacitor_SMD:C_0603_1608Metric
- C48: renamed from C90; footprint Capacitor_SMD:C_01005_0402Metric_Pad0.57x0.30mm_HandSolder -> Capacitor_SMD:C_0603_1608Metric
- C49: renamed from C28; footprint Capacitor_SMD:C_01005_0402Metric_Pad0.57x0.30mm_HandSolder -> Capacitor_SMD:C_0603_1608Metric
- C50: renamed from C49; footprint Capacitor_SMD:C_01005_0402Metric_Pad0.57x0.30mm_HandSolder -> Capacitor_SMD:C_0603_1608Metric
- C51: renamed from C70; footprint Capacitor_SMD:C_01005_0402Metric_Pad0.57x0.30mm_HandSolder -> Capacitor_SMD:C_0603_1608Metric
- C52: renamed from C91; footprint Capacitor_SMD:C_01005_0402Metric_Pad0.57x0.30mm_HandSolder -> Capacitor_SMD:C_0603_1608Metric
- C53: renamed from C29; footprint Capacitor_SMD:C_01005_0402Metric_Pad0.57x0.30mm_HandSolder -> Capacitor_SMD:C_0603_1608Metric
- C54: renamed from C50; footprint Capacitor_SMD:C_01005_0402Metric_Pad0.57x0.30mm_HandSolder -> Capacitor_SMD:C_0603_1608Metric
- C55: renamed from C71; footprint Capacitor_SMD:C_01005_0402Metric_Pad0.57x0.30mm_HandSolder -> Capacitor_SMD:C_0603_1608Metric
- C56: renamed from C92; footprint Capacitor_SMD:C_01005_0402Metric_Pad0.57x0.30mm_HandSolder -> Capacitor_SMD:C_0603_1608Metric
- C57: renamed from C22; footprint Capacitor_SMD:C_01005_0402Metric_Pad0.57x0.30mm_HandSolder -> Capacitor_SMD:C_0603_1608Metric
- C58: renamed from C43; footprint Capacitor_SMD:C_01005_0402Metric_Pad0.57x0.30mm_HandSolder -> Capacitor_SMD:C_0603_1608Metric
- C59: renamed from C64; footprint Capacitor_SMD:C_01005_0402Metric_Pad0.57x0.30mm_HandSolder -> Capacitor_SMD:C_0603_1608Metric
- C60: renamed from C85; footprint Capacitor_SMD:C_01005_0402Metric_Pad0.57x0.30mm_HandSolder -> Capacitor_SMD:C_0603_1608Metric
- C61: renamed from C34; footprint Capacitor_SMD:C_01005_0402Metric_Pad0.57x0.30mm_HandSolder -> Capacitor_SMD:C_0603_1608Metric
- C62: renamed from C55; footprint Capacitor_SMD:C_01005_0402Metric_Pad0.57x0.30mm_HandSolder -> Capacitor_SMD:C_0603_1608Metric
- C63: renamed from C76; footprint Capacitor_SMD:C_01005_0402Metric_Pad0.57x0.30mm_HandSolder -> Capacitor_SMD:C_0603_1608Metric
- C64: renamed from C97; footprint Capacitor_SMD:C_01005_0402Metric_Pad0.57x0.30mm_HandSolder -> Capacitor_SMD:C_0603_1608Metric
- C65: renamed from C17; footprint Capacitor_SMD:C_01005_0402Metric_Pad0.57x0.30mm_HandSolder -> Capacitor_SMD:C_0603_1608Metric
- C66: renamed from C38; footprint Capacitor_SMD:C_01005_0402Metric_Pad0.57x0.30mm_HandSolder -> Capacitor_SMD:C_0603_1608Metric
- C67: renamed from C59; footprint Capacitor_SMD:C_01005_0402Metric_Pad0.57x0.30mm_HandSolder -> Capacitor_SMD:C_0603_1608Metric
- C68: renamed from C80; footprint Capacitor_SMD:C_01005_0402Metric_Pad0.57x0.30mm_HandSolder -> Capacitor_SMD:C_0603_1608Metric
- C69: renamed from C18; footprint Capacitor_SMD:C_01005_0402Metric_Pad0.57x0.30mm_HandSolder -> Capacitor_SMD:C_0603_1608Metric
- C70: renamed from C39; footprint Capacitor_SMD:C_01005_0402Metric_Pad0.57x0.30mm_HandSolder -> Capacitor_SMD:C_0603_1608Metric
- C71: renamed from C60; footprint Capacitor_SMD:C_01005_0402Metric_Pad0.57x0.30mm_HandSolder -> Capacitor_SMD:C_0603_1608Metric
- C72: renamed from C81; footprint Capacitor_SMD:C_01005_0402Metric_Pad0.57x0.30mm_HandSolder -> Capacitor_SMD:C_0603_1608Metric
- C73: renamed from C30; footprint Capacitor_SMD:C_01005_0402Metric_Pad0.57x0.30mm_HandSolder -> Capacitor_SMD:C_0603_1608Metric
- C74: renamed from C51; footprint Capacitor_SMD:C_01005_0402Metric_Pad0.57x0.30mm_HandSolder -> Capacitor_SMD:C_0603_1608Metric
- C75: renamed from C72; footprint Capacitor_SMD:C_01005_0402Metric_Pad0.57x0.30mm_HandSolder -> Capacitor_SMD:C_0603_1608Metric
- C76: renamed from C93; footprint Capacitor_SMD:C_01005_0402Metric_Pad0.57x0.30mm_HandSolder -> Capacitor_SMD:C_0603_1608Metric
- C77: renamed from C31; footprint Capacitor_SMD:C_01005_0402Metric_Pad0.57x0.30mm_HandSolder -> Capacitor_SMD:C_0603_1608Metric
- C78: renamed from C52; footprint Capacitor_SMD:C_01005_0402Metric_Pad0.57x0.30mm_HandSolder -> Capacitor_SMD:C_0603_1608Metric
- C79: renamed from C73; footprint Capacitor_SMD:C_01005_0402Metric_Pad0.57x0.30mm_HandSolder -> Capacitor_SMD:C_0603_1608Metric
- C80: renamed from C94; footprint Capacitor_SMD:C_01005_0402Metric_Pad0.57x0.30mm_HandSolder -> Capacitor_SMD:C_0603_1608Metric
- C81: renamed from C32; footprint Capacitor_SMD:C_01005_0402Metric_Pad0.57x0.30mm_HandSolder -> Capacitor_SMD:C_0603_1608Metric
- C82: renamed from C53; footprint Capacitor_SMD:C_01005_0402Metric_Pad0.57x0.30mm_HandSolder -> Capacitor_SMD:C_0603_1608Metric
- C83: renamed from C74; footprint Capacitor_SMD:C_01005_0402Metric_Pad0.57x0.30mm_HandSolder -> Capacitor_SMD:C_0603_1608Metric
- C84: renamed from C95; footprint Capacitor_SMD:C_01005_0402Metric_Pad0.57x0.30mm_HandSolder -> Capacitor_SMD:C_0603_1608Metric
- C85: renamed from C23; footprint Capacitor_SMD:C_01005_0402Metric_Pad0.57x0.30mm_HandSolder -> Capacitor_SMD:C_0603_1608Metric
- C86: renamed from C44; footprint Capacitor_SMD:C_01005_0402Metric_Pad0.57x0.30mm_HandSolder -> Capacitor_SMD:C_0603_1608Metric
- C87: renamed from C65; footprint Capacitor_SMD:C_01005_0402Metric_Pad0.57x0.30mm_HandSolder -> Capacitor_SMD:C_0603_1608Metric
- C88: renamed from C86; footprint Capacitor_SMD:C_01005_0402Metric_Pad0.57x0.30mm_HandSolder -> Capacitor_SMD:C_0603_1608Metric
- C89: renamed from C35; footprint Capacitor_SMD:C_01005_0402Metric_Pad0.57x0.30mm_HandSolder -> Capacitor_SMD:C_0603_1608Metric
- C90: renamed from C56; footprint Capacitor_SMD:C_01005_0402Metric_Pad0.57x0.30mm_HandSolder -> Capacitor_SMD:C_0603_1608Metric
- C91: renamed from C77; footprint Capacitor_SMD:C_01005_0402Metric_Pad0.57x0.30mm_HandSolder -> Capacitor_SMD:C_0603_1608Metric
- C92: renamed from C98; footprint Capacitor_SMD:C_01005_0402Metric_Pad0.57x0.30mm_HandSolder -> Capacitor_SMD:C_0603_1608Metric
- C93: renamed from C19; footprint Capacitor_SMD:C_01005_0402Metric_Pad0.57x0.30mm_HandSolder -> Capacitor_SMD:C_0603_1608Metric
- C94: renamed from C40; footprint Capacitor_SMD:C_01005_0402Metric_Pad0.57x0.30mm_HandSolder -> Capacitor_SMD:C_0603_1608Metric
- C95: renamed from C61; footprint Capacitor_SMD:C_01005_0402Metric_Pad0.57x0.30mm_HandSolder -> Capacitor_SMD:C_0603_1608Metric
- C96: renamed from C82; footprint Capacitor_SMD:C_01005_0402Metric_Pad0.57x0.30mm_HandSolder -> Capacitor_SMD:C_0603_1608Metric
- C97: renamed from C20; footprint Capacitor_SMD:C_01005_0402Metric_Pad0.57x0.30mm_HandSolder -> Capacitor_SMD:C_0603_1608Metric
- C98: renamed from C41; footprint Capacitor_SMD:C_01005_0402Metric_Pad0.57x0.30mm_HandSolder -> Capacitor_SMD:C_0603_1608Metric
- C99: renamed from C62; footprint Capacitor_SMD:C_01005_0402Metric_Pad0.57x0.30mm_HandSolder -> Capacitor_SMD:C_0603_1608Metric
- renumbered C15 to C37, L13 to L11, L5 to L12, L8 to L13, L11 to L14, L14 to L15, L3 to L4, L6 to L5, L9 to L6, L12 to L7, L4 to L8, L7 to L9, R34 to R10, R13 to R11, R22 to R12, R31 to R13, R40 to R14, R8 to R15, R17 to R16, R26 to R17, R35 to R18, R9 to R19, R18 to R20, R27 to R21, R36 to R22, R14 to R23, R23 to R24, R32 to R25, R41 to R26, R10 to R27, R19 to R28, R28 to R29, R37 to R30, R11 to R31, R20 to R32, R29 to R33, R38 to R34, R15 to R35, R24 to R36, R33 to R37, R42 to R38, R12 to R39, R21 to R40, R30 to R41, R39 to R42, R16 to R8, R25 to R9, U13 to U10, U5 to U11, U8 to U12, U11 to U13, U6 to U4, U9 to U5, U12 to U6, U4 to U7, U7 to U8, U10 to U9

Commit message: update
Parts:
- removed C17, C18: 22uF, Capacitor_SMD:C_0603_1608Metric, symbol Device:C_Small
- added C101: 22uF, Capacitor_SMD:C_1206_3216Metric, symbol Device:C_Small
- added C102, C104, C105, C107, C108, C110, C111: 10uF, Capacitor_SMD:C_1206_3216Metric, symbol Device:C_Small
- added C103, C106, C109: 0.1uF, Capacitor_SMD:C_0603_1608Metric, symbol Device:C_Small
- added C112, C113, C114: 10pF, Capacitor_SMD:C_0603_1608Metric, symbol Device:C_Small
- C100, C22, C23, C25, C26, C28, C46, C47, C49, C50, C52, C53, C70, C71, C73, C74, C76, C77, C94, C95, C97, C98: footprint Capacitor_SMD:C_0603_1608Metric -> Capacitor_SMD:C_1206_3216Metric
- C19, C20, C21, C37, C43, C44, C45, C55, C67, C68, C69, C79, C82, C93: value 22uF -> 0.1uF
- C24, C27, C38, C39, C48, C51, C54, C56, C72, C75, C78, C80, C81, C83, C84, C96, C99: value 22uF -> 10uF; footprint Capacitor_SMD:C_0603_1608Metric -> Capacitor_SMD:C_1206_3216Metric
- C29: value 0.1uF -> 22uF; footprint Capacitor_SMD:C_0603_1608Metric -> Capacitor_SMD:C_1206_3216Metric
- C30, C32, C57, C59, C60, C86, C87: value 0.1uF -> 10uF; footprint Capacitor_SMD:C_0603_1608Metric -> Capacitor_SMD:C_1206_3216Metric
- C33, C35, C36, C62, C63: value 220uF -> 10uF; footprint Capacitor_SMD:C_0603_1608Metric -> Capacitor_SMD:C_1206_3216Metric
- C34, C61, C91, C92: value 220uF -> 0.1uF
- C40, C41, C42, C65, C66: value 22uF -> 10pF
- C64, C89, C90: value 220uF -> 10pF
- C88: value 0.1uF -> 10pF
- L10, L11, L12, L13, L14, L15, L4, L5, L6, L7, L8, L9: footprint Inductor_SMD:L_0603_1608Metric_Pad1.05x0.95mm_HandSolder -> Inductor_SMD:L_6.3x6.3_H3
- R10, R11, R12, R19, R20, R21, R37, R38: value 10K -> 82K
- R15, R16, R17, R18, R27, R40, R41, R42: value 82K -> 10K
Connections:
- net +12V: now also C31.1, C32.1, C33.1, C34.1, C35.1, C36.1, C37.1, C38.1, C39.1, C57.1, C58.1, C59.1, C60.1, C61.1, C62.1, C63.1, C85.1, C86.1, C87.1, R16.2, R17.2, R18.2, R25.2, R26.2, R27.2, R35.2, R36.2, C103.1, C104.1, C105.1, C106.1, C107.1, C108.1, C109.1, C110.1, C111.1; no longer C19.1, C20.1, C21.1, C22.1, C23.1, C24.1, C25.1, C26.1, C27.1, C28.1, C45.1, C46.1, C47.1, C48.1, C49.1, C50.1, C51.1, C52.1, C53.1, C54.1, C73.1, C74.1, C75.1, C76.1, C77.1, C78.1, R10.2, R19.2, R20.2, R21.2, R22.2, R31.2, R32.2, R33.2
- net +7V_M1: now also C22.1, C23.1, C24.1, C40.2, R10.1; no longer C33.2, C37.2, C41.2, R15.1
- net +7V_M10: now also C94.1, C95.1, C96.1, R37.1, C112.2; no longer C90.2, C94.2, C98.2, R40.1
- net +7V_M11: now also C97.1, C98.1, C99.1, R38.1, C113.2; no longer C91.2, C95.2, C99.2, R41.1
- net +7V_M12: now also C100.1, R39.1, C101.1, C102.1, C114.2; no longer C100.2, C92.2, C96.2, R42.1
- net +7V_M2: now also C25.1, C26.1, C27.1, C41.2, R11.1; no longer C34.2, C38.2, C42.2, R16.1
- net +7V_M3: now also C28.1, C29.1, C30.1, C42.2, R12.1; no longer C35.2, C39.2, C43.2, R17.1
- net +7V_M4: now also C46.1, C47.1, C48.1, C64.2, R19.1; no longer C36.2, C40.2, C44.2, R18.1
- net +7V_M5: now also C49.1, C50.1, C51.1, R20.1; no longer C61.2, C69.2, R27.1
- net +7V_M6: now also C52.1, C53.1, C54.1, R21.1; no longer C62.2, C70.2, R28.1
- net +7V_M7: now also C70.1, C71.1, C72.1, C88.2, R28.1; no longer C63.2, C67.2, C71.2, R29.1
- net +7V_M8: now also C73.1, C74.1, C75.1, C89.2, R29.1; no longer C64.2, C68.2, C72.2, R30.1
- net +7V_M9: now also C76.1, C77.1, C78.1, C90.2, R30.1; no longer C89.2, C93.2, C97.2, R39.1
- net GND: now also C100.2, C29.2, C30.2, C31.2, C32.2, C33.2, C34.2, C35.2, C36.2, C37.2, C38.2, C39.2, C57.2, C58.2, C59.2, C60.2, C61.2, C62.2, C63.2, C70.2, C71.2, C72.2, C85.2, C86.2, C87.2, C94.2, C95.2, C96.2, C97.2, C98.2, C99.2, R15.2, R22.2, R31.2, R32.2, R33.2, R40.2, R41.2, R42.2, C101.2, C102.2, C103.2, C104.2, C105.2, C106.2, C107.2, C108.2, C109.2, C110.2, C111.2; no longer C100.1, C19.2, C20.2, C21.2, C37.1, C38.1, C39.1, C40.1, C41.1, C42.1, C43.1, C44.1, C45.2, C65.1, C66.1, C67.1, C68.1, C69.1, C70.1, C71.1, C72.1, C93.1, C94.1, C95.1, C96.1, C97.1, C98.1, C99.1, R11.2, R12.2, R25.2, R26.2, R35.2, R36.2, R37.2, R38.2
- net at U7.5 (EN): now also R17.1; no longer R19.1
- net at L14.1, U13.2 (SW): now also C92.2; no longer C87.2
- net at R31.1: now also C88.1, R28.2, U9.4 (VFB); no longer U11.5 (EN)
- net at U13.5 (EN): now also R35.1; no longer R33.1
- net at L13.1, U12.2 (SW): now also C91.2; no longer C86.2
- net at R32.1: now also C89.1, R29.2, U10.4 (VFB); no longer U12.5 (EN)
- net at U12.6 (VBST): now also C91.1; no longer C86.1
- net at R22.1: now also C64.1, R19.2, U6.4 (VFB); no longer U10.5 (EN)
- net at U6.6 (VBST): now also C43.1; no longer C32.1
- net at L7.1, U6.2 (SW): now also C43.2; no longer C32.2
- net at L8.1, U7.2 (SW): now also C44.2; no longer C57.2
- net at R23.1, U7.4 (VFB): now also C65.1, R20.2; no longer C61.1, R27.2
- net at U7.6 (VBST): now also C44.1; no longer C57.1
- net at L15.1, U14.2 (SW): now also C93.2; no longer C88.2
- net at U14.5 (EN): now also R36.1; no longer R34.1
- net at U14.6 (VBST): now also C93.1; no longer C88.1
- net at U13.6 (VBST): now also C92.1; no longer C87.1
- net at U11.6 (VBST): now also C69.1; no longer C85.1
- net at L12.1, U11.2 (SW): now also C69.2; no longer C85.2
- net at U5.6 (VBST): now also C21.1; no longer C31.1
- net at L6.1, U5.2 (SW): now also C21.2; no longer C31.2
- net at L9.1, U8.2 (SW): now also C45.2; no longer C58.2
- net at L10.1, U9.2 (SW): now also C67.2; no longer C59.2
- net at L5.1, U4.2 (SW): now also C20.2; no longer C30.2
- net at U8.6 (VBST): now also C45.1; no longer C58.1
- net at U8.5 (EN): now also R18.1; no longer R20.1
- net at L11.1, U10.2 (SW): now also C68.2; no longer C60.2
- net at U4.6 (VBST): now also C20.1; no longer C30.1
- net at L4.1, U3.2 (SW): now also C19.2; no longer C29.2
- net at U3.6 (VBST): now also C19.1; no longer C29.1
- net at R24.1, U8.4 (VFB): now also C66.1, R21.2; no longer C62.1, R28.2
- net at U9.5 (EN): now also R25.1; no longer R21.1
- net at U9.6 (VBST): now also C67.1; no longer C59.1
- net at U6.5 (EN): now also R16.1; no longer R10.1
- net at U10.6 (VBST): now also C68.1; no longer C60.1
- new net: C114.1, R39.2, R42.1, U14.4 (VFB)
- new net: C112.1, R37.2, R40.1, U12.4 (VFB)
- new net: C113.1, R38.2, R41.1, U13.4 (VFB)
- new net: C41.1, R11.2, R14.1, U4.4 (VFB)
- new net: R27.1, U11.5 (EN)
- new net: C42.1, R12.2, R15.1, U5.4 (VFB)
- new net: R34.1, U12.5 (EN)
- new net: R26.1, U10.5 (EN)
- new net: C90.1, R30.2, R33.1, U11.4 (VFB)
- new net: C40.1, R10.2, R13.1, U3.4 (VFB)

Commit message: update
Parts:
- removed C100, C101, C76, C77, C94, C95, C97, C98: 22uF, Capacitor_SMD:C_1206_3216Metric, symbol Device:C_Small
- removed C102, C104, C105, C107, C108, C110, C111, C78, C86, C87, C96, C99: 10uF, Capacitor_SMD:C_1206_3216Metric, symbol Device:C_Small
- removed C103, C106, C109, C69, C85, C91, C92, C93: 0.1uF, Capacitor_SMD:C_0603_1608Metric, symbol Device:C_Small
- removed C112, C113, C114, C90: 10pF, Capacitor_SMD:C_0603_1608Metric, symbol Device:C_Small
- removed L12, L13, L14, L15: 2.2uH, Inductor_SMD:L_6.3x6.3_H3, symbol Device:L_Small
- removed R27, R33, R34, R35, R36, R40, R41, R42: 10K, Resistor_SMD:R_0603_1608Metric, symbol Device:R_Small
- removed R30, R37, R38, R39: 82K, Resistor_SMD:R_0603_1608Metric, symbol Device:R_Small
- removed U11, U12, U13, U14: TPS563201, Package_TO_SOT_SMD:SOT-23-6, symbol Regulator_Switching:TPS563200
- L10, L11, L4, L5, L6, L7, L8, L9: footprint Inductor_SMD:L_6.3x6.3_H3 -> Inductor_SMD:L_Changjiang_FXL0630
- renumbered C70 to C69, C71 to C70, C72 to C71, C73 to C72, C74 to C73, C75 to C74, C79 to C75, C80 to C76, C81 to C77, C82 to C78, C83 to C79, C84 to C80, C88 to C81, C89 to C82, R28 to R27, R29 to R28, R31 to R29, R32 to R30

Commit message: update
Connections:
- net +7V_M1 renamed V_M1
- net +7V_M2 renamed V_M2
- net +7V_M3 renamed V_M3
- net +7V_M4 renamed V_M4
- net +7V_M5 renamed V_M5
- net +7V_M6 renamed V_M6
- net +7V_M7 renamed V_M7
- net +7V_M8 renamed V_M8
Other:
- moved on the sheet: C19, C20, C21, C22, C23, C24, C25, C26, C27, C28, C29, C30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

Commit message: update
Other:
- note added: "TPS563201 Output Voltage Resistors Selection Vout = 0.768 x (1.0+R1/R2) R1: 82K R2: 10K Output: 7.06V"
Changed lines of the file:
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@@
 	(generator_version "9.0")
 	(paper "A3")
+	(text "TPS563201 Output Voltage Resistors Selection\nVout = 0.768 x (1.0+R1/R2)\nR1: 82K\nR2: 10K\nOutput: 7.06V"
+		(exclude_from_sim no)
+		(at 73.406 36.83 0)
+		(effects
+			(font
+				(size 1.27 1.27)
+			)
+			(justify left)
+		)
+	)
 	(junction
 		(at 308.61 71.12)

Commit message: update
Parts:
- C23: renamed from C38; footprint Capacitor_SMD:C_1206_3216Metric -> Capacitor_SMD:C_0603_1608Metric
- C24: renamed from C32; footprint Capacitor_SMD:C_1206_3216Metric -> Capacitor_SMD:C_0603_1608Metric
- C25: renamed from C59; footprint Capacitor_SMD:C_1206_3216Metric -> Capacitor_SMD:C_0603_1608Metric
- C26: renamed from C76; footprint Capacitor_SMD:C_1206_3216Metric -> Capacitor_SMD:C_0603_1608Metric
- C27: renamed from C39; footprint Capacitor_SMD:C_1206_3216Metric -> Capacitor_SMD:C_0603_1608Metric
- C28: renamed from C33; footprint Capacitor_SMD:C_1206_3216Metric -> Capacitor_SMD:C_0603_1608Metric
- C29: renamed from C60; footprint Capacitor_SMD:C_1206_3216Metric -> Capacitor_SMD:C_0603_1608Metric
- C30: renamed from C77; footprint Capacitor_SMD:C_1206_3216Metric -> Capacitor_SMD:C_0603_1608Metric
- C35: renamed from C28; footprint Capacitor_SMD:C_1206_3216Metric -> Capacitor_SMD:C_0603_1608Metric
- C36: renamed from C22; footprint Capacitor_SMD:C_1206_3216Metric -> Capacitor_SMD:C_0603_1608Metric
- C37: renamed from C49; footprint Capacitor_SMD:C_1206_3216Metric -> Capacitor_SMD:C_0603_1608Metric
- C38: renamed from C69; footprint Capacitor_SMD:C_1206_3216Metric -> Capacitor_SMD:C_0603_1608Metric
- C39: renamed from C29; footprint Capacitor_SMD:C_1206_3216Metric -> Capacitor_SMD:C_0603_1608Metric
- C40: renamed from C23; footprint Capacitor_SMD:C_1206_3216Metric -> Capacitor_SMD:C_0603_1608Metric
- C41: renamed from C50; footprint Capacitor_SMD:C_1206_3216Metric -> Capacitor_SMD:C_0603_1608Metric
- C42: renamed from C70; footprint Capacitor_SMD:C_1206_3216Metric -> Capacitor_SMD:C_0603_1608Metric
- C43: renamed from C30; footprint Capacitor_SMD:C_1206_3216Metric -> Capacitor_SMD:C_0603_1608Metric
- C44: renamed from C24; footprint Capacitor_SMD:C_1206_3216Metric -> Capacitor_SMD:C_0603_1608Metric
- C45: renamed from C51; footprint Capacitor_SMD:C_1206_3216Metric -> Capacitor_SMD:C_0603_1608Metric
- C46: renamed from C71; footprint Capacitor_SMD:C_1206_3216Metric -> Capacitor_SMD:C_0603_1608Metric
- C55: renamed from C62; footprint Capacitor_SMD:C_1206_3216Metric -> Capacitor_SMD:C_0603_1608Metric
- C56: renamed from C35; footprint Capacitor_SMD:C_1206_3216Metric -> Capacitor_SMD:C_0603_1608Metric
- C57: renamed from C56; footprint Capacitor_SMD:C_1206_3216Metric -> Capacitor_SMD:C_0603_1608Metric
- C58: renamed from C79; footprint Capacitor_SMD:C_1206_3216Metric -> Capacitor_SMD:C_0603_1608Metric
- C59: renamed from C63; footprint Capacitor_SMD:C_1206_3216Metric -> Capacitor_SMD:C_0603_1608Metric
- C60: renamed from C36; footprint Capacitor_SMD:C_1206_3216Metric -> Capacitor_SMD:C_0603_1608Metric
- C61: renamed from C57; footprint Capacitor_SMD:C_1206_3216Metric -> Capacitor_SMD:C_0603_1608Metric
- C62: renamed from C80; footprint Capacitor_SMD:C_1206_3216Metric -> Capacitor_SMD:C_0603_1608Metric
- C67: renamed from C52; footprint Capacitor_SMD:C_1206_3216Metric -> Capacitor_SMD:C_0603_1608Metric
- C68: renamed from C25; footprint Capacitor_SMD:C_1206_3216Metric -> Capacitor_SMD:C_0603_1608Metric
- C69: renamed from C46; footprint Capacitor_SMD:C_1206_3216Metric -> Capacitor_SMD:C_0603_1608Metric
- C70: renamed from C72; footprint Capacitor_SMD:C_1206_3216Metric -> Capacitor_SMD:C_0603_1608Metric
- C71: renamed from C53; footprint Capacitor_SMD:C_1206_3216Metric -> Capacitor_SMD:C_0603_1608Metric
- C72: renamed from C26; footprint Capacitor_SMD:C_1206_3216Metric -> Capacitor_SMD:C_0603_1608Metric
- C73: renamed from C47; footprint Capacitor_SMD:C_1206_3216Metric -> Capacitor_SMD:C_0603_1608Metric
- C74: renamed from C73; footprint Capacitor_SMD:C_1206_3216Metric -> Capacitor_SMD:C_0603_1608Metric
- C75: renamed from C54; footprint Capacitor_SMD:C_1206_3216Metric -> Capacitor_SMD:C_0603_1608Metric
- C76: renamed from C27; footprint Capacitor_SMD:C_1206_3216Metric -> Capacitor_SMD:C_0603_1608Metric
- C77: renamed from C48; footprint Capacitor_SMD:C_1206_3216Metric -> Capacitor_SMD:C_0603_1608Metric
- C78: renamed from C74; footprint Capacitor_SMD:C_1206_3216Metric -> Capacitor_SMD:C_0603_1608Metric
- renumbered C37 to C19, C31 to C20, C58 to C21, C75 to C22, C21 to C31, C19 to C32, C44 to C33, C67 to C34, C42 to C47, C40 to C48, C65 to C49, C81 to C50, C61 to C51, C34 to C52, C55 to C53, C78 to C54, C45 to C63, C20 to C64, C43 to C65, C68 to C66, C66 to C79, C41 to C80, C64 to C81, L7 to L10, L6 to L4, L4 to L5, L8 to L6, L10 to L7, L9 to L8, L5 to L9, R7 to R10, R17 to R11, R25 to R12, R12 to R13, R15 to R14, R10 to R15, R13 to R16, R20 to R17, R23 to R18, R27 to R19, R29 to R20, R18 to R21, R8 to R22, R16 to R23, R26 to R24, R21 to R25, R24 to R26, R11 to R27, R14 to R28, R19 to R29, R22 to R30, R28 to R31, R30 to R32, U5 to U3, U3 to U4, U7 to U5, U9 to U6, U8 to U7, U4 to U8, U6 to U9

Commit message: update
Parts:
- added D10, D11, D12, D13, D14, D7, D8, D9: WHITE LED, LED_SMD:LED_0603_1608Metric, symbol Device:LED
- added R76, R77, R78, R79, R80, R81, R82, R83: 220, Resistor_SMD:R_0603_1608Metric, symbol Device:R_Small
Connections:
- net GND: now also D10.1 (K), D11.1 (K), D12.1 (K), D13.1 (K), D14.1 (K), D7.1 (K), D8.1 (K), D9.1 (K)
- net V_M1: now also R76.2
- net V_M2: now also R77.2
- net V_M3: now also R78.2
- net V_M4: now also R79.2
- net V_M5: now also R80.2
- net V_M6: now also R81.2
- net V_M7: now also R82.2
- net V_M8: now also R83.2
- new net: D10.2 (A), R79.1
- new net: D8.2 (A), R77.1
- new net: D11.2 (A), R80.1
- new net: D12.2 (A), R81.1
- new net: D13.2 (A), R82.1
- new net: D14.2 (A), R83.1
- new net: D7.2 (A), R76.1
- new net: D9.2 (A), R78.1
