File: sac_board.kicad_pcb (KiCad board)
At the start: 4 copper layers, 120 x 80 mm, 279 parts, among them J1 12V_Input, J10 Conn_02x04_Odd_Even, J11 Conn_02x04_Odd_Even, J12 Micro_SD_Card_Det1, J2 RJ45_Hanrun_HR911105A_Horizon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, J3 USB_B_Mini, J4 Conn_02x16_Odd_Even, J5 DE9_Pins, J6 ARM JTAG/SWD, J7 Conn_01x08, J8 Conn_02x08_Odd_Even, J9 Conn_02x04_Odd_Even, U1 TPS563201, U10 TPS563201, U11 MAX3232, U12 STM32F407VETx, U13 DP83848C, U2 TPS563201, U3 TPS563201, U4 TPS563201, U5 TPS563201, U6 TPS563201, U7 TPS563201, U8 TPS563201, U9 TPS563201, Y1 8MHz, Y2 32.768KHz, Y3 25MHz

Commit message: update
Parts:
- removed D6: RED LED, LED_SMD:LED_0603_1608Metric
- removed R54, R58, R59, R69, R73, R75: 2.2K, Resistor_SMD:R_0603_1608Metric
- removed R55, R56, R57, R61, R64, R68, R70, R72: 33R, Resistor_SMD:R_0603_1608Metric
- removed R60: 1.5K, Resistor_SMD:R_0603_1608Metric
- removed R63, R67, R78, R79: 0R, Resistor_SMD:R_0603_1608Metric
- removed R76: 4.87K, Resistor_SMD:R_0603_1608Metric
- removed R77: DNI, Resistor_SMD:R_0603_1608Metric
- removed R89: 220, Resistor_SMD:R_0603_1608Metric
- removed U13: DP83848C, Package_QFP:LQFP-48_7x7mm_P0.5mm
- added C109: 10pF, Capacitor_SMD:C_0603_1608Metric, F.Cu at (68.9, 73.0)
- added C110: 10pF, Capacitor_SMD:C_0603_1608Metric, F.Cu at (68.9, 76.2)
- added C111: 10pF, Capacitor_SMD:C_0603_1608Metric, F.Cu at (68.9, 74.6)
- added C112: 0.1uF, Capacitor_SMD:C_0603_1608Metric, F.Cu at (85.0, 76.4)
- added C113: 0.1uF, Capacitor_SMD:C_0603_1608Metric, F.Cu at (85.0, 78.3)
- added U14: LAN8742A, Package_DFN_QFN:VQFN-24-1EP_4x4mm_P0.5mm_EP2.5x2.5mm, F.Cu at (79.0, 72.9)
- C100, C106: value 0.1uF -> 22nF
- C101, C96: value 33pF -> 22pF
- C107: value 0.1uF -> 10pF
- C99: value 10uF -> 0.1uF
- J12: value Micro_SD_Card_Det1 -> Micro_SD
- J2: value RJ45_Hanrun_HR911105A_Horizontal -> RJ45
- J4: value Conn_02x16_Odd_Even -> Conn_02x10_Odd_Even; footprint Connector_PinHeader_2.54mm:PinHeader_2x16_P2.54mm_Vertical -> Connector_PinHeader_2.54mm:PinHeader_2x10_P2.54mm_Vertical
- J5: value DE9_Pins -> UART
- J7: value Conn_01x08 -> Conn_02x08_Odd_Even; footprint Connector_PinHeader_2.54mm:PinHeader_1x08_P2.54mm_Vertical -> Connector_PinHeader_2.54mm:PinHeader_2x08_P2.54mm_Vertical
- R49, R50: value 470R -> 1K
- R51: value 33R -> 12.1K
- R52: value 33R -> 510
- R53: value 2.2K -> 1M
- R66, R71: value 2.2K -> 10K
- moved R38 132.0 mm to (93.8, 73.7), turned to 90 degrees
- moved R36 130.4 mm to (92.1, 73.7), turned to 90 degrees
- moved R37 130.3 mm to (95.5, 73.7), turned to 90 degrees
- moved R66 128.0 mm to (74.5, 81.1), turned to 180 degrees
- moved C99 125.9 mm to (85.0, 74.1), turned to 180 degrees
- moved R71 125.1 mm to (74.5, 79.5), turned to 180 degrees
- moved C107 120.8 mm to (68.9, 70.5), turned to 180 degrees
- moved SW5 115.8 mm to (85.3, 90.9), turned to -90 degrees
- moved C97 115.5 mm to (73.3, 70.5)
- moved R46 115.5 mm to (68.9, 83.7), turned to 0 degrees
- moved SW4 115.2 mm to (94.6, 90.9), turned to -90 degrees
- moved SW3 114.5 mm to (103.8, 90.9), turned to -90 degrees
- moved R47 114.2 mm to (68.9, 81.9), turned to 0 degrees
- moved C98 114.0 mm to (74.5, 77.2)
- moved R52 113.9 mm to (85.0, 70.9)
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- renumbered SW5 to SW2, SW4 to SW3, SW3 to SW4, SW2 to SW5
Connections:
- C100 pad 2: Net-(U13-PFBIN1) -> /mcu/+3.3V
- C101 pad 2: Net-(C101-Pad2) -> Net-(U14-XTAL2)
- C102 pad 2: /mcu/PD4 -> /mcu/PE10
- C103 pad 2: /mcu/PD5 -> /mcu/PD10
- C104 pad 2: /mcu/PD6 -> /mcu/PC7
- C105 pad 2: /mcu/PD7 -> /mcu/PA8
- C107 pad 2: /mcu/+3.3V -> /mcu/TD-P
- C96 pad 2: Net-(U13-X1) -> Net-(U14-XTAL1/CLKIN)
- C97 pad 2: Net-(U13-PFBIN1) -> /mcu/+3.3V
- C98 pad 2: Net-(U13-PFBIN1) -> /mcu/+3.3V
- C99 pad 2: Net-(U13-PFBIN1) -> /mcu/+3.3V
- J2 pad 10: /mcu/LEDACT -> Net-(J2-Pad10)
- J2 pad 11: /mcu/LEDLINK -> Net-(J2-Pad11)
- J2 pad 12: Net-(J2-Pad12) -> /mcu/LED-LINK
- J2 pad 9: Net-(J2-Pad9) -> /mcu/LED-SPEED
- J4 pad 1: /mcu/PB5 -> unconnected-(J4-Pin_1-Pad1)
- J4 pad 10: /mcu/PD12 -> unconnected-(J4-Pin_10-Pad10)
- J4 pad 11: /mcu/PD11 -> unconnected-(J4-Pin_11-Pad11)
- J4 pad 12: /mcu/PD10 -> unconnected-(J4-Pin_12-Pad12)
- J4 pad 13: /mcu/PD9 -> unconnected-(J4-Pin_13-Pad13)
- J4 pad 14: /mcu/PD8 -> unconnected-(J4-Pin_14-Pad14)
- J4 pad 15: /mcu/PB15 -> unconnected-(J4-Pin_15-Pad15)
- J4 pad 16: /mcu/PB14 -> unconnected-(J4-Pin_16-Pad16)
- J4 pad 17: /mcu/PE10 -> unconnected-(J4-Pin_17-Pad17)
- J4 pad 18: /mcu/PE11 -> unconnected-(J4-Pin_18-Pad18)
- J4 pad 19: /mcu/PE13 -> unconnected-(J4-Pin_19-Pad19)
- J4 pad 2: /mcu/PD0 -> unconnected-(J4-Pin_2-Pad2)
- J4 pad 20: /mcu/PE15 -> unconnected-(J4-Pin_20-Pad20)
- J4 pad 3: /mcu/PD1 -> unconnected-(J4-Pin_3-Pad3)
- J4 pad 4: /mcu/PA8 -> unconnected-(J4-Pin_4-Pad4)
- J4 pad 5: /mcu/PC7 -> unconnected-(J4-Pin_5-Pad5)
- J4 pad 6: /mcu/PC6 -> unconnected-(J4-Pin_6-Pad6)
- J4 pad 7: /mcu/PD15 -> unconnected-(J4-Pin_7-Pad7)
- J4 pad 8: /mcu/PD14 -> unconnected-(J4-Pin_8-Pad8)
- J4 pad 9: /mcu/PD13 -> unconnected-(J4-Pin_9-Pad9)
- J7 pad 1: /mcu/PE2 -> /mcu/PB5
- J7 pad 2: /mcu/PE3 -> /mcu/PD7
- J7 pad 3: /mcu/PE4 -> /mcu/PB7
- J7 pad 4: /mcu/PE5 -> /mcu/PB6
- J7 pad 5: /mcu/PE6 -> /mcu/PB9
- J7 pad 6: /mcu/PC13 -> /mcu/PB8
- J7 pad 7: /mcu/PC2 -> /mcu/PE1
- J7 pad 8: /mcu/PC3 -> /mcu/PE0
- J9 pad 1: /mcu/PA4 -> /mcu/PA0
- J9 pad 2: /mcu/PA5 -> /mcu/PA3
- J9 pad 3: /mcu/PA0 -> /mcu/PA4
- J9 pad 4: /mcu/PA3 -> /mcu/PA5
- J9 pad 6: /mcu/PE9 -> /mcu/PB0
- J9 pad 8: GND -> /mcu/PE7
- R49 pad 1: Net-(J2-Pad12) -> GND
- R49 pad 2: /mcu/+3.3V -> Net-(J2-Pad11)
- R50 pad 1: Net-(J2-Pad9) -> GND
- R50 pad 2: /mcu/+3.3V -> Net-(J2-Pad10)
- R51 pad 1: /mcu/PB12-RMII-TXD0 -> Net-(U14-RBIAS)
- R51 pad 2: Net-(U13-TXD_0) -> GND
- R52 pad 1: /mcu/PB13-RMII-TXD1 -> /mcu/PA2-ETH-MDIO
- R53 pad 1: GND -> Net-(U14-XTAL2)
- R53 pad 2: Net-(U13-TXD_2) -> Net-(U14-XTAL1/CLKIN)
- R66 pad 1: /mcu/LEDLINK -> /mcu/LED-LINK
- R66 pad 2: /mcu/+3.3V -> GND
- R71 pad 1: /mcu/LEDACT -> /mcu/LED-SPEED
- R71 pad 2: /mcu/+3.3V -> GND
- R80 pad 1: /mcu/PD4 -> /mcu/PE10
- R81 pad 1: /mcu/PD5 -> /mcu/PD10
- R82 pad 1: /mcu/PD6 -> /mcu/PC7
- R83 pad 1: /mcu/PD7 -> /mcu/PA8
- R84 pad 2: /mcu/PB6 -> /mcu/PD6
- R85 pad 2: /mcu/PB7 -> /mcu/PD5
- R86 pad 2: /mcu/PB8 -> /mcu/PD4
- R87 pad 2: /mcu/PB9 -> /mcu/PD0
- R88 pad 2: /mcu/PE0 -> /mcu/PD1
- SW2 pad 1: /mcu/PD7 -> /mcu/PA8
- SW3 pad 1: /mcu/PD6 -> /mcu/PC7
- SW4 pad 1: /mcu/PD5 -> /mcu/PD10
- SW5 pad 1: /mcu/PD4 -> /mcu/PE10
- Y3 pad 1: Net-(C101-Pad2) -> Net-(U14-XTAL2)
- Y3 pad 2: Net-(U13-X1) -> Net-(U14-XTAL1/CLKIN)
Routing:
- net /led_servo/V_M1: track 0.00 -> 194.1 mm
- net /led_servo/V_M2: track 0.00 -> 177.9 mm
- net GND: track 66.1 -> 242.6 mm, vias 53 -> 130
- net /led_servo/V_M3: track 0.00 -> 155.9 mm
- net /led_servo/V_M4: track 0.00 -> 114.5 mm
- net /mcu/+3.3V: track 25.0 -> 135.1 mm, vias 18 -> 34
- net +12V: track 693.5 -> 802.8 mm, vias 4 -> 10
- net /mcu/+5V: track 0.00 -> 74.9 mm
- net /mcu/PA12-USB-DP: track 0.00 -> 67.9 mm, vias 0 -> 2
- net /mcu/PA11-USB-DM: track 0.00 -> 63.9 mm, vias 0 -> 2
- net RESET: track 32.4 -> 81.7 mm, vias 2 -> 4
- net /mcu/PB1: track 0.00 -> 47.8 mm
- net /mcu/PE7: track 0.00 -> 47.0 mm
- net /mcu/LED-SPEED: track 0.00 -> 46.0 mm, vias 0 -> 1
- net /mcu/PB5: track 0.00 -> 45.7 mm
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Other:
- board text added: "PB6"
- board text added: "PB7"
- board text added: "PB8"
- board text added: "PB9"
- board text added: "PD7"
- board text added: "PE0"
- board text added: "PE1"
- board text removed: "PE12"
- board text removed: "PE14"
- board text removed: "PE8"
- board text removed: "PE9"

Commit message: update
Parts:
- removed D10, D11, D12, D13, D14, D15, D16, D9: GREEN LED, LED_SMD:LED_0603_1608Metric
- removed R92, R93, R94, R95, R96, R97, R98, R99: 680, Resistor_SMD:R_0603_1608Metric
- C112: value 0.1uF -> 10uF
- J12: value Micro_SD -> Micro_SD_Card_TF_01A; footprint Connector_Card:microSD_HC_Molex_104031-0811 -> Connector_Card:microSD_HC_Hirose_DM3AT-SF-PEJM5
- J5: footprint Connector_Dsub:DSUB-9_Pins_Horizontal_P2.77x2.84mm_EdgePinOffset4.94mm_Housed_MountingHolesOffset4.94mm -> Connector_Dsub:DSUB-9_Pins_Horizontal_P2.77x2.84mm_EdgePinOffset7.70mm_Housed_MountingHolesOffset9.12mm
- moved C105 60.7 mm to (58.2, 103.9)
- moved SW2 60.6 mm to (53.6, 103.1)
- moved R83 60.6 mm to (58.2, 100.0)
- moved C104 42.0 mm to (68.3, 103.9)
- moved SW3 41.9 mm to (63.7, 103.1)
- moved R82 41.9 mm to (68.3, 100.0)
- moved SW4 24.1 mm to (73.8, 103.1)
- moved C103 24.1 mm to (78.5, 103.9)
- moved R81 24.0 mm to (78.5, 100.1)
- moved R100 16.4 mm to (137.5, 92.2)
- moved R105 16.2 mm to (123.7, 92.2)
- moved R106 13.3 mm to (121.4, 92.2)
- moved C102 12.4 mm to (88.7, 103.9)
- moved SW5 12.2 mm to (84.0, 103.1)
- moved R80 12.2 mm to (88.7, 100.0)
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Connections:
- net /led_servo/V_M1 renamed /mcu/V_M1
- net /led_servo/V_M2 renamed /mcu/V_M2
- net /led_servo/V_M3 renamed /mcu/V_M3
- net /led_servo/V_M4 renamed /mcu/V_M4
- net /led_servo/V_M5 renamed /mcu/V_M5
- net /led_servo/V_M6 renamed /mcu/V_M6
- net /led_servo/V_M7 renamed /mcu/V_M7
- net /led_servo/V_M8 renamed /mcu/V_M8
- C102 pad 2: /mcu/PE10 -> /mcu/PE11
- C103 pad 2: /mcu/PD10 -> /mcu/PE10
- C104 pad 2: /mcu/PC7 -> /mcu/PE9
- C105 pad 2: /mcu/PA8 -> /mcu/PE8
- J4 pad 1: unconnected-(J4-Pin_1-Pad1) -> /mcu/PA8
- J4 pad 10: unconnected-(J4-Pin_10-Pad10) -> /mcu/PD9
- J4 pad 11: unconnected-(J4-Pin_11-Pad11) -> /mcu/PD8
- J4 pad 12: unconnected-(J4-Pin_12-Pad12) -> /mcu/PB15
- J4 pad 13: unconnected-(J4-Pin_13-Pad13) -> /mcu/PB14
- J4 pad 14: unconnected-(J4-Pin_14-Pad14) -> /mcu/PB10
- J4 pad 15: unconnected-(J4-Pin_15-Pad15) -> /mcu/PE15
- J4 pad 16: unconnected-(J4-Pin_16-Pad16) -> /mcu/PE14
- J4 pad 17: unconnected-(J4-Pin_17-Pad17) -> /mcu/PE13
- J4 pad 18: unconnected-(J4-Pin_18-Pad18) -> /mcu/PE12
- J4 pad 19: unconnected-(J4-Pin_19-Pad19) -> GND
- J4 pad 2: unconnected-(J4-Pin_2-Pad2) -> /mcu/PC7
- J4 pad 20: unconnected-(J4-Pin_20-Pad20) -> GND
- J4 pad 3: unconnected-(J4-Pin_3-Pad3) -> /mcu/PC6
- J4 pad 4: unconnected-(J4-Pin_4-Pad4) -> /mcu/PD15
- J4 pad 5: unconnected-(J4-Pin_5-Pad5) -> /mcu/PD14
- J4 pad 6: unconnected-(J4-Pin_6-Pad6) -> /mcu/PD13
- J4 pad 7: unconnected-(J4-Pin_7-Pad7) -> /mcu/PD12
- J4 pad 8: unconnected-(J4-Pin_8-Pad8) -> /mcu/PD11
- J4 pad 9: unconnected-(J4-Pin_9-Pad9) -> /mcu/PD10
- R80 pad 1: /mcu/PE10 -> /mcu/PE11
- R81 pad 1: /mcu/PD10 -> /mcu/PE10
- R82 pad 1: /mcu/PC7 -> /mcu/PE9
- R83 pad 1: /mcu/PA8 -> /mcu/PE8
- SW2 pad 1: /mcu/PA8 -> /mcu/PE8
- SW3 pad 1: /mcu/PC7 -> /mcu/PE9
- SW4 pad 1: /mcu/PD10 -> /mcu/PE10
- SW5 pad 1: /mcu/PE10 -> /mcu/PE11
- U12 pad 47: /mcu/PB10-RMII-RX-ER -> /mcu/PB10
Routing:
- net /mcu/PE8: track 34.8 -> 72.5 mm
- net /mcu/PB10: track 0.00 -> 31.2 mm
- net /mcu/PE9: track 34.1 -> 61.9 mm
- net /mcu/PC11-SDIO-D3: track 33.0 -> 56.7 mm, vias 4 -> 2
- net /mcu/PD2-SDIO-CMD: track 35.1 -> 58.2 mm, vias 4 -> 2
- net /mcu/PC10-SDIO-D2: track 32.6 -> 54.2 mm, vias 4 -> 2
- net /mcu/PE10: track 31.6 -> 51.3 mm
- net /mcu/PC8-SDIO-D0: track 52.4 -> 35.2 mm
- net /mcu/PE11: track 27.4 -> 43.9 mm
- net /mcu/PC9-SDIO-D1: track 48.6 -> 33.5 mm, vias 0 -> 2
- net /mcu/PD3-Card-CD: track 42.8 -> 31.1 mm, vias 4 -> 2
- net /mcu/PD15: track 17.4 -> 28.2 mm
- net /mcu/PD13: track 17.4 -> 27.4 mm
- net /mcu/PE14: track 22.9 -> 32.6 mm
- net /mcu/PC7: track 20.4 -> 28.6 mm
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Other:
- board text added: "PB10"
- board text added: "PE12"
- board text added: "PE14"
- board text added: "SAC MODULE V1.0.0 Produced by Lazycat Design"
- board text removed: "PD0"
- board text removed: "PD1"
- board text removed: "PE10"
- board text removed: "PE11"
- board text removed: "SAC BOARD V1.0.0 Produced by Lazycat Design"

Commit message: update
Parts:
- H1, H2, H3, H4: footprint MountingHole:MountingHole_2.2mm_M2 -> MountingHole:MountingHole_2.5mm
- moved R53 6.59 mm to (81.6, 81.1)
- moved C96 6.38 mm to (85.0, 82.9), turned to 180 degrees
- moved Y3 5.33 mm to (80.0, 84.3)
- moved C101 4.81 mm to (74.5, 83.0), turned to 0 degrees
- moved R74 3.85 mm to (74.4, 67.6), turned to 180 degrees
- moved C97 1.10 mm to (74.4, 70.6)
- moved C91 0.81 mm to (99.6, 81.0)
- moved C92 0.25 mm to (117.0, 80.0)
- moved R66 0.10 mm to (74.5, 81.2)
Routing:
- net /mcu/PA13-JTMS: track 70.1 -> 65.3 mm
- net Net-(U14-XTAL2): track 17.7 -> 14.7 mm
- net /mcu/PA9-USART1-TX: track 28.9 -> 25.9 mm, vias 2 -> 0
- net Net-(U14-XTAL1/CLKIN): track 16.8 -> 14.2 mm
- net /mcu/PB11-RMII-TXEN: track 36.2 -> 34.3 mm
- net /mcu/PA10-USART1-RX: track 27.2 -> 25.6 mm, vias 2 -> 0
- net GND: track 239.4 -> 240.6 mm, vias 141 -> 139
- net /mcu/LED-LINK: track 42.1 -> 43.1 mm
- net /mcu/PC0-ETH-RESET: track 40.0 -> 41.0 mm
- net Net-(U12-VCAP_1): track 6.07 -> 5.24 mm
- net Net-(U12-VCAP_2): track 7.16 -> 6.42 mm
- net /mcu/PB12-RMII-TXD0: track 35.2 -> 34.5 mm
- net /mcu/+3.3V: track 135.9 -> 135.3 mm
- net /mcu/PE6: track 27.8 -> 28.4 mm
- net /mcu/PA0: track 36.0 -> 36.5 mm

Commit message: update
Parts:
- U11: footprint Package_SO:SOIC-16W_5.3x10.2mm_P1.27mm -> Package_SO:SOIC-16_4.55x10.3mm_P1.27mm
- moved C101 6.58 mm to (80.5, 85.7)
- moved C96 3.05 mm to (83.8, 85.7), turned to 0 degrees
- moved Y3 2.70 mm to (82.1, 82.6)
- moved R53 1.94 mm to (80.5, 79.5)
- moved C97 1.92 mm to (73.2, 69.1), turned to 90 degrees
- moved R74 1.70 mm to (75.2, 69.1), turned to -90 degrees
- moved BT1 0.19 mm to (131.2, 65.3)
Routing:
- net /mcu/+3.3V: track 135.3 -> 153.3 mm, vias 33 -> 28
- net GND: track 240.6 -> 246.8 mm
- net Net-(U14-XTAL2): track 14.7 -> 11.7 mm
- net /mcu/PD7: track 44.6 -> 47.6 mm
- net Net-(BT1-+): track 26.3 -> 25.3 mm
- net Net-(U14-XTAL1/CLKIN): track 14.2 -> 13.2 mm
- net /mcu/PD1: vias 4 -> 2
- net /mcu/PD0: vias 4 -> 2

Commit message: update
Parts:
- removed the C102 at (88.7, 103.9)
- removed the C68 at (66.5, 50.5)
- removed the C72 at (75.4, 60.2)
- removed the C73 at (72.3, 60.1)
- removed the C79 at (66.0, 60.1)
- removed the C80 at (63.0, 60.1)
- removed the D4 at (145.2, 69.7)
- removed the D5 at (145.2, 71.6)
- removed J12: Micro_SD_Card_TF_01A, Connector_Card:microSD_HC_Hirose_DM3AT-SF-PEJM5
- removed the J7 at (135.4, 38.0)
- removed the J9 at (86.8, 38.0)
- removed the R2 at (91.8, 61.3)
- removed the R26 at (62.1, 53.6)
- removed R80: 10K, Resistor_SMD:R_0603_1608Metric
- removed R87, R88: 220, Resistor_SMD:R_0603_1608Metric
- removed SW5: ~, Button_Switch_SMD:SW_Push_1P1T_NO_CK_KSC7xxJ
- added C54: 0.1uF, Capacitor_SMD:C_0603_1608Metric, B.Cu at (65.0, 55.2)
- added C58: 10uF, Capacitor_SMD:C_0603_1608Metric, B.Cu at (63.0, 55.2)
- added C62: 10uF, Capacitor_SMD:C_0603_1608Metric, B.Cu at (61.0, 55.2)
- added C66: 0.1uF, Capacitor_SMD:C_0603_1608Metric, B.Cu at (62.1, 46.2)
- added C70: 22uF, Capacitor_SMD:C_0603_1608Metric, B.Cu at (74.2, 55.1)
- added J10: Conn_02x12_Odd_Even, Connector_PinHeader_2.54mm:PinHeader_2x12_P2.54mm_Vertical, F.Cu at (135.8, 38.0)
- added J3: Micro_SD_Card_Det1, Connector_Card:microSD_HC_Hirose_DM3AT-SF-PEJM5, F.Cu at (133.5, 103.5)
- added R24: 10K, Resistor_SMD:R_0603_1608Metric, B.Cu at (58.8, 45.8)
- added R3: 33K, Resistor_SMD:R_0603_1608Metric, F.Cu at (92.9, 64.4)
- C10: renamed from C12; footprint Capacitor_SMD:C_1206_3216Metric -> Capacitor_SMD:C_0603_1608Metric
- C11: renamed from C3; footprint Capacitor_SMD:C_1206_3216Metric -> Capacitor_SMD:C_0603_1608Metric
- C12: renamed from C13; footprint Capacitor_SMD:C_1206_3216Metric -> Capacitor_SMD:C_0603_1608Metric
- C13: renamed from C4; footprint Capacitor_SMD:C_1206_3216Metric -> Capacitor_SMD:C_0603_1608Metric
- C14: footprint Capacitor_SMD:C_1206_3216Metric -> Capacitor_SMD:C_0603_1608Metric
- C23: renamed from C38; footprint Capacitor_SMD:C_1206_3216Metric -> Capacitor_SMD:C_0603_1608Metric
- C24: renamed from C32; footprint Capacitor_SMD:C_1206_3216Metric -> Capacitor_SMD:C_0603_1608Metric
- C25: renamed from C59; footprint Capacitor_SMD:C_1206_3216Metric -> Capacitor_SMD:C_0603_1608Metric
- C26: renamed from C76; footprint Capacitor_SMD:C_1206_3216Metric -> Capacitor_SMD:C_0603_1608Metric
- C27: renamed from C39; footprint Capacitor_SMD:C_1206_3216Metric -> Capacitor_SMD:C_0603_1608Metric
- C28: renamed from C33; footprint Capacitor_SMD:C_1206_3216Metric -> Capacitor_SMD:C_0603_1608Metric
- C29: renamed from C60; footprint Capacitor_SMD:C_1206_3216Metric -> Capacitor_SMD:C_0603_1608Metric
- C3: renamed from C6; footprint Capacitor_SMD:C_1206_3216Metric -> Capacitor_SMD:C_0603_1608Metric
- C30: renamed from C77; footprint Capacitor_SMD:C_1206_3216Metric -> Capacitor_SMD:C_0603_1608Metric
- C35: renamed from C28; footprint Capacitor_SMD:C_1206_3216Metric -> Capacitor_SMD:C_0603_1608Metric
- C36: renamed from C22; footprint Capacitor_SMD:C_1206_3216Metric -> Capacitor_SMD:C_0603_1608Metric
- C37: renamed from C49; footprint Capacitor_SMD:C_1206_3216Metric -> Capacitor_SMD:C_0603_1608Metric
- C38: renamed from C69; footprint Capacitor_SMD:C_1206_3216Metric -> Capacitor_SMD:C_0603_1608Metric
- C39: renamed from C29; footprint Capacitor_SMD:C_1206_3216Metric -> Capacitor_SMD:C_0603_1608Metric
- C4: renamed from C16; footprint Capacitor_SMD:C_1206_3216Metric -> Capacitor_SMD:C_0603_1608Metric
- C40: renamed from C23; footprint Capacitor_SMD:C_1206_3216Metric -> Capacitor_SMD:C_0603_1608Metric
- C41: renamed from C50; footprint Capacitor_SMD:C_1206_3216Metric -> Capacitor_SMD:C_0603_1608Metric
- C42: renamed from C70; footprint Capacitor_SMD:C_1206_3216Metric -> Capacitor_SMD:C_0603_1608Metric
- C43: renamed from C30; footprint Capacitor_SMD:C_1206_3216Metric -> Capacitor_SMD:C_0603_1608Metric
- C44: renamed from C24; footprint Capacitor_SMD:C_1206_3216Metric -> Capacitor_SMD:C_0603_1608Metric
- C45: renamed from C51; footprint Capacitor_SMD:C_1206_3216Metric -> Capacitor_SMD:C_0603_1608Metric
- C46: renamed from C71; footprint Capacitor_SMD:C_1206_3216Metric -> Capacitor_SMD:C_0603_1608Metric
- C5: renamed from C7; footprint Capacitor_SMD:C_1206_3216Metric -> Capacitor_SMD:C_0603_1608Metric
- C55: renamed from C62; footprint Capacitor_SMD:C_1206_3216Metric -> Capacitor_SMD:C_0603_1608Metric
- C56: renamed from C35; footprint Capacitor_SMD:C_1206_3216Metric -> Capacitor_SMD:C_0603_1608Metric
- C57: renamed from C56; footprint Capacitor_SMD:C_1206_3216Metric -> Capacitor_SMD:C_0603_1608Metric
- C59: renamed from C63; footprint Capacitor_SMD:C_1206_3216Metric -> Capacitor_SMD:C_0603_1608Metric
- C6: renamed from C17; footprint Capacitor_SMD:C_1206_3216Metric -> Capacitor_SMD:C_0603_1608Metric
- C60: renamed from C36; footprint Capacitor_SMD:C_1206_3216Metric -> Capacitor_SMD:C_0603_1608Metric
- C61: renamed from C57; footprint Capacitor_SMD:C_1206_3216Metric -> Capacitor_SMD:C_0603_1608Metric
- C67: renamed from C52; footprint Capacitor_SMD:C_1206_3216Metric -> Capacitor_SMD:C_0603_1608Metric
- C68: renamed from C25; footprint Capacitor_SMD:C_1206_3216Metric -> Capacitor_SMD:C_0603_1608Metric
- C69: renamed from C46; footprint Capacitor_SMD:C_1206_3216Metric -> Capacitor_SMD:C_0603_1608Metric
- C71: renamed from C53; footprint Capacitor_SMD:C_1206_3216Metric -> Capacitor_SMD:C_0603_1608Metric
- C72: renamed from C26; footprint Capacitor_SMD:C_1206_3216Metric -> Capacitor_SMD:C_0603_1608Metric
- C73: renamed from C47; footprint Capacitor_SMD:C_1206_3216Metric -> Capacitor_SMD:C_0603_1608Metric
- C74: value 10uF -> 22uF; footprint Capacitor_SMD:C_1206_3216Metric -> Capacitor_SMD:C_0603_1608Metric
- C75: renamed from C54; footprint Capacitor_SMD:C_1206_3216Metric -> Capacitor_SMD:C_0603_1608Metric
- C76: renamed from C27; footprint Capacitor_SMD:C_1206_3216Metric -> Capacitor_SMD:C_0603_1608Metric
- C77: renamed from C48; footprint Capacitor_SMD:C_1206_3216Metric -> Capacitor_SMD:C_0603_1608Metric
- C78: value 0.1uF -> 10uF
- C9: renamed from C2; footprint Capacitor_SMD:C_1206_3216Metric -> Capacitor_SMD:C_0603_1608Metric
- J5: value UART -> DE9_Socket; footprint Connector_Dsub:DSUB-9_Pins_Horizontal_P2.77x2.84mm_EdgePinOffset7.70mm_Housed_MountingHolesOffset9.12mm -> Custom:DSUB-9_Pins_Horizontal_P2.77x2.84mm_EdgePinOffset7.70mm_Housed_MountingHolesOffset9.12mm_Female
- moved J2 72.0 mm to (116.2, 105.7), turned to 0 degrees
- moved R36 63.1 mm to (117.2, 98.3), turned to -90 degrees
- moved R37 61.5 mm to (115.5, 98.3), turned to -90 degrees
- moved BT1 54.7 mm to (185.8, 64.0), turned to 180 degrees
- moved D5 41.2 mm to (186.0, 74.0)
- moved D4 41.2 mm to (186.0, 72.0)
- moved D3 41.2 mm to (186.0, 70.0)
- moved R70 41.0 mm to (182.6, 74.0)
- moved R69 41.0 mm to (182.6, 72.0)
- moved R62 40.9 mm to (182.6, 70.0)
- moved R33 16.3 mm to (122.4, 76.2), turned to 0 degrees
- moved R34 16.3 mm to (122.4, 74.4), turned to 0 degrees
- moved R39 16.3 mm to (122.4, 72.7)
- moved C86 14.7 mm to (114.4, 53.0)
- moved J6 14.4 mm to (97.0, 38.1)
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- renumbered C5 to C1, C113 to C100, C97 to C101, C98 to C102, C107 to C103, C109 to C104, C110 to C105, C103 to C106, C111 to C107, C100 to C108, C106 to C109, C104 to C110, C95 to C111, C105 to C112, C8 to C15, C18 to C16, C9 to C17, C10 to C18, C37 to C19, C15 to C2, C31 to C20, C58 to C21, C75 to C22, C21 to C31, C19 to C32, C44 to C33, C67 to C34, C42 to C47, C40 to C48, C65 to C49, C81 to C50, C61 to C51, C34 to C52, C55 to C53, C45 to C63, C20 to C64, C43 to C65, C1 to C7, C66 to C79, C11 to C8, C41 to C80, C64 to C81, C89 to C83, C90 to C84, C108 to C85, C84 to C86, C91 to C87, C92 to C88, C93 to C89, C94 to C90, C85 to C91, C96 to C92, C101 to C93, C99 to C94, C83 to C95, C112 to C96, C86 to C97, C87 to C98, C88 to C99, D7 to D1, D8 to D2, D1 to D3, D2 to D4, D3 to D5, J10 to J11, J3 to J2, J6 to J4, J8 to J6, J11 to J7, J4 to J8, J2 to J9, L7 to L10, L3 to L2, L2 to L3, L6 to L4, L4 to L5, L8 to L6, L10 to L7, L9 to L8, L5 to L9, R7 to R10, R17 to R11, R25 to R12, R12 to R13, R15 to R14, R10 to R15, R13 to R16, R20 to R17, R23 to R18, R27 to R19, R4 to R2, R29 to R20, R18 to R21, R8 to R22, R16 to R23, R21 to R25, R24 to R26, R11 to R27, R14 to R28, R19 to R29, R22 to R30, R28 to R31, R30 to R32, R32 to R33, R33 to R34, R62 to R36, R65 to R37, R31 to R38, R34 to R39, R3 to R4, R106 to R40, R105 to R41, R104 to R42, R103 to R43, R102 to R44, R101 to R45, R100 to R46, R44 to R47, R37 to R48, R36 to R49, R38 to R50, R74 to R51, R39 to R54, R43 to R55, R40 to R56, R41 to R57, R42 to R58, R51 to R59, R66 to R60, R71 to R61, R84 to R62, R81 to R63, R45 to R64, R46 to R65, R47 to R66, R48 to R67, R82 to R68, R85 to R69, R90 to R7, R86 to R70, R83 to R71, R50 to R72, R49 to R73, R91 to R8, SW4 to SW2, SW2 to SW4, U12 to U11, U11 to U12, U14 to U13, U5 to U3, U3 to U4, U7 to U5, U9 to U6, U8 to U7, U4 to U8, U6 to U9
Connections:
- C78 pad 1: +12V -> /mcu/V_M8
- J5 pad 5: unconnected-(J5-Pad5) -> GND
Routing:
- net GND: track 246.8 -> 54.9 mm, vias 139 -> 13
- net +12V: track 802.8 -> 633.0 mm, vias 10 -> 17
- net /mcu/PE8: track 72.5 -> 0.00 mm
- net RESET: track 81.8 -> 16.8 mm, vias 4 -> 0
- net /mcu/PE9: track 61.9 -> 0.00 mm
- net /mcu/PD2-SDIO-CMD: track 58.2 -> 0.00 mm, vias 2 -> 0
- net /mcu/PC11-SDIO-D3: track 56.5 -> 0.00 mm, vias 2 -> 0
- net /mcu/PA12-USB-DP: track 67.9 -> 12.4 mm, vias 2 -> 0
- net /mcu/PC10-SDIO-D2: track 54.2 -> 0.00 mm, vias 2 -> 0
- net /mcu/PA11-USB-DM: track 63.9 -> 11.1 mm, vias 2 -> 0
- net /mcu/PE10: track 51.3 -> 0.00 mm
- net /mcu/PB1: track 47.8 -> 0.00 mm
- net /mcu/PD7: track 47.6 -> 0.00 mm, vias 2 -> 0
- net /mcu/LED-SPEED: track 46.0 -> 0.00 mm, vias 1 -> 0
- net /mcu/PB5: track 45.1 -> 0.00 mm
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- added copper zone on B.Cu, net GND
- removed copper zone on In2.Cu, net /mcu/+3.3V
- removed copper zone on In1.Cu, net GND
Other:
- copper layers 4 -> 2
- board text removed: "PA0"
- board text removed: "PA3"
- board text removed: "PA4"
- board text removed: "PA5"
- board text removed: "PA6"
- board text removed: "PB0"
- board text removed: "PB1"
- board text removed: "PE7"
