File: sac_board.kicad_pcb (KiCad board)
At the start: 2 copper layers, 120 x 80 mm, 237 parts, among them J1 12V_Input, J10 Conn_02x12_Odd_Even, J11 Conn_02x04_Odd_Even, J2 USB_B_Mini, J3 Micro_SD_Card_Det1, J4 ARM JTAG/SWD, J5 DE9_Socket, J6 Conn_02x08_Odd_Even, J7 Conn_02x04_Odd_Even, J8 Conn_02x10_Odd_Even, J9 RJ45, U1 TPS563201, U10 TPS563201, U11 STM32F407VETx, U12 MAX3232, U13 LAN8742A, U2 TPS563201, U3 TPS563201, U4 TPS563201, U5 TPS563201, U6 TPS563201, U7 TPS563201, U8 TPS563201, U9 TPS563201, Y1 8MHz, Y2 32.768KHz, Y3 25MHz

Commit message: update
Parts:
- added C113: 0.1uF, Capacitor_SMD:C_0603_1608Metric, F.Cu at (65.7, 103.8)
- added D10: WHITE LED, LED_SMD:LED_0603_1608Metric, F.Cu at (91.5, 47.7)
- added D11: WHITE LED, LED_SMD:LED_0603_1608Metric, F.Cu at (89.0, 47.7)
- added D12: WHITE LED, LED_SMD:LED_0603_1608Metric, F.Cu at (86.5, 47.7)
- added D13: WHITE LED, LED_SMD:LED_0603_1608Metric, F.Cu at (83.9, 47.7)
- added D14: WHITE LED, LED_SMD:LED_0603_1608Metric, F.Cu at (81.4, 47.7)
- added D6: ORANGE LED, LED_SMD:LED_0603_1608Metric, F.Cu at (142.0, 65.0)
- added D7: WHITE LED, LED_SMD:LED_0603_1608Metric, F.Cu at (99.2, 47.7)
- added D8: WHITE LED, LED_SMD:LED_0603_1608Metric, F.Cu at (96.7, 47.7)
- added D9: WHITE LED, LED_SMD:LED_0603_1608Metric, F.Cu at (94.1, 47.7)
- added R74: 220, Resistor_SMD:R_0603_1608Metric, F.Cu at (138.5, 65.0)
- added R75: 10K, Resistor_SMD:R_0603_1608Metric, F.Cu at (65.7, 99.8)
- added R76: 220, Resistor_SMD:R_0603_1608Metric, F.Cu at (99.2, 44.4)
- added R77: 220, Resistor_SMD:R_0603_1608Metric, F.Cu at (96.7, 44.4)
- added R78: 220, Resistor_SMD:R_0603_1608Metric, F.Cu at (94.1, 44.4)
- added R79: 220, Resistor_SMD:R_0603_1608Metric, F.Cu at (91.6, 44.4)
- added R80: 220, Resistor_SMD:R_0603_1608Metric, F.Cu at (89.0, 44.4)
- added R81: 220, Resistor_SMD:R_0603_1608Metric, F.Cu at (86.5, 44.4)
- added R82: 220, Resistor_SMD:R_0603_1608Metric, F.Cu at (83.9, 44.4)
- added R83: 220, Resistor_SMD:R_0603_1608Metric, F.Cu at (81.4, 44.4)
- added SW5: ~, Button_Switch_SMD:SW_Push_1P1T_NO_CK_KSC7xxJ, F.Cu at (60.9, 102.9)
- J10: value Conn_02x12_Odd_Even -> Conn_02x09_Odd_Even; footprint Connector_PinHeader_2.54mm:PinHeader_2x12_P2.54mm_Vertical -> Connector_PinHeader_2.54mm:PinHeader_2x09_P2.54mm_Vertical
- J8: value Conn_02x10_Odd_Even -> Conn_02x14_Odd_Even; footprint Connector_PinHeader_2.54mm:PinHeader_2x10_P2.54mm_Vertical -> Connector_PinHeader_2.54mm:PinHeader_2x14_P2.54mm_Vertical
- moved BT1 54.6 mm to (131.3, 62.3), turned to 0 degrees
- moved R70 44.6 mm to (138.5, 67.0)
- moved D5 44.5 mm to (142.0, 67.0)
- moved R69 44.2 mm to (138.5, 69.0)
- moved R62 44.1 mm to (138.5, 71.0)
- moved D4 44.1 mm to (142.0, 69.0)
- moved D3 44.0 mm to (142.0, 71.0)
- moved C106 27.6 mm to (53.9, 90.8)
- moved R63 27.6 mm to (53.9, 87.0), turned to 90 degrees
- moved SW2 27.6 mm to (49.2, 90.0)
- moved C108 20.2 mm to (64.0, 76.1), turned to 90 degrees
- moved R51 19.1 mm to (93.8, 70.6), turned to 0 degrees
- moved C36 17.7 mm to (56.0, 105.6), turned to 180 degrees
- moved C40 15.6 mm to (56.0, 103.6), turned to 180 degrees
- moved R61 14.9 mm to (71.2, 68.5), turned to 0 degrees
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Connections:
- C106 pad 2: /mcu/PE10 -> /mcu/PA4
- C110 pad 2: /mcu/PE9 -> /mcu/PA3
- C112 pad 2: /mcu/PE8 -> /mcu/PA5
- J10 pad 1: /mcu/PA0 -> /mcu/PD6
- J10 pad 10: /mcu/PD7 -> /mcu/PE2
- J10 pad 11: /mcu/PB7 -> /mcu/PE3
- J10 pad 12: /mcu/PB6 -> /mcu/PE4
- J10 pad 13: /mcu/PB9 -> /mcu/PE5
- J10 pad 14: /mcu/PB8 -> /mcu/PE6
- J10 pad 15: /mcu/PE1 -> /mcu/PC13
- J10 pad 16: /mcu/PE0 -> /mcu/PC2
- J10 pad 17: /mcu/PE3 -> /mcu/PC3
- J10 pad 18: /mcu/PE2 -> /mcu/PA0
- J10 pad 2: /mcu/PA3 -> /mcu/PD7
- J10 pad 3: /mcu/PA4 -> /mcu/PB5
- J10 pad 4: /mcu/PA5 -> /mcu/PB6
- J10 pad 5: /mcu/PA6 -> /mcu/PB7
- J10 pad 6: /mcu/PB0 -> /mcu/PB8
- J10 pad 7: /mcu/PB1 -> /mcu/PB9
- J10 pad 8: /mcu/PE7 -> /mcu/PE0
- J10 pad 9: /mcu/PB5 -> /mcu/PE1
- J8 pad 1: /mcu/PA8 -> /mcu/PC7
- J8 pad 10: /mcu/PD9 -> /mcu/PD10
- J8 pad 11: /mcu/PD8 -> /mcu/PB15
- J8 pad 12: /mcu/PB15 -> /mcu/PD8
- J8 pad 13: /mcu/PB14 -> /mcu/PB10
- J8 pad 14: /mcu/PB10 -> /mcu/PB14
- J8 pad 15: /mcu/PE15 -> /mcu/PE14
- J8 pad 16: /mcu/PE14 -> /mcu/PE15
- J8 pad 17: /mcu/PE13 -> /mcu/PE12
- J8 pad 18: /mcu/PE12 -> /mcu/PE13
- J8 pad 19: GND -> /mcu/PE10
- J8 pad 2: /mcu/PC7 -> /mcu/PA8
- J8 pad 20: GND -> /mcu/PE11
- J8 pad 3: /mcu/PC6 -> /mcu/PD15
- J8 pad 4: /mcu/PD15 -> /mcu/PC6
- J8 pad 5: /mcu/PD14 -> /mcu/PD13
- J8 pad 6: /mcu/PD13 -> /mcu/PD14
- J8 pad 7: /mcu/PD12 -> /mcu/PD11
- J8 pad 8: /mcu/PD11 -> /mcu/PD12
- J8 pad 9: /mcu/PD10 -> /mcu/PD9
- R62 pad 2: /mcu/PD6 -> /mcu/PD0
- R63 pad 1: /mcu/PE10 -> /mcu/PA4
- R68 pad 1: /mcu/PE9 -> /mcu/PA3
- R69 pad 2: /mcu/PD5 -> /mcu/PD1
- R71 pad 1: /mcu/PE8 -> /mcu/PA5
- SW2 pad 1: /mcu/PE10 -> /mcu/PA4
- SW3 pad 1: /mcu/PE9 -> /mcu/PA3
- SW4 pad 1: /mcu/PE8 -> /mcu/PA5
Routing:
- net /mcu/+3.3V: track 162.2 -> 487.6 mm, vias 6 -> 31
- net GND: track 54.9 -> 202.9 mm, vias 13 -> 66
- net RESET: track 16.8 -> 96.1 mm, vias 0 -> 2
- net /mcu/PD6: track 0.00 -> 54.8 mm, vias 0 -> 2
- net /mcu/PA4: track 15.5 -> 70.0 mm, vias 3 -> 0
- net /mcu/PA5: track 17.9 -> 69.8 mm, vias 3 -> 0
- net /mcu/PD7: track 0.00 -> 51.1 mm, vias 0 -> 2
- net /mcu/PB5: track 0.00 -> 49.5 mm
- net /mcu/PB7: track 0.00 -> 48.9 mm
- net /mcu/PB9: track 0.00 -> 48.0 mm
- net /mcu/LED-LINK: track 0.00 -> 46.2 mm
- net /mcu/PB6: track 0.00 -> 46.1 mm
- net /mcu/PE1: track 0.00 -> 45.8 mm, vias 0 -> 2
- net /mcu/LED-SPEED: track 0.00 -> 45.7 mm, vias 0 -> 2
- net /mcu/PB8: track 0.00 -> 45.2 mm
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- added copper zone on F.Cu, net GND
Other:
- board text added: "PA0"
- board text added: "PB0"
- board text added: "PB1"
- board text added: "PD6"
- board text added: "PE10"
- board text added: "PE11"
- board text added: "PE7"
- board text added: "PE8"
- board text added: "PE9"
- board text added: "SAC MODULE V1.0.1 Produced by Lazycat Design"
- board text removed: "SAC MODULE V1.0.0 Produced by Lazycat Design"
