File: sac_board.kicad_pcb (KiCad board)
At the start: 2 copper layers, 120 x 80 mm, 258 parts, among them J1 12V_Input, J10 Conn_02x09_Odd_Even, J11 Conn_02x04_Odd_Even, J2 USB_B_Mini, J3 Micro_SD_Card_Det1, J4 ARM JTAG/SWD, J5 DE9_Socket, J6 Conn_02x08_Odd_Even, J7 Conn_02x04_Odd_Even, J8 Conn_02x14_Odd_Even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

Commit message: update
Parts:
- H1, H2, H3, H4: footprint MountingHole:MountingHole_2.5mm -> MountingHole:MountingHole_2.7mm_M2.5
- moved J10 1.84 mm to (126.1, 38.3)
- moved J5 0.50 mm to (147.8, 94.8)
- moved H3 0.45 mm to (43.0, 108.7)
- moved H4 0.35 mm to (155.1, 108.8)
- moved H1 0.30 mm to (155.1, 35.4)
- moved H2 0.27 mm to (42.9, 35.5)
- moved J4 0.16 mm to (152.4, 44.4)
Routing:
- net /mcu/PC2: track 36.3 -> 39.0 mm
- net /mcu/PC3: track 39.8 -> 42.4 mm
- net /mcu/PC13: track 47.2 -> 49.8 mm
- net /mcu/PA0: track 39.1 -> 41.6 mm
- net /mcu/PE6: track 43.4 -> 45.8 mm
- net /mcu/PE5: track 46.2 -> 48.3 mm
- net /mcu/PA5: track 70.8 -> 69.5 mm
- net /mcu/PA6: track 58.7 -> 57.5 mm
- net /mcu/PA4: track 75.9 -> 74.8 mm
- net /mcu/PA3: track 55.4 -> 54.3 mm
- net /mcu/PE4: track 44.3 -> 45.1 mm
- net /mcu/PD7: track 51.1 -> 51.9 mm
- net /mcu/PB6: track 46.1 -> 46.9 mm
- net /mcu/PB5: track 49.5 -> 50.3 mm
- net /mcu/PE1: track 46.6 -> 47.3 mm
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
Commit message: update
Parts:
- C6: footprint Resistor_SMD:R_0805_2012Metric -> Capacitor_SMD:C_0805_2012Metric
Changed lines of the file:
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@@
 		)
 	)
-	(footprint "Resistor_SMD:R_0805_2012Metric"
+	(footprint "Capacitor_SMD:C_0805_2012Metric"
 		(layer "F.Cu")
 		(at 70.8 53.695 90)
-		(descr "Resistor SMD 0805 (2012 Metric), square (rectangular) end terminal, IPC-7351 nominal, (Body size source: IPC-SM-782 page 72, https://www.pcb-3d.com/wordpress/wp-content/uploads/ipc-sm-782a_amendment_1_and_2.pdf), generated with kicad-footprint-generator")
-		(tags "resistor")
+		(descr "Capacitor SMD 0805 (2012 Metric), square (rectangular) end terminal, IPC-7351 nominal, (Body size source: IPC-SM-782 page 76, https://www.pcb-3d.com/wordpress/wp-content/uploads/ipc-sm-782a_amendment_1_and_2.pdf, https://docs.google.com/spreadsheets/d/1BsfQQcO9C6DZCsRaXUlFlo91Tg2WpOkGARC1WS5S8t0/edit?usp=sharing), generated with kicad-footprint-generator")
+		(tags "capacitor")
 		(property "Reference" "C6"
-			(at 2.75 -0.095 90)
+			(at 2.795 0.1 90)
 			(layer "F.SilkS")
 			(effects
@@
 		)
 		(property "Value" "10uF"
-			(at 0 1.65 90)
+			(at 0 1.68 90)
 			(layer "F.Fab")
 			(effects
@@
 		(attr smd)
 		(fp_line
-			(start -0.227064 -0.735)
-			(end 0.227064 -0.735)
+			(start -0.261252 -0.735)
+			(end 0.261252 -0.735)
 			(stroke
 				(width 0.12)
@@
 		)
 		(fp_line
-			(start -0.227064 0.735)
-			(end 0.227064 0.735)
+			(start -0.261252 0.735)
+			(end 0.261252 0.735)
 			(stroke
 				(width 0.12)
@@
 		)
 		(fp_line
-			(start 1.68 -0.95)
-			(end 1.68 0.95)
+			(start 1.7 -0.98)
+			(end 1.7 0.98)
 			(stroke
 				(width 0.05)
@@
 		)
 		(fp_line
-			(start -1.68 -0.95)
-			(end 1.68 -0.95)
+			(start -1.7 -0.98)
+			(end 1.7 -0.98)
 			(stroke
 				(width 0.05)
@@
 		)
 		(fp_line
-			(start 1.68 0.95)
-			(end -1.68 0.95)
+			(start 1.7 0.98)
+			(end -1.7 0.98)
 			(stroke
 				(width 0.05)
@@
 		)
 		(fp_line
-			(start -1.68 0.95)
-			(end -1.68 -0.95)
+			(start -1.7 0.98)
+			(end -1.7 -0.98)
 			(stroke
 				(width 0.05)
@@
 		)
 		(pad "1" smd roundrect
-			(at -0.9125 0 90)
-			(size 1.025 1.4)
+			(at -0.95 0 90)
+			(size 1 1.45)
 			(layers "F.Cu" "F.Mask" "F.Paste")
-			(roundrect_rratio 0.243902)
+			(roundrect_rratio 0.25)
 			(net 5 "+12V")
 			(pintype "passive")
 		)
 		(pad "2" smd roundrect
-			(at 0.9125 0 90)
-			(size 1.025 1.4)
+			(at 0.95 0 90)
+			(size 1 1.45)
 			(layers "F.Cu" "F.Mask" "F.Paste")
-			(roundrect_rratio 0.243902)
+			(roundrect_rratio 0.25)
 			(net 1 "GND")
 			(pintype "passive")
 		)
 		(embedded_fonts no)
-		(model "${KICAD9_3DMODEL_DIR}/Resistor_SMD.3dshapes/R_0805_2012Metric.step"
+		(model "${KICAD9_3DMODEL_DIR}/Capacitor_SMD.3dshapes/C_0805_2012Metric.step"
 			(offset
 				(xyz 0 0 0)

Commit message: update
Parts:
- D1, D2: value GREEN LED -> LED
- D10, D11, D12, D13, D14, D3, D4, D7, D8, D9: value WHITE LED -> LED
- D5, D6: value ORANGE LED -> LED
- turned SW1 to 180 degrees

Commit message: update
Parts:
- D1, D2: value LED -> GREEN LED
- D10, D11, D12, D13, D14, D3, D4, D7, D8, D9: value LED -> WHITE LED
- D5, D6: value LED -> ORANGE LED
- turned SW1 to 90 degrees
Changed lines of the file:
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@@
 			)
 		)
-		(property "Value" "LED"
+		(property "Value" "GREEN LED"
 			(at 0 1.65 90)
 			(layer "F.Fab")
@@
 			)
 		)
-		(property "Value" "LED"
+		(property "Value" "GREEN LED"
 			(at -2.45 0 90)
 			(layer "F.Fab")
@@
 			)
 		)
-		(property "Value" "LED"
+		(property "Value" "WHITE LED"
 			(at -2.4 0.1 90)
 			(layer "F.Fab")
@@
 			)
 		)
-		(property "Value" "LED"
+		(property "Value" "WHITE LED"
 			(at -2.4 0.1 90)
 			(layer "F.Fab")
@@
 	(footprint "Button_Switch_SMD:SW_Push_1P1T_NO_CK_KSC7xxJ"
 		(layer "F.Cu")
-		(at 108.95 55.5 180)
+		(at 108.95 55.5 90)
 		(descr "CK components KSC7 tactile switch https://www.ckswitches.com/media/1973/ksc7.pdf")
 		(tags "tactile switch ksc7")
 		(property "Reference" "SW1"
-			(at -5.5 -1.75 90)
+			(at -5.5 -1.75 0)
 			(layer "F.SilkS")
 			(effects
@@
 		)
 		(property "Value" "~"
-			(at 0 -4.23 0)
+			(at 0 -4.23 90)
 			(layer "F.Fab")
 			(effects
@@
 		)
 		(property "Datasheet" "~"
-			(at 0 0 180)
+			(at 0 0 90)
 			(unlocked yes)
 			(layer "F.Fab")
@@
 		)
 		(property "Description" "Push button switch, generic, two pins"
-			(at 0 0 180)
+			(at 0 0 90)
 			(unlocked yes)
 			(layer "F.Fab")
@@
 		)
 		(property "Sim.Device" ""
-			(at 0 0 180)
+			(at 0 0 90)
 			(unlocked yes)
 			(layer "F.Fab")
@@
 		)
 		(property "Sim.Pins" ""
-			(at 0 0 180)
+			(at 0 0 90)
 			(unlocked yes)
 			(layer "F.Fab")
@@
 		(attr smd)
 		(fp_line
-			(start 3.21 3.21)
-			(end 3.21 2.93)
+			(start 3.21 -3.21)
+			(end -3.21 -3.21)
 			(stroke
 				(width 0.12)
@@
 		)
 		(fp_line
-			(start 3.21 1.2)
-			(end 3.21 -1.2)
+			(start -3.21 -3.21)
+			(end -3.21 -2.8)
 			(stroke
 				(width 0.12)
@@
 		)
 		(fp_line
-			(start 3.21 -3.21)
-			(end -3.21 -3.21)
+			(start -3.21 -1.2)
+			(end -3.21 1.2)
 			(stroke
 				(width 0.12)
@@
 		)
 		(fp_line
-			(start -3.21 3.21)
-			(end 3.21 3.21)
+			(start 3.21 1.2)
+			(end 3.21 -1.2)
 			(stroke
 				(width 0.12)
@@
 		)
 		(fp_line
-			(start -3.21 -1.2)
-			(end -3.21 1.2)
+			(start 3.21 3.21)
+			(end 3.21 2.93)
 			(stroke
 				(width 0.12)
@@
 		)
 		(fp_line
-			(start -3.21 -3.21)
-			(end -3.21 -2.8)
+			(start -3.21 3.21)
+			(end 3.21 3.21)
 			(stroke
 				(width 0.12)
@@
 		)
 		(fp_line
-			(start 4.55 3.35)
-			(end -4.55 3.35)
+			(start 4.55 -3.35)
+			(end 4.55 3.35)
 			(stroke
 				(width 0.05)
@@
 		)
 		(fp_line
-			(start 4.55 -3.35)
-			(end 4.55 3.35)
+			(start -4.55 -3.35)
+			(end 4.55 -3.35)
 			(stroke
 				(width 0.05)
@@
 		)
 		(fp_line
-			(start -4.55 3.35)
-			(end -4.55 -3.35)
+			(start 4.55 3.35)
+			(end -4.55 3.35)
 			(stroke
 				(width 0.05)
@@
 		)
 		(fp_line
-			(start -4.55 -3.35)
-			(end 4.55 -3.35)
+			(start -4.55 3.35)
+			(end -4.55 -3.35)
 			(stroke
 				(width 0.05)
@@
 		)
 		(fp_line
-			(start 3.1 3.1)
-			(end -3.1 3.1)
+			(start 3.1 -3.1)
+			(end 3.1 3.1)
 			(stroke
 				(width 0.1)
@@
 		)
 		(fp_line
-			(start 3.1 -3.1)
-			(end 3.1 3.1)
+			(start -3.1 -3.1)
+			(end 3.1 -3.1)
 			(stroke
 				(width 0.1)
@@
 		)
 		(fp_line
-			(start -3.1 3.1)
-			(end -3.1 -3.1)
+			(start 3.1 3.1)
+			(end -3.1 3.1)
 			(stroke
 				(width 0.1)
@@
 		)
 		(fp_line
-			(start -3.1 -3.1)
-			(end 3.1 -3.1)
+			(start -3.1 3.1)
+			(end -3.1 -3.1)
 			(stroke
 				(width 0.1)
@@
 		)
 		(fp_text user "${REFERENCE}"
-			(at 0 0 0)
+			(at 0 0 90)
 			(layer "F.Fab")
 			(effects
@@
 		)
 		(pad "1" smd roundrect
-			(at -2.9 -2 180)
+			(at -2.9 -2 90)
 			(size 2.8 1)
 			(layers "F.Cu" "F.Mask" "F.Paste")
@@
 		)
 		(pad "1" smd roundrect
-			(at 2.9 -2 180)
+			(at 2.9 -2 90)
 			(size 2.8 1)
 			(layers "F.Cu" "F.Mask" "F.Paste")
@@
 		)
 		(pad "2" smd roundrect
-			(at -2.9 2 180)
+			(at -2.9 2 90)
 			(size 2.8 1)
 			(layers "F.Cu" "F.Mask" "F.Paste")
@@
 		)
 		(pad "2" smd roundrect
-			(at 2.9 2 180)
+			(at 2.9 2 90)
 			(size 2.8 1)
 			(layers "F.Cu" "F.Mask" "F.Paste")
@@
 			)
 		)
-		(property "Value" "LED"
+		(property "Value" "WHITE LED"
 			(at -2.6 0.15 90)
 			(layer "F.Fab")
@@
 			)
 		)
-		(property "Value" "LED"
+		(property "Value" "WHITE LED"
 			(at -2.4 0.15 90)
 			(layer "F.Fab")
@@
 			)
 		)
-		(property "Value" "LED"
+		(property "Value" "WHITE LED"
 			(at -2.4125 0.15 180)
 			(layer "F.Fab")
@@
 			)
 		)
-		(property "Value" "LED"
+		(property "Value" "ORANGE LED"
 			(at -2.4125 -0.05 180)
 			(layer "F.Fab")
@@
 			)
 		)
-		(property "Value" "LED"
+		(property "Value" "WHITE LED"
 			(at -2.5 0 90)
 			(layer "F.Fab")
@@
 			)
 		)
-		(property "Value" "LED"
+		(property "Value" "ORANGE LED"
 			(at -2.4125 0.15 180)
 			(layer "F.Fab")
@@
 			)
 		)
-		(property "Value" "LED"
+		(property "Value" "WHITE LED"
 			(at -2.4125 0.15 180)
 			(layer "F.Fab")
@@
 			)
 		)
-		(property "Value" "LED"
+		(property "Value" "WHITE LED"
 			(at -2.5 0.1 90)
 			(layer "F.Fab")
@@
 			)
 		)
-		(property "Value" "LED"
+		(property "Value" "WHITE LED"
 			(at -2.5 0.14 90)
 			(layer "F.Fab")
@@
 			)
 		)
-		(property "Value" "LED"
+		(property "Value" "WHITE LED"
 			(at -2.5 0.1 90)
 			(layer "F.Fab")

Commit message: update
Parts:
- removed D10, D11, D12, D13, D14, D7, D8, D9: WHITE LED, LED_SMD:LED_0805_2012Metric
- removed J11: Conn_02x04_Odd_Even, Connector_PinHeader_2.54mm:PinHeader_2x04_P2.54mm_Vertical
- removed the J7 at (60.3, 38.2)
- removed R76, R77, R78, R79, R80, R81, R82, R83: 220, Resistor_SMD:R_0805_2012Metric
- J6: value Conn_02x08_Odd_Even -> Conn_02x16_Odd_Even; footprint Connector_PinHeader_2.54mm:PinHeader_2x08_P2.54mm_Vertical -> Connector_PinHeader_2.54mm:PinHeader_2x16_P2.54mm_Vertical
- moved J6 3.50 mm to (95.6, 38.2)
- renumbered J10 to J7
Routing:
- net +12V: track 634.8 -> 673.1 mm
- net GND: track 219.0 -> 199.7 mm, vias 67 -> 66
- net /mcu/+5V: track 74.7 -> 68.6 mm
- net /mcu/V_M8: track 48.1 -> 42.1 mm
- net Net-(D13-A): track 2.29 -> 0.00 mm
- net Net-(D12-A): track 2.28 -> 0.00 mm
- net Net-(D11-A): track 2.28 -> 0.00 mm
- net Net-(D10-A): track 2.28 -> 0.00 mm
- net Net-(D8-A): track 2.27 -> 0.00 mm
- net Net-(D7-A): track 2.27 -> 0.00 mm
- net Net-(D14-A): track 2.27 -> 0.00 mm
- net Net-(D9-A): track 1.95 -> 0.00 mm
- net /mcu/V_M4: track 140.4 -> 141.4 mm
- net /mcu/V_M3: track 178.1 -> 179.0 mm
- net /mcu/V_M6: track 78.0 -> 78.7 mm
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Other:
- board text added: "7.4V"
- board text added: "SAC MODULE V1.0.2 Produced by Lazycat Design"
- board text removed: "SAC MODULE V1.0.1 Produced by Lazycat Design"

Commit message: update
Routing:
- net +12V: track 673.1 -> 673.9 mm
Changed lines of the file:
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@@
-	)
-	(gr_line
-		(start 101.8 40.55)
-		(end 101.8 49.25)
-		(stroke
-			(width 0.1)
-			(type default)
-		)
-		(layer "F.SilkS")
 	)
 	(gr_line
@@
 	)
 	(gr_line
-		(start 130 35.7)
-		(end 130.5 35.7)
-		(stroke
-			(width 0.1)
-			(type solid)
-		)
-		(layer "F.SilkS")
-	)
-	(gr_line
 		(start 75.25 43.2)
 		(end 75.25 42.7)
-		(stroke
-			(width 0.1)
-			(type solid)
-		)
-		(layer "F.SilkS")
-	)
-	(gr_line
-		(start 101.225 40.55)
-		(end 101.775 40.55)
 		(stroke
 			(width 0.1)
@@
 	)
 	(gr_line
-		(start 101.8 46.6)
-		(end 130 46.6)
-		(stroke
-			(width 0.1)
-			(type solid)
-		)
-		(layer "F.SilkS")
-	)
-	(gr_line
 		(start 77.85 43.2)
 		(end 77.85 42.7)
@@
 			(width 0.1)
 			(type solid)
-		)
-		(layer "F.SilkS")
-	)
-	(gr_line
-		(start 130 46.575)
-		(end 130 35.725)
-		(stroke
-			(width 0.1)
-			(type default)
 		)
 		(layer "F.SilkS")
@@
 	)
 	(gr_text "V_M6"
-		(at 134.33 37.876191 90)
+		(at 82.8 46.2 90)
 		(layer "F.SilkS")
 		(effects
@@
 	)
 	(gr_text "V_M5"
-		(at 135.9 37.876191 90)
+		(at 85.6 46.2 90)
 		(layer "F.SilkS")
 		(effects
@@
 	)
 	(gr_text "V_M4"
-		(at 137.5 37.876191 90)
+		(at 88.2 46.2 90)
 		(layer "F.SilkS")
 		(effects
@@
 	)
 	(gr_text "V_M7"
-		(at 132.95 37.876191 90)
+		(at 80.4 46.2 90)
 		(layer "F.SilkS")
 		(effects
@@
 	)
 	(gr_text "V_M2"
-		(at 140.3 37.876191 90)
+		(at 93.2 46.2 90)
 		(layer "F.SilkS")
 		(effects
@@
 	)
 	(gr_text "V_M8"
-		(at 131.45 37.876191 90)
+		(at 78 46.2 90)
 		(layer "F.SilkS")
 		(effects
@@
 	)
 	(gr_text "V_M1"
-		(at 141.7 37.876191 90)
+		(at 95.6 46.2 90)
 		(layer "F.SilkS")
 		(effects
@@
 	)
 	(gr_text "V_M3"
-		(at 139 37.876191 90)
+		(at 90.6 46.2 90)
 		(layer "F.SilkS")
 		(effects
@@
 	)
 	(segment
+		(start 97.361 33.761)
+		(end 99.2 35.6)
+		(width 0.6)
+		(layer "F.Cu")
+		(net 5)
+	)
+	(segment
 		(start 53.3 51.75)
 		(end 53.5 51.75)
@@
 	)
 	(segment
+		(start 99.2 45.2)
+		(end 97.4 47)
+		(width 0.6)
+		(layer "F.Cu")
+		(net 5)
+	)
+	(segment
 		(start 89.9375 58.05)
 		(end 90.1375 58.25)
@@
 	)
 	(segment
-		(start 99.2 36.2)
-		(end 99.2 44.4)
+		(start 77 33.761)
+		(end 97.361 33.761)
 		(width 0.6)
 		(layer "F.Cu")
@@
 	)
 	(segment
-		(start 96.6 47)
-		(end 79.2 47)
-		(width 0.6)
-		(layer "F.Cu")
-		(net 5)
-	)
-	(segment
 		(start 90.9625 56.8375)
 		(end 89.9375 56.8375)
@@
 	)
 	(segment
-		(start 96.761 33.761)
-		(end 99.2 36.2)
-		(width 0.6)
-		(layer "F.Cu")
-		(net 5)
-	)
-	(segment
 		(start 123.25 110.25)
 		(end 123.25 101)
@@
 	)
 	(segment
-		(start 77 33.761)
-		(end 96.761 33.761)
-		(width 0.6)
-		(layer "F.Cu")
-		(net 5)
-	)
-	(segment
 		(start 66.32125 56.90375)
 		(end 65.69625 56.90375)
@@
 	)
 	(segment
+		(start 97.4 47)
+		(end 79.2 47)
+		(width 0.6)
+		(layer "F.Cu")
+		(net 5)
+	)
+	(segment
 		(start 68.5 102.3)
 		(end 68.5 110.359)
@@
 	)
 	(segment
+		(start 99.2 35.6)
+		(end 99.2 45.2)
+		(width 0.6)
+		(layer "F.Cu")
+		(net 5)
+	)
+	(segment
 		(start 63.25 56.5)
 		(end 65.2925 56.5)
@@
 		(width 0.6)
 		(layer "F.Cu")
-		(net 5)
-	)
-	(segment
-		(start 99.2 44.4)
-		(end 96.6 47)
-		(width 0.6)
-		(layer "F.Cu")
