File: sac_board.kicad_pcb (KiCad board)
At the start: 2 copper layers, 120 x 80 mm, 240 parts, among them J1 12V_Input, J2 USB_B_Mini, J3 Micro_SD_Card_Det1, J4 ARM JTAG/SWD, J5 DE9_Socket, J6 Conn_02x16_Odd_Even, J7 Conn_02x09_Odd_Even, J8 Conn_02x14_Odd_Even, J9 RJ45, U1 TPS563201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

Commit message: update
Parts:
- added C114: 0.1uF, Capacitor_SMD:C_0805_2012Metric, F.Cu at (31.8, 61.1)
- added C115: 0.1uF, Capacitor_SMD:C_0805_2012Metric, F.Cu at (31.8, 64.1)
- added C116: 0.1uF, Capacitor_SMD:C_0805_2012Metric, F.Cu at (31.8, 67.1)
- added C117: 0.1uF, Capacitor_SMD:C_0805_2012Metric, F.Cu at (31.8, 70.1)
- added C118: 0.1uF, Capacitor_SMD:C_0805_2012Metric, F.Cu at (31.8, 73.1)
Other:
- board text added: "SAC MODULE V1.0.3 Produced by Lazycat Design"
- board text removed: "SAC MODULE V1.0.2 Produced by Lazycat Design"

Commit message: update
Parts:
- added C119: 0.1uF, Capacitor_SMD:C_0805_2012Metric, B.Cu at (102.9, 75.5)
- C100, C101, C102, C114, C115, C116, C117, C94, C96: moved to B.Cu
- moved C118 87.2 mm to (117.5, 88.8), turned to 180 degrees
- moved C115 82.1 mm to (113.0, 75.5), turned to 90 degrees
- moved C114 79.0 mm to (109.4, 75.5), turned to 90 degrees
- moved C116 74.9 mm to (106.2, 75.5), turned to 90 degrees
- moved C117 74.9 mm to (105.2, 84.5), turned to 90 degrees
- moved C94 2.97 mm to (85.5, 74.2)
- moved C96 2.93 mm to (82.8, 81.0), turned to -90 degrees
- moved C102 2.90 mm to (78.3, 79.1), turned to 90 degrees
- moved R53 2.10 mm to (78.4, 80.5)
- moved R60 2.10 mm to (74.2, 80.5)
- moved Y3 2.10 mm to (78.2, 83.9)
- moved C93 2.10 mm to (73.6, 83.9)
- moved C92 1.72 mm to (82.7, 83.9)
- moved C88 1.54 mm to (114.3, 91.2)
- moved C87 1.28 mm to (97.5, 87.0), turned to 180 degrees
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Routing:
- net GND: track 199.7 -> 186.8 mm, vias 66 -> 65
- net /mcu/+3.3V: track 481.3 -> 471.1 mm, vias 30 -> 31
- net /mcu/PC0-ETH-RESET: track 35.3 -> 39.6 mm
- net /mcu/PC1-ETH-MDC: track 30.2 -> 34.1 mm
- net /mcu/PB13-RMII-TXD1: track 42.2 -> 39.0 mm
- net /mcu/PB12-RMII-TXD0: track 42.0 -> 38.8 mm
- net Net-(U13-XTAL2): track 16.5 -> 13.7 mm
- net Net-(U13-XTAL1/CLKIN): track 16.1 -> 13.4 mm
- net /mcu/PC8-SDIO-D0: track 26.7 -> 28.5 mm
- net /mcu/PE4: track 45.1 -> 43.5 mm
- net /mcu/PB11-RMII-TXEN: track 30.4 -> 31.8 mm
- net /mcu/V_M3: track 179.0 -> 178.1 mm
- net /mcu/PA9-USART1-TX: track 29.5 -> 28.8 mm
- net /mcu/PA12-USB-DP: track 12.7 -> 12.0 mm
- net /mcu/LED-LINK: track 45.4 -> 44.7 mm
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
Commit message: update
Routing:
- net /mcu/LED-SPEED: track 45.8 -> 45.1 mm
Changed lines of the file:
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@@
-	)
-	(segment
-		(start 80 76.683884)
-		(end 80 75.9375)
-		(width 0.2)
-		(layer "F.Cu")
-		(net 131)
 	)
 	(segment
@@
 	)
 	(segment
+		(start 79.716942 76.966942)
+		(end 80 76.683884)
+		(width 0.2)
+		(layer "F.Cu")
+		(net 131)
+	)
+	(segment
+		(start 80 76.683884)
+		(end 80 75.9375)
+		(width 0.2)
+		(layer "F.Cu")
+		(net 131)
+	)
+	(segment
 		(start 75.2 68.6625)
 		(end 74.5375 68)
@@
 		(start 49.135 62.25)
 		(end 54.25 62.25)
-		(width 0.2)
-		(layer "F.Cu")
-		(net 131)
-	)
-	(segment
-		(start 79.391942 77.291942)
-		(end 80 76.683884)
 		(width 0.2)
 		(layer "F.Cu")
@@
 	)
 	(via
-		(at 79.391942 77.291942)
+		(at 79.716942 76.966942)
 		(size 0.6)
 		(drill 0.3)
@@
 	)
 	(segment
-		(start 75.899943 70.3)
-		(end 75.899943 70.299943)
-		(width 0.2)
-		(layer "B.Cu")
-		(net 131)
-	)
-	(segment
-		(start 79.562947 77.120937)
+		(start 79.712947 76.962947)
 		(end 79.562947 76.962947)
 		(width 0.2)
@@
 	)
 	(segment
-		(start 79.562947 76.962947)
-		(end 77.7 75.1)
+		(start 77.7 75.1)
+		(end 77.7 72.100057)
 		(width 0.2)
 		(layer "B.Cu")
@@
 	)
 	(segment
-		(start 79.391942 77.291942)
-		(end 79.562947 77.120937)
+		(start 79.716942 76.966942)
+		(end 79.712947 76.962947)
 		(width 0.2)
 		(layer "B.Cu")
@@
 	)
 	(segment
-		(start 77.7 75.1)
-		(end 77.7 72.100057)
+		(start 75.899943 70.3)
+		(end 75.899943 70.299943)
 		(width 0.2)
 		(layer "B.Cu")
@@
 		(width 0.2)
 		(layer "B.Cu")
+		(net 131)
+	)
+	(segment
+		(start 79.562947 76.962947)
+		(end 77.7 75.1)
+		(width 0.2)
+		(layer "B.Cu")

Commit message: update
Parts:
- moved L3 4.65 mm to (102.8, 65.0)
- moved C17 2.30 mm to (105.1, 65.1)
- moved C18 2.30 mm to (107.5, 65.1)
- moved C117 1.80 mm to (104.0, 85.8), turned to 180 degrees
Routing:
- net /mcu/+3.3V: track 471.1 -> 464.3 mm
- net /mcu/PB13-RMII-TXD1: track 39.0 -> 44.1 mm
- net /mcu/PB12-RMII-TXD0: track 38.8 -> 41.1 mm
- net /mcu/VDDA: track 18.2 -> 16.5 mm
- net /mcu/LED-SPEED: track 45.1 -> 45.8 mm

Commit message: update
Parts:
- removed J4: ARM JTAG/SWD, Connector_IDC:IDC-Header_2x10_P2.54mm_Vertical
- removed U12: MAX3232, Package_SO:SOIC-16_4.55x10.3mm_P1.27mm
- added C120: 10uF, Capacitor_SMD:C_0805_2012Metric, B.Cu at (74.9, 73.6)
- added C121: 10uF, Capacitor_SMD:C_0805_2012Metric, B.Cu at (84.7, 79.6)
- added H5: MountingHole, MountingHole:MountingHole_3mm, F.Cu at (189.5, 50.5)
- added H6: MountingHole, MountingHole:MountingHole_3mm, F.Cu at (188.0, 60.0)
- added H7: MountingHole, MountingHole:MountingHole_3mm, F.Cu at (188.0, 70.0)
- added H8: MountingHole, MountingHole:MountingHole_3mm, F.Cu at (188.0, 79.0)
- C91, C95, C97, C99: value 0.1uF -> 10uF; moved to B.Cu
- C98: value 0.1uF -> 10uF
- H1, H2, H3, H4: footprint MountingHole:MountingHole_2.7mm_M2.5 -> MountingHole:MountingHole_3mm
- J5: value DE9_Socket -> Conn_02x08_Odd_Even; footprint Custom:DSUB-9_Pins_Horizontal_P2.77x2.84mm_EdgePinOffset7.70mm_Housed_MountingHolesOffset9.12mm_Female -> Connector_PinHeader_2.54mm:PinHeader_2x08_P2.54mm_Vertical
- moved C99 67.1 mm to (74.9, 79.6), turned to 0 degrees
- moved C97 39.2 mm to (103.4, 87.1), turned to 180 degrees
- moved C91 32.9 mm to (111.2, 78.9), turned to 90 degrees
- moved J5 28.6 mm to (149.7, 66.3), turned to 0 degrees
- moved R54 26.6 mm to (141.9, 74.9)
- moved C98 26.0 mm to (118.2, 93.6)
- moved C95 23.2 mm to (106.7, 78.9), turned to 90 degrees
- moved R55 19.4 mm to (141.9, 77.4)
- moved R56 19.3 mm to (141.9, 72.4)
- moved SW2 17.8 mm to (54.6, 106.8)
- moved R70 17.0 mm to (137.9, 82.9)
- moved R71 16.9 mm to (69.2, 91.0), turned to -90 degrees
- moved D5 16.9 mm to (141.9, 82.9)
- moved R62 16.9 mm to (137.9, 87.9)
- moved R69 16.9 mm to (137.9, 85.4)
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Connections:
- C91 pad 1: Net-(U12-C1-) -> GND
- C91 pad 2: Net-(U12-C1+) -> /mcu/+3.3V
- C97 pad 1: Net-(U12-C2+) -> GND
- C97 pad 2: Net-(U12-C2-) -> /mcu/+3.3V
- C98 pad 2: Net-(U12-VS+) -> /mcu/+3.3V
- C99 pad 2: Net-(U12-VS-) -> /mcu/+3.3V
- J5 pad 1: unconnected-(J5-Pad1) -> /mcu/PB4-JNTRST
- J5 pad 2: Net-(U12-T2OUT) -> /mcu/+3.3V
- J5 pad 3: Net-(U12-R2IN) -> /mcu/PA15-JTDI
- J5 pad 4: unconnected-(J5-Pad4) -> GND
- J5 pad 5: GND -> /mcu/PA13-JTMS
- J5 pad 6: unconnected-(J5-Pad6) -> GND
- J5 pad 7: unconnected-(J5-Pad7) -> /mcu/PB3-JTDO
- J5 pad 8: unconnected-(J5-Pad8) -> GND
- J5 pad 9: unconnected-(J5-Pad9) -> /mcu/PA14-JTCK
- R54 pad 2: /mcu/PB4-JNTRST -> /mcu/PB3-JTDO
- R57 pad 2: /mcu/PB3-JTDO -> /mcu/PA15-JTDI
- R58 pad 2: /mcu/PA15-JTDI -> /mcu/PB4-JNTRST
Routing:
- net /mcu/+3.3V: track 464.3 -> 398.2 mm, vias 31 -> 25
- net GND: track 186.8 -> 138.0 mm, vias 65 -> 57
- net /mcu/PA4: track 74.8 -> 30.3 mm
- net /mcu/PA5: track 69.5 -> 32.2 mm
- net /mcu/PA6: track 57.5 -> 32.1 mm
- net Net-(U12-R2IN): track 25.3 -> 0.00 mm
- net Net-(U12-T2OUT): track 22.0 -> 0.00 mm
- net /mcu/PA14-JTCK: track 67.9 -> 47.1 mm
- net /mcu/PA9-USART1-TX: track 28.8 -> 44.4 mm
- net /mcu/PB4-JNTRST: track 55.8 -> 40.7 mm
- net /mcu/PB3-JTDO: track 52.8 -> 37.8 mm
- net /mcu/PA13-JTMS: track 63.2 -> 48.7 mm
- net /mcu/PA15-JTDI: track 62.9 -> 48.5 mm
- net /mcu/PA3: track 54.3 -> 67.9 mm
- net /mcu/PD5: track 37.0 -> 23.5 mm
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Other:
- board text added: "JNTRST"
- board text added: "JTCK/SWCLK"
- board text added: "JTDI"
- board text added: "JTDO/SWO"
- board text added: "JTMS/SWDIO"
- board text added: "REST"
- board text added: "USART1_RX"
- board text added: "USART1_TX"

Commit message: update
Parts:
- removed H5, H6, H7, H8: MountingHole, MountingHole:MountingHole_3mm
- moved R63 18.4 mm to (68.8, 91.2), turned to 90 degrees
- moved C112 17.3 mm to (53.0, 101.0), turned to 0 degrees
- moved SW4 16.4 mm to (54.5, 107.0)
- moved R71 16.0 mm to (56.8, 101.0), turned to 0 degrees
- moved SW2 16.0 mm to (64.0, 93.9)
- moved C106 13.3 mm to (68.8, 94.9), turned to 90 degrees
- moved H4 7.42 mm to (150.7, 105.5)
- moved H1 7.36 mm to (150.7, 45.5)
- moved R75 3.90 mm to (66.2, 101.0), turned to 0 degrees
- moved C113 3.70 mm to (62.4, 101.0)
- moved SW5 0.30 mm to (64.0, 107.0)
- turned R68 to 0 degrees
Routing:
- net /mcu/+3.3V: track 398.2 -> 448.3 mm, vias 25 -> 29
- net /mcu/PA5: track 32.2 -> 65.0 mm
- net GND: track 138.0 -> 169.9 mm, vias 57 -> 61
- net /mcu/PA6: track 32.1 -> 56.1 mm
- net /mcu/PA4: track 30.3 -> 48.7 mm
- net +12V: track 662.4 -> 655.2 mm
- net /mcu/PA3: track 67.9 -> 68.7 mm
Other:
- board text removed: "RESET"

Commit message: update
Routing:
- net +12V: track 655.2 -> 656.9 mm
Changed lines of the file:
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@@
 	)
 	(segment
-		(start 51.1556 109.3216)
-		(end 55.59075 113.75675)
-		(width 2.4)
-		(layer "B.Cu")
-		(net 5)
-	)
-	(segment
 		(start 62.67725 57.82275)
 		(end 62.67725 57.59775)
@@
 	)
 	(segment
-		(start 49.6545 50.4)
-		(end 44.3 50.4)
-		(width 2.4)
-		(layer "B.Cu")
-		(net 5)
-	)
-	(segment
 		(start 102.87725 60.67275)
 		(end 102.92725 60.62275)
@@
 	)
 	(segment
-		(start 51.1556 101.6)
-		(end 51.1556 109.3216)
-		(width 2.4)
-		(layer "B.Cu")
-		(net 5)
-	)
-	(segment
 		(start 104.70225 60.62275)
 		(end 105.17725 61.09775)
@@
 	)
 	(segment
-		(start 40.40825 54.29175)
-		(end 40.40825 90.85265)
-		(width 2.4)
-		(layer "B.Cu")
-		(net 5)
-	)
-	(segment
 		(start 100.92725 60.62275)
 		(end 101.42725 60.62275)
@@
 	)
 	(segment
+		(start 49.6545 50.4)
+		(end 44.3 50.4)
+		(width 2.4)
+		(layer "B.Cu")
+		(net 5)
+	)
+	(segment
 		(start 78.87725 54.59775)
 		(end 77.17725 56.29775)
@@
 	)
 	(segment
-		(start 122.87125 113.75675)
-		(end 122.92725 113.70075)
-		(width 2.4)
-		(layer "B.Cu")
-		(net 5)
-	)
-	(segment
 		(start 124.42725 101.72275)
 		(end 124.42725 102.14775)
@@
 	)
 	(segment
+		(start 51.1556 101.6)
+		(end 51.1556 112.1556)
+		(width 2.4)
+		(layer "B.Cu")
+		(net 5)
+	)
+	(segment
 		(start 82.87725 61.82275)
 		(end 82.92725 61.77275)
@@
 	)
 	(segment
+		(start 40.40825 90.85265)
+		(end 51.1556 101.6)
+		(width 2.4)
+		(layer "B.Cu")
+		(net 5)
+	)
+	(segment
+		(start 52.97725 55.14775)
+		(end 52.97725 53.72275)
+		(width 2.4)
+		(layer "B.Cu")
+		(net 5)
+	)
+	(segment
 		(start 62.07725 57.64775)
 		(end 61.67725 57.24775)
@@
 	)
 	(segment
-		(start 40.40825 90.85265)
-		(end 51.1556 101.6)
-		(width 2.4)
-		(layer "B.Cu")
-		(net 5)
-	)
-	(segment
-		(start 52.97725 55.14775)
-		(end 52.97725 53.72275)
-		(width 2.4)
-		(layer "B.Cu")
-		(net 5)
-	)
-	(segment
 		(start 58.07725 95.74775)
 		(end 58.17725 95.64775)
@@
 	)
 	(segment
+		(start 122.87125 113.75675)
+		(end 122.92725 113.70075)
+		(width 2.4)
+		(layer "B.Cu")
+		(net 5)
+	)
+	(segment
 		(start 101.17725 53.39775)
 		(end 99.87725 54.69775)
@@
 	)
 	(segment
+		(start 51.1556 112.1556)
+		(end 52.75675 113.75675)
+		(width 2.4)
+		(layer "B.Cu")
+		(net 5)
+	)
+	(segment
 		(start 58.17725 96.64775)
 		(end 58.67725 97.14775)
@@
 	)
 	(segment
-		(start 52.97725 53.72275)
-		(end 49.6545 50.4)
-		(width 2.4)
-		(layer "B.Cu")
-		(net 5)
-	)
-	(segment
 		(start 108.97725 104.24775)
 		(end 108.97725 103.99775)
@@
 	)
 	(segment
-		(start 55.59075 113.75675)
-		(end 122.87125 113.75675)
-		(width 2.4)
-		(layer "B.Cu")
-		(net 5)
-	)
-	(segment
 		(start 104.92725 61.97275)
 		(end 104.87725 62.02275)
@@
 	)
 	(segment
-		(start 44.3 50.4)
-		(end 40.40825 54.29175)
-		(width 2.4)
-		(layer "B.Cu")
-		(net 5)
-	)
-	(segment
 		(start 56.82725 97.89775)
 		(end 57.57725 97.14775)
@@
 	)
 	(segment
+		(start 52.97725 53.72275)
+		(end 49.6545 50.4)
+		(width 2.4)
+		(layer "B.Cu")
+		(net 5)
+	)
+	(segment
+		(start 44.3 50.4)
+		(end 40.40825 54.29175)
+		(width 2.4)
+		(layer "B.Cu")
+		(net 5)
+	)
+	(segment
 		(start 125.67725 103.39775)
 		(end 125.67725 104.69775)
@@
 	)
 	(segment
+		(start 40.40825 54.29175)
+		(end 40.40825 90.85265)
+		(width 2.4)
+		(layer "B.Cu")
+		(net 5)
+	)
+	(segment
 		(start 59.77725 55.89775)
 		(end 58.47725 54.59775)
@@
 	)
 	(segment
+		(start 52.75675 113.75675)
+		(end 122.87125 113.75675)
+		(width 2.4)
+		(layer "B.Cu")
+		(net 5)
+	)
+	(segment
 		(start 58.67725 92.89775)
 		(end 58.17725 93.39775)
@@
 	)
 	(segment
+		(start 77 73.25)
+		(end 77 72.5205)
+		(width 0.2)
+		(layer "F.Cu")
+		(net 131)
+	)
+	(segment
 		(start 53.92725 65.64775)
 		(end 58.87725 70.59775)
@@
 	)
 	(segment
-		(start 79.394192 80.364692)
-		(end 79.67725 80.081634)
+		(start 77 72.5205)
+		(end 75.87725 71.39775)
 		(width 0.2)
 		(layer "F.Cu")
@@
 	)
 	(segment
-		(start 75.87725 71.39775)
-		(end 77.47725 72.99775)
+		(start 79.394192 80.364692)
+		(end 79.67725 80.081634)
 		(width 0.2)
 		(layer "F.Cu")
@@
 	)
 	(segment
-		(start 74.21475 71.39775)
+		(start 75.87725 71.39775)
 		(end 75.60225 71.39775)
 		(width 0.2)
@@
 	)
 	(segment
-		(start 75.60225 71.39775)
-		(end 75.87725 71.39775)
+		(start 74.21475 71.39775)
+		(end 75.60225 71.39775)
 		(width 0.2)
 		(layer "F.Cu")
@@
 	)
 	(via
-		(at 77.47725 72.99775)
+		(at 77 73.25)
 		(size 0.6)
 		(drill 0.3)
@@
 	)
 	(segment
-		(start 77.47725 79.69775)
-		(end 78.140197 80.360697)
+		(start 77 73.25)
+		(end 77 79.2205)
 		(width 0.2)
 		(layer "B.Cu")
@@
 	)
 	(segment
-		(start 78.140197 80.360697)
-		(end 79.390197 80.360697)
+		(start 77 79.2205)
+		(end 78.140197 80.360697)
 		(width 0.2)
 		(layer "B.Cu")
@@
 	)
 	(segment
-		(start 77.47725 72.99775)
-		(end 77.47725 79.69775)
+		(start 78.140197 80.360697)
+		(end 79.390197 80.360697)
 		(width 0.2)
 		(layer "B.Cu")
