File: sac_board.kicad_sch (KiCad schematic)
At the start: 0 parts

Commit message: update
Other:
- sheet mcu ports: added none; removed +7V_M10, +7V_M11, +7V_M12, +7V_M9
- sheet power_servo ports: added none; removed +7V_M10, +7V_M11, +7V_M12, +7V_M9
Changed lines of the file:
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@@
-	(wire
-		(pts
-			(xy 172.72 95.25) (xy 172.72 152.4)
-		)
-		(stroke
-			(width 0)
-			(type default)
-		)
-	)
-	(wire
-		(pts
-			(xy 96.52 137.16) (xy 157.48 137.16)
-		)
-		(stroke
-			(width 0)
-			(type default)
-		)
-	)
-	(wire
-		(pts
-			(xy 157.48 83.82) (xy 212.09 83.82)
-		)
-		(stroke
-			(width 0)
-			(type default)
-		)
-	)
 	(wire
 		(pts
@@
 	(wire
 		(pts
-			(xy 162.56 87.63) (xy 212.09 87.63)
-		)
-		(stroke
-			(width 0)
-			(type default)
-		)
-	)
-	(wire
-		(pts
 			(xy 147.32 76.2) (xy 212.09 76.2)
 		)
@@
 	(wire
 		(pts
-			(xy 157.48 137.16) (xy 157.48 83.82)
-		)
-		(stroke
-			(width 0)
-			(type default)
-		)
-	)
-	(wire
-		(pts
 			(xy 121.92 57.15) (xy 212.09 57.15)
 		)
@@
 	(wire
 		(pts
-			(xy 162.56 87.63) (xy 162.56 142.24)
-		)
-		(stroke
-			(width 0)
-			(type default)
-		)
-	)
-	(wire
-		(pts
-			(xy 96.52 152.4) (xy 172.72 152.4)
-		)
-		(stroke
-			(width 0)
-			(type default)
-		)
-	)
-	(wire
-		(pts
-			(xy 167.64 147.32) (xy 167.64 91.44)
-		)
-		(stroke
-			(width 0)
-			(type default)
-		)
-	)
-	(wire
-		(pts
 			(xy 96.52 127) (xy 147.32 127)
 		)
@@
 	(wire
 		(pts
-			(xy 96.52 147.32) (xy 167.64 147.32)
-		)
-		(stroke
-			(width 0)
-			(type default)
-		)
-	)
-	(wire
-		(pts
 			(xy 121.92 101.6) (xy 121.92 57.15)
 		)
@@
 	(wire
 		(pts
-			(xy 172.72 95.25) (xy 212.09 95.25)
-		)
-		(stroke
-			(width 0)
-			(type default)
-		)
-	)
-	(wire
-		(pts
-			(xy 96.52 142.24) (xy 162.56 142.24)
-		)
-		(stroke
-			(width 0)
-			(type default)
-		)
-	)
-	(wire
-		(pts
 			(xy 95.25 48.26) (xy 212.09 48.26)
 		)
@@
 		(pts
 			(xy 127 106.68) (xy 127 60.96)
-		)
-		(stroke
-			(width 0)
-			(type default)
-		)
-	)
-	(wire
-		(pts
-			(xy 167.64 91.44) (xy 212.09 91.44)
 		)
 		(stroke
@@
 			)
 		)
-		(pin "+7V_M9" input
-			(at 212.09 83.82 180)
-			(effects
-				(font
-					(size 1.27 1.27)
-				)
-				(justify left)
-			)
-		)
-		(pin "+7V_M10" input
-			(at 212.09 87.63 180)
-			(effects
-				(font
-					(size 1.27 1.27)
-				)
-				(justify left)
-			)
-		)
-		(pin "+7V_M11" input
-			(at 212.09 91.44 180)
-			(effects
-				(font
-					(size 1.27 1.27)
-				)
-				(justify left)
-			)
-		)
-		(pin "+7V_M12" input
-			(at 212.09 95.25 180)
-			(effects
-				(font
-					(size 1.27 1.27)
-				)
-				(justify left)
-			)
-		)
 		(pin "VDDA" input
 			(at 212.09 48.26 180)
@@
 			(effects
 				(font
-					(size 1.27 1.27)
-				)
-				(justify right)
-			)
-		)
-		(pin "+7V_M9" output
-			(at 96.52 137.16 0)
-			(effects
-				(font
-					(size 1.27 1.27)
-				)
-				(justify right)
-			)
-		)
-		(pin "+7V_M10" output
-			(at 96.52 142.24 0)
-			(effects
-				(font
-					(size 1.27 1.27)
-				)
-				(justify right)
-			)
-		)
-		(pin "+7V_M11" output
-			(at 96.52 147.32 0)
-			(effects
-				(font
-					(size 1.27 1.27)
-				)
-				(justify right)
-			)
-		)
-		(pin "+7V_M12" output
-			(at 96.52 152.4 0)
-			(effects
-				(font

Commit message: update
Other:
- sheet mcu ports: added V_M1, V_M2, V_M3, V_M4, V_M5, V_M6, V_M7, V_M8; removed +7V_M1, +7V_M2, +7V_M3, +7V_M4, +7V_M5, +7V_M6, +7V_M7, +7V_M8
- sheet power_servo ports: added V_M1, V_M2, V_M3, V_M4, V_M5, V_M6, V_M7, V_M8; removed +7V_M1, +7V_M2, +7V_M3, +7V_M4, +7V_M5, +7V_M6, +7V_M7, +7V_M8
Changed lines of the file:
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@@
 	(sheet
 		(at 212.09 35.56)
-		(size 45.72 77.47)
+		(size 45.72 48.895)
 		(exclude_from_sim no)
 		(in_bom yes)
@@
 		)
 		(property "Sheetfile" "mcu.kicad_sch"
-			(at 212.09 113.6146 0)
+			(at 212.09 85.0396 0)
 			(effects
 				(font
@@
 			)
 		)
-		(pin "+7V_M1" input
+		(pin "V_M1" input
 			(at 212.09 53.34 180)
 			(effects
@@
 			)
 		)
-		(pin "+7V_M2" input
+		(pin "V_M2" input
 			(at 212.09 57.15 180)
 			(effects
@@
 			)
 		)
-		(pin "+7V_M3" input
+		(pin "V_M3" input
 			(at 212.09 60.96 180)
 			(effects
@@
 			)
 		)
-		(pin "+7V_M4" input
+		(pin "V_M4" input
 			(at 212.09 64.77 180)
 			(effects
@@
 			)
 		)
-		(pin "+7V_M5" input
+		(pin "V_M5" input
 			(at 212.09 68.58 180)
 			(effects
@@
 			)
 		)
-		(pin "+7V_M6" input
+		(pin "V_M6" input
 			(at 212.09 72.39 180)
 			(effects
@@
 			)
 		)
-		(pin "+7V_M7" input
+		(pin "V_M7" input
 			(at 212.09 76.2 180)
 			(effects
@@
 			)
 		)
-		(pin "+7V_M8" input
+		(pin "V_M8" input
 			(at 212.09 80.01 180)
 			(effects
@@
 	(sheet
 		(at 49.53 90.17)
-		(size 46.99 67.945)
+		(size 46.99 48.895)
 		(exclude_from_sim no)
 		(in_bom yes)
@@
 		)
 		(property "Sheetfile" "power_servo.kicad_sch"
-			(at 49.53 158.6996 0)
+			(at 49.53 139.6496 0)
 			(effects
 				(font
@@
 			)
 		)
-		(pin "+7V_M1" output
+		(pin "V_M1" output
 			(at 96.52 96.52 0)
 			(effects
@@
 			)
 		)
-		(pin "+7V_M2" output
+		(pin "V_M2" output
 			(at 96.52 101.6 0)
 			(effects
@@
 			)
 		)
-		(pin "+7V_M3" output
+		(pin "V_M3" output
 			(at 96.52 106.68 0)
 			(effects
@@
 			)
 		)
-		(pin "+7V_M4" output
+		(pin "V_M4" output
 			(at 96.52 111.76 0)
 			(effects
@@
 			)
 		)
-		(pin "+7V_M5" output
+		(pin "V_M5" output
 			(at 96.52 116.84 0)
 			(effects
@@
 			)
 		)
-		(pin "+7V_M6" output
+		(pin "V_M6" output
 			(at 96.52 121.92 0)
 			(effects
@@
 			)
 		)
-		(pin "+7V_M7" output
+		(pin "V_M7" output
 			(at 96.52 127 0)
 			(effects
@@
 			)
 		)
-		(pin "+7V_M8" output
+		(pin "V_M8" output
 			(at 96.52 132.08 0)
 			(effects

Commit message: update
Other:
- added sheet led_servo (led_servo.kicad_sch)

Commit message: update
Changed lines of the file:
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@@
 	(wire
 		(pts
-			(xy 95.25 40.64) (xy 212.09 40.64)
+			(xy 87.63 29.21) (xy 212.09 29.21)
 		)
 		(stroke
@@
 	(wire
 		(pts
-			(xy 95.25 44.45) (xy 212.09 44.45)
+			(xy 87.63 33.02) (xy 212.09 33.02)
 		)
 		(stroke
@@
 	(wire
 		(pts
-			(xy 95.25 48.26) (xy 212.09 48.26)
-		)
-		(stroke
-			(width 0)
-			(type default)
-		)
-	)
-	(wire
-		(pts
 			(xy 171.45 124.46) (xy 212.09 124.46)
 		)
@@
 		(pts
 			(xy 142.24 121.92) (xy 142.24 72.39)
+		)
+		(stroke
+			(width 0)
+			(type default)
+		)
+	)
+	(wire
+		(pts
+			(xy 87.63 36.83) (xy 212.09 36.83)
 		)
 		(stroke
@@
 	)
 	(sheet
-		(at 212.09 35.56)
-		(size 45.72 48.895)
+		(at 212.09 24.765)
+		(size 45.72 67.31)
 		(exclude_from_sim no)
 		(in_bom yes)
@@
 		)
 		(property "Sheetname" "mcu"
-			(at 212.09 34.8484 0)
+			(at 212.09 24.0534 0)
 			(effects
 				(font
@@
 		)
 		(property "Sheetfile" "mcu.kicad_sch"
-			(at 212.09 85.0396 0)
+			(at 212.09 92.6596 0)
 			(effects
 				(font
@@
 		)
 		(pin "+3.3V" input
-			(at 212.09 40.64 180)
+			(at 212.09 29.21 180)
 			(effects
 				(font
@@
 		)
 		(pin "+5V" input
-			(at 212.09 44.45 180)
+			(at 212.09 33.02 180)
 			(effects
 				(font
@@
 		)
 		(pin "VDDA" input
-			(at 212.09 48.26 180)
+			(at 212.09 36.83 180)
 			(effects
 				(font
@@
 	)
 	(sheet
-		(at 48.26 38.1)
-		(size 46.99 18.415)
+		(at 40.64 24.13)
+		(size 46.99 20.955)
 		(exclude_from_sim no)
 		(in_bom yes)
@@
 		)
 		(property "Sheetname" "power_mcu"
-			(at 48.26 37.3884 0)
+			(at 40.64 23.4184 0)
 			(effects
 				(font
@@
 		)
 		(property "Sheetfile" "power_mcu.kicad_sch"
-			(at 48.26 57.0996 0)
+			(at 40.64 45.6696 0)
 			(effects
 				(font
@@
 		)
 		(pin "+3.3V" output
-			(at 95.25 40.64 0)
+			(at 87.63 29.21 0)
 			(effects
 				(font
@@
 		)
 		(pin "+5V" output
-			(at 95.25 44.45 0)
+			(at 87.63 33.02 0)
 			(effects
 				(font
@@
 		)
 		(pin "VDDA" output
-			(at 95.25 48.26 0)
-			(effects
-				(font
+			(at 87.63 36.83 0)
+			(effects
+				(font

Commit message: update
Other:
- removed sheet led_servo

Commit message: update
Changed lines of the file:
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@@
 	(wire
 		(pts
-			(xy 96.52 116.84) (xy 137.16 116.84)
-		)
-		(stroke
-			(width 0)
-			(type default)
-		)
-	)
-	(wire
-		(pts
-			(xy 152.4 80.01) (xy 152.4 132.08)
-		)
-		(stroke
-			(width 0)
-			(type default)
-		)
-	)
-	(wire
-		(pts
-			(xy 116.84 96.52) (xy 116.84 53.34)
-		)
-		(stroke
-			(width 0)
-			(type default)
-		)
-	)
-	(wire
-		(pts
-			(xy 147.32 127) (xy 147.32 76.2)
-		)
-		(stroke
-			(width 0)
-			(type default)
-		)
-	)
-	(wire
-		(pts
-			(xy 96.52 106.68) (xy 127 106.68)
-		)
-		(stroke
-			(width 0)
-			(type default)
-		)
-	)
-	(wire
-		(pts
-			(xy 132.08 111.76) (xy 132.08 64.77)
-		)
-		(stroke
-			(width 0)
-			(type default)
-		)
-	)
-	(wire
-		(pts
-			(xy 95.25 30.48) (xy 96.52 30.48)
-		)
-		(stroke
-			(width 0)
-			(type default)
-		)
-	)
-	(wire
-		(pts
-			(xy 96.52 121.92) (xy 142.24 121.92)
+			(xy 95.25 82.55) (xy 137.16 82.55)
+		)
+		(stroke
+			(width 0)
+			(type default)
+		)
+	)
+	(wire
+		(pts
+			(xy 152.4 80.01) (xy 152.4 97.79)
+		)
+		(stroke
+			(width 0)
+			(type default)
+		)
+	)
+	(wire
+		(pts
+			(xy 116.84 62.23) (xy 116.84 53.34)
+		)
+		(stroke
+			(width 0)
+			(type default)
+		)
+	)
+	(wire
+		(pts
+			(xy 147.32 92.71) (xy 147.32 76.2)
+		)
+		(stroke
+			(width 0)
+			(type default)
+		)
+	)
+	(wire
+		(pts
+			(xy 95.25 72.39) (xy 127 72.39)
+		)
+		(stroke
+			(width 0)
+			(type default)
+		)
+	)
+	(wire
+		(pts
+			(xy 132.08 77.47) (xy 132.08 64.77)
+		)
+		(stroke
+			(width 0)
+			(type default)
+		)
+	)
+	(wire
+		(pts
+			(xy 95.25 29.21) (xy 212.09 29.21)
+		)
+		(stroke
+			(width 0)
+			(type default)
+		)
+	)
+	(wire
+		(pts
+			(xy 95.25 87.63) (xy 142.24 87.63)
 		)
 		(stroke
@@
 	(wire
 		(pts
-			(xy 96.52 132.08) (xy 152.4 132.08)
-		)
-		(stroke
-			(width 0)
-			(type default)
-		)
-	)
-	(wire
-		(pts
-			(xy 96.52 101.6) (xy 121.92 101.6)
-		)
-		(stroke
-			(width 0)
-			(type default)
-		)
-	)
-	(wire
-		(pts
-			(xy 95.25 34.29) (xy 97.79 34.29)
-		)
-		(stroke
-			(width 0)
-			(type default)
-		)
-	)
-	(wire
-		(pts
-			(xy 137.16 116.84) (xy 137.16 68.58)
+			(xy 95.25 97.79) (xy 152.4 97.79)
+		)
+		(stroke
+			(width 0)
+			(type default)
+		)
+	)
+	(wire
+		(pts
+			(xy 95.25 67.31) (xy 121.92 67.31)
+		)
+		(stroke
+			(width 0)
+			(type default)
+		)
+	)
+	(wire
+		(pts
+			(xy 95.25 33.02) (xy 212.09 33.02)
+		)
+		(stroke
+			(width 0)
+			(type default)
+		)
+	)
+	(wire
+		(pts
+			(xy 137.16 82.55) (xy 137.16 68.58)
 		)
 		(stroke
@@
 	(wire
 		(pts
-			(xy 99.06 36.83) (xy 212.09 36.83)
-		)
-		(stroke
-			(width 0)
-			(type default)
-		)
-	)
-	(wire
-		(pts
-			(xy 96.52 111.76) (xy 132.08 111.76)
-		)
-		(stroke
-			(width 0)
-			(type default)
-		)
-	)
-	(wire
-		(pts
-			(xy 99.06 38.1) (xy 99.06 36.83)
+			(xy 95.25 77.47) (xy 132.08 77.47)
 		)
 		(stroke
@@
 	(wire
 		(pts
-			(xy 96.52 96.52) (xy 116.84 96.52)
-		)
-		(stroke
-			(width 0)
-			(type default)
-		)
-	)
-	(wire
-		(pts
-			(xy 96.52 30.48) (xy 96.52 29.21)
+			(xy 95.25 62.23) (xy 116.84 62.23)
 		)
 		(stroke
@@
 	(wire
 		(pts
-			(xy 97.79 34.29) (xy 97.79 33.02)
-		)
-		(stroke
-			(width 0)
-			(type default)
-		)
-	)
-	(wire
-		(pts
-			(xy 97.79 33.02) (xy 212.09 33.02)
-		)
-		(stroke
-			(width 0)
-			(type default)
-		)
-	)
-	(wire
-		(pts
-			(xy 96.52 127) (xy 147.32 127)
+			(xy 95.25 92.71) (xy 147.32 92.71)
 		)
 		(stroke
@@
 	(wire
 		(pts
-			(xy 121.92 101.6) (xy 121.92 57.15)
+			(xy 121.92 67.31) (xy 121.92 57.15)
 		)
 		(stroke
@@
 	(wire
 		(pts
-			(xy 142.24 121.92) (xy 142.24 72.39)
-		)
-		(stroke
-			(width 0)
-			(type default)
-		)
-	)
-	(wire
-		(pts
-			(xy 95.25 38.1) (xy 99.06 38.1)
-		)
-		(stroke
-			(width 0)
-			(type default)
-		)
-	)
-	(wire
-		(pts
-			(xy 127 106.68) (xy 127 60.96)
-		)
-		(stroke
-			(width 0)
-			(type default)
-		)
-	)
-	(wire
-		(pts
-			(xy 96.52 29.21) (xy 212.09 29.21)
+			(xy 142.24 87.63) (xy 142.24 72.39)
+		)
+		(stroke
+			(width 0)
+			(type default)
+		)
+	)
+	(wire
+		(pts
+			(xy 95.25 36.83) (xy 212.09 36.83)
+		)
+		(stroke
+			(width 0)
+			(type default)
+		)
+	)
+	(wire
+		(pts
+			(xy 127 72.39) (xy 127 60.96)
 		)
 		(stroke
@@
 	)
 	(sheet
-		(at 49.53 90.17)
+		(at 48.26 55.88)
 		(size 46.99 48.895)
 		(exclude_from_sim no)
@@
 		)
 		(property "Sheetname" "power_servo"
-			(at 49.53 89.4584 0)
+			(at 48.26 55.1684 0)
 			(effects
 				(font
@@
 		)
 		(property "Sheetfile" "power_servo.kicad_sch"
-			(at 49.53 139.6496 0)
+			(at 48.26 105.3596 0)
 			(effects
 				(font
@@
 		)
 		(pin "V_M1" output
-			(at 96.52 96.52 0)
+			(at 95.25 62.23 0)
 			(effects
 				(font
@@
 		)
 		(pin "V_M2" output
-			(at 96.52 101.6 0)
+			(at 95.25 67.31 0)
 			(effects
 				(font
@@
 		)
 		(pin "V_M3" output
-			(at 96.52 106.68 0)
+			(at 95.25 72.39 0)
 			(effects
 				(font
@@
 		)
 		(pin "V_M4" output
-			(at 96.52 111.76 0)
+			(at 95.25 77.47 0)
 			(effects
 				(font
@@
 		)
 		(pin "V_M5" output
-			(at 96.52 116.84 0)
+			(at 95.25 82.55 0)
 			(effects
 				(font
@@
 		)
 		(pin "V_M6" output
-			(at 96.52 121.92 0)
+			(at 95.25 87.63 0)
 			(effects
 				(font
@@
 		)
 		(pin "V_M7" output
-			(at 96.52 127 0)
+			(at 95.25 92.71 0)
 			(effects
 				(font
@@
 		)
 		(pin "V_M8" output
-			(at 96.52 132.08 0)
+			(at 95.25 97.79 0)
 			(effects
 				(font
@@
 	)
 	(sheet
-		(at 48.26 25.4)
+		(at 48.26 24.13)
 		(size 46.99 20.955)
 		(exclude_from_sim no)
@@
 		)
 		(property "Sheetname" "power_mcu"
-			(at 48.26 24.6884 0)
+			(at 48.26 23.4184 0)
 			(effects
 				(font
@@
 		)
 		(property "Sheetfile" "power_mcu.kicad_sch"
-			(at 48.26 46.9396 0)
+			(at 48.26 45.6696 0)
 			(effects
 				(font
@@
 		)
 		(pin "+3.3V" output
-			(at 95.25 30.48 0)
+			(at 95.25 29.21 0)
 			(effects
 				(font
@@
 		)
 		(pin "+5V" output
-			(at 95.25 34.29 0)
+			(at 95.25 33.02 0)
 			(effects
 				(font
@@
 		)
 		(pin "VDDA" output
-			(at 95.25 38.1 0)
-			(effects
-				(font
+			(at 95.25 36.83 0)
+			(effects
+				(font
